File: mcu/digital-amplifier2/circuit/AudioPower.sch (KiCad schematic (older format))
At the start: 41 parts, among them U10 LT3094xMSE, U8 TPS54360DDA, U9 LT3045xMSE-1

Commit message: pcb ok
Parts:
- C58, C66: value 22uf -> 10uf
- C59, C67: footprint Capacitor_SMD:C_0805_2012Metric -> Capacitor_SMD:C_1210_3225Metric
- C62, C71: value 1uf -> 100nf
- D7, D8: value 50v 5A -> 60v 3A; footprint Diode_SMD:D_SMB -> Diode_SMD:D_SMA
- L3: footprint Inductor_SMD:L_CommonMode_Wuerth_WE-SL2 -> misc:MSD1278
Connections:
- net +15V: now also C58.1, C59.1, C60.1, C62.1, C65.1
- net GND: no longer C69.1, C72.1, D7.1 (K), R44.1, R46.2
- new net: C69.1, C72.1, D7.1 (K), R44.1, R46.2
Other:
- moved on the sheet: C58, C59, C66, C67
Changed lines of the file:
@@
 $Descr A4 11693 8268
 encoding utf-8
-Sheet 7 10
+Sheet 6 9
 Title ""
 Date ""
@@
 F 0 "L3" H 4375 2303 50  0000 C CNN
 F 1 "150uh" H 4375 2212 50  0000 C CNN
-F 2 "Inductor_SMD:L_CommonMode_Wuerth_WE-SL2" H 4375 2025 50  0001 C CNN
+F 2 "misc:MSD1278" H 4375 2025 50  0001 C CNN
 F 3 "~" H 4375 2025 50  0001 C CNN
 	1    4375 2025
@@
 AR Path="/5F9D81B7/5FF87CA8/5FCADD35" Ref="D8"  Part="1"
 F 0 "D8" V 3554 2604 50  0000 L CNN
-F 1 "50v 5A" V 3645 2604 50  0000 L CNN
-F 2 "Diode_SMD:D_SMB" H 3600 2525 50  0001 C CNN
+F 1 "60v 3A" V 3645 2604 50  0000 L CNN
+F 2 "Diode_SMD:D_SMA" H 3600 2525 50  0001 C CNN
 F 3 "~" H 3600 2525 50  0001 C CNN
 	1    3600 2525
@@
 AR Path="/5F9D81B7/5FF87CA8/5FCB69BF" Ref="D7"  Part="1"
 F 0 "D7" V 3554 1604 50  0000 L CNN
-F 1 "50v 5A" V 3645 1604 50  0000 L CNN
-F 2 "Diode_SMD:D_SMB" H 3600 1525 50  0001 C CNN
+F 1 "60v 3A" V 3645 1604 50  0000 L CNN
+F 2 "Diode_SMD:D_SMA" H 3600 1525 50  0001 C CNN
 F 3 "~" H 3600 1525 50  0001 C CNN
 	1    3600 1525
@@
 AR Path="/5F9D81B7/5FF87CA8/60129F66" Ref="C71"  Part="1"
 F 0 "C71" H 5742 6746 50  0000 L CNN
-F 1 "1uf" H 5742 6655 50  0000 L CNN
+F 1 "100nf" H 5742 6655 50  0000 L CNN
 F 2 "Capacitor_SMD:C_0805_2012Metric" H 5650 6700 50  0001 C CNN
 F 3 "~" H 5650 6700 50  0001 C CNN
@@
 	6050 6950 6050 6800
 Wire Wire Line
-	4900 6950 5275 6950
-Wire Wire Line
-	4500 6950 4900 6950
-Connection ~ 4900 6950
-Wire Wire Line
-	4900 6950 4900 6800
-Wire Wire Line
-	4500 6800 4500 6950
-Wire Wire Line
-	5275 6425 4900 6425
-Wire Wire Line
-	4500 6425 4900 6425
-Connection ~ 4900 6425
-Wire Wire Line
-	4900 6425 4900 6600
-Wire Wire Line
-	4500 6600 4500 6425
+	4500 6950 4500 6800
+Wire Wire Line
+	4900 6800 4900 6950
+Wire Wire Line
+	4500 6425 4500 6600
+Wire Wire Line
+	4900 6600 4900 6425
 $Comp
 L Device:C_Small C?
 U 1 1 601233D8
-P 4900 6700
+P 4500 6700
 AR Path="/5F115848/5FEDDDE8/601233D8" Ref="C?"  Part="1"
 AR Path="/5FBB5CE4/601233D8" Ref="C?"  Part="1"
 AR Path="/5F9D81B7/5FF87CA8/601233D8" Ref="C67"  Part="1"
-F 0 "C67" H 4992 6746 50  0000 L CNN
-F 1 "100uf" H 4992 6655 50  0000 L CNN
+F 0 "C67" H 4592 6746 50  0000 L CNN
+F 1 "100uf" H 4592 6655 50  0000 L CNN
+F 2 "Capacitor_SMD:C_1210_3225Metric" H 4500 6700 50  0001 C CNN
+F 3 "~" H 4500 6700 50  0001 C CNN
+	1    4500 6700
+	1    0    0    -1
+$EndComp
+$Comp
+L Device:C_Small C?
+U 1 1 6011FDF6
+P 4900 6700
+AR Path="/5F115848/5FEDDDE8/6011FDF6" Ref="C?"  Part="1"
+AR Path="/5FBB5CE4/6011FDF6" Ref="C?"  Part="1"
+AR Path="/5F9D81B7/5FF87CA8/6011FDF6" Ref="C66"  Part="1"
+F 0 "C66" H 4992 6746 50  0000 L CNN
+F 1 "10uf" H 4992 6655 50  0000 L CNN
 F 2 "Capacitor_SMD:C_0805_2012Metric" H 4900 6700 50  0001 C CNN
 F 3 "~" H 4900 6700 50  0001 C CNN
 	1    4900 6700
-	1    0    0    -1
-$EndComp
-$Comp
-L Device:C_Small C?
-U 1 1 6011FDF6
-P 4500 6700
-AR Path="/5F115848/5FEDDDE8/6011FDF6" Ref="C?"  Part="1"
-AR Path="/5FBB5CE4/6011FDF6" Ref="C?"  Part="1"
-AR Path="/5F9D81B7/5FF87CA8/6011FDF6" Ref="C66"  Part="1"
-F 0 "C66" H 4592 6746 50  0000 L CNN
-F 1 "22uf" H 4592 6655 50  0000 L CNN
-F 2 "Capacitor_SMD:C_0805_2012Metric" H 4500 6700 50  0001 C CNN
-F 3 "~" H 4500 6700 50  0001 C CNN
-	1    4500 6700
 	1    0    0    -1
 $EndComp
@@
 AR Path="/5F9D81B7/5FF87CA8/601583D0" Ref="C62"  Part="1"
 F 0 "C62" H 2967 6746 50  0000 L CNN
-F 1 "1uf" H 2967 6655 50  0000 L CNN
+F 1 "100nf" H 2967 6655 50  0000 L CNN
 F 2 "Capacitor_SMD:C_0805_2012Metric" H 2875 6700 50  0001 C CNN
 F 3 "~" H 2875 6700 50  0001 C CNN
@@
 	3275 6950 3275 6800
 Wire Wire Line
-	2125 6950 2500 6950
-Wire Wire Line
-	1725 6950 2125 6950
-Connection ~ 2125 6950
-Wire Wire Line
-	2125 6950 2125 6800
-Wire Wire Line
-	1725 6800 1725 6950
-Wire Wire Line
-	2500 6425 2125 6425
-Connection ~ 2125 6425
-Wire Wire Line
-	2125 6425 2125 6600
-Wire Wire Line
-	1725 6600 1725 6425
+	2125 6800 2125 6950
+Wire Wire Line
+	2125 6600 2125 6425
 $Comp
 L Device:C_Small C?
@@
 L Device:C_Small C?
 U 1 1 601583C2
-P 2125 6700
+P 1725 6700
 AR Path="/5F115848/5FEDDDE8/601583C2" Ref="C?"  Part="1"
 AR Path="/5FBB5CE4/601583C2" Ref="C?"  Part="1"
 AR Path="/5F9D81B7/5FF87CA8/601583C2" Ref="C59"  Part="1"
-F 0 "C59" H 2217 6746 50  0000 L CNN
-F 1 "100uf" H 2217 6655 50  0000 L CNN
+F 0 "C59" H 1817 6746 50  0000 L CNN
+F 1 "100uf" H 1817 6655 50  0000 L CNN
+F 2 "Capacitor_SMD:C_1210_3225Metric" H 1725 6700 50  0001 C CNN
+F 3 "~" H 1725 6700 50  0001 C CNN
+	1    1725 6700
+	1    0    0    -1
+$EndComp
+$Comp
+L Device:C_Small C?
+U 1 1 601583BB
+P 2125 6700
+AR Path="/5F115848/5FEDDDE8/601583BB" Ref="C?"  Part="1"
+AR Path="/5FBB5CE4/601583BB" Ref="C?"  Part="1"
+AR Path="/5F9D81B7/5FF87CA8/601583BB" Ref="C58"  Part="1"
+F 0 "C58" H 2217 6746 50  0000 L CNN
+F 1 "10uf" H 2217 6655 50  0000 L CNN
 F 2 "Capacitor_SMD:C_0805_2012Metric" H 2125 6700 50  0001 C CNN
 F 3 "~" H 2125 6700 50  0001 C CNN
@@
 $EndComp
 $Comp
-L Device:C_Small C?
-U 1 1 601583BB
-P 1725 6700
-AR Path="/5F115848/5FEDDDE8/601583BB" Ref="C?"  Part="1"
-AR Path="/5FBB5CE4/601583BB" Ref="C?"  Part="1"
-AR Path="/5F9D81B7/5FF87CA8/601583BB" Ref="C58"  Part="1"
-F 0 "C58" H 1817 6746 50  0000 L CNN
-F 1 "22uf" H 1817 6655 50  0000 L CNN
-F 2 "Capacitor_SMD:C_0805_2012Metric" H 1725 6700 50  0001 C CNN
-F 3 "~" H 1725 6700 50  0001 C CNN
-	1    1725 6700
-	1    0    0    -1
-$EndComp
-$Comp
 L power:+15V #PWR?
 U 1 1 5FD732E6
-P 1725 6200
+P 1725 6225
 AR Path="/5F115848/5FEDDDE8/5FD732E6" Ref="#PWR?"  Part="1"
 AR Path="/5FBB5CE4/5FD732E6" Ref="#PWR?"  Part="1"
 AR Path="/5F9D81B7/5FF87CA8/5FD732E6" Ref="#PWR072"  Part="1"
-F 0 "#PWR072" H 1725 6050 50  0001 C CNN
-F 1 "+15V" H 1740 6373 50  0000 C CNN
-F 2 "" H 1725 6200 50  0001 C CNN
-F 3 "" H 1725 6200 50  0001 C CNN
-	1    1725 6200
+F 0 "#PWR072" H 1725 6075 50  0001 C CNN
+F 1 "+15V" H 1740 6398 50  0000 C CNN
+F 2 "" H 1725 6225 50  0001 C CNN
+F 3 "" H 1725 6225 50  0001 C CNN
+	1    1725 6225
 	1    0    0    -1
 $EndComp
@@
 Wire Wire Line
 	4500 6200 4500 6425
-Connection ~ 4500 6425
-Wire Wire Line
-	1725 6225 1725 6425
-Connection ~ 1725 6425
 $Comp
 L power:GND #PWR?
@@
 	4500 7100 4500 6950
 Wire Wire Line
-	1725 6425 2125 6425
-Connection ~ 4500 6950
-Wire Wire Line
 	1725 7100 1725 6950
-Connection ~ 1725 6950
 Wire Wire Line
 	2950 2875 4175 2875
@@
 	9350 2525 9350 2925
 Connection ~ 5375 2525
-Wire Wire Line
-	5375 2525 4825 2525
 Connection ~ 5850 2525
-Wire Wire Line
-	5850 2525 5375 2525
 Wire Wire Line
 	5375 1800 5375 2525
@@
 Wire Wire Line
 	5850 1800 5850 2525
-Wire Wire Line
-	4825 1225 4825 2125
-Wire Wire Line
-	4650 2125 4825 2125
 Connection ~ 4650 2125
-Connection ~ 4825 2125
-Wire Wire Line
-	4825 2125 4825 2525
 Connection ~ 8600 3850
 Wire Wire Line
@@
 	4825 2875 4825 2975
 Wire Wire Line
-	4825 2525 4825 2625
-Connection ~ 4825 2525
+	1725 6225 1725 6425
+Wire Wire Line
+	1725 6950 1725 6800
+Wire Wire Line
+	1725 6425 1725 6600
+Connection ~ 1725 6425
+Connection ~ 1725 6950
+Wire Wire Line
+	1725 6425 2125 6425
+Wire Wire Line
+	1725 6950 2125 6950
+Connection ~ 2125 6425
+Wire Wire Line
+	2125 6425 2500 6425
+Connection ~ 2125 6950
+Wire Wire Line
+	2125 6950 2500 6950
+Connection ~ 4500 6425
+Connection ~ 4500 6950
+Wire Wire Line
+	4500 6950 4900 6950
+Wire Wire Line
+	4500 6425 4900 6425
+Connection ~ 4900 6425
+Wire Wire Line
+	4900 6425 5275 6425
+Connection ~ 4900 6950
+Wire Wire Line
+	4900 6950 5275 6950
+Wire Wire Line
+	4650 2125 4650 2525
+Wire Wire Line
+	4825 1225 4825 2625
+Wire Wire Line
+	4650 2525 5375 2525
+Wire Wire Line
+	5375 2525 5850 2525
 $EndSCHEMATC
