File: mcu/digital-amplifier2/circuit/TAS6424.sch (KiCad schematic (older format))
At the start: 53 parts, among them J10 Audio outA, J11 Audio outB, J12 Audio outC, J13 Audio outD, U12 TAS6424QDKQRQ1

Commit message: pcb ok
Parts:
- added C32, C33, C34, C35: 100uf, Capacitor_SMD:C_1210_3225Metric, symbol Device:C_Small
- C100, C101, C102, C103, C104, C105, C106, C99: footprint Capacitor_SMD:C_0805_2012Metric -> Capacitor_SMD:C_0603_1608Metric
Connections:
- net labels removed: VCC
- wire segments 233 -> 249
Changed lines of the file:
@@
 $Descr A4 11693 8268
 encoding utf-8
-Sheet 9 10
+Sheet 8 9
 Title ""
 Date ""
@@
 F 0 "C100" H 8042 1496 50  0000 L CNN
 F 1 "1uf" H 8042 1405 50  0000 L CNN
-F 2 "Capacitor_SMD:C_0805_2012Metric" H 7950 1450 50  0001 C CNN
+F 2 "Capacitor_SMD:C_0603_1608Metric" H 7950 1450 50  0001 C CNN
 F 3 "~" H 7950 1450 50  0001 C CNN
 	1    7950 1450
@@
 F 0 "C99" H 8042 1071 50  0000 L CNN
 F 1 "1uf" H 8042 980 50  0000 L CNN
-F 2 "Capacitor_SMD:C_0805_2012Metric" H 7950 1025 50  0001 C CNN
+F 2 "Capacitor_SMD:C_0603_1608Metric" H 7950 1025 50  0001 C CNN
 F 3 "~" H 7950 1025 50  0001 C CNN
 	1    7950 1025
@@
 F 0 "C102" H 8042 2546 50  0000 L CNN
 F 1 "1uf" H 8042 2455 50  0000 L CNN
-F 2 "Capacitor_SMD:C_0805_2012Metric" H 7950 2500 50  0001 C CNN
+F 2 "Capacitor_SMD:C_0603_1608Metric" H 7950 2500 50  0001 C CNN
 F 3 "~" H 7950 2500 50  0001 C CNN
 	1    7950 2500
@@
 F 0 "C101" H 8042 2121 50  0000 L CNN
 F 1 "1uf" H 8042 2030 50  0000 L CNN
-F 2 "Capacitor_SMD:C_0805_2012Metric" H 7950 2075 50  0001 C CNN
+F 2 "Capacitor_SMD:C_0603_1608Metric" H 7950 2075 50  0001 C CNN
 F 3 "~" H 7950 2075 50  0001 C CNN
 	1    7950 2075
@@
 F 0 "C104" H 8042 3596 50  0000 L CNN
 F 1 "1uf" H 8042 3505 50  0000 L CNN
-F 2 "Capacitor_SMD:C_0805_2012Metric" H 7950 3550 50  0001 C CNN
+F 2 "Capacitor_SMD:C_0603_1608Metric" H 7950 3550 50  0001 C CNN
 F 3 "~" H 7950 3550 50  0001 C CNN
 	1    7950 3550
@@
 F 0 "C103" H 8042 3171 50  0000 L CNN
 F 1 "1uf" H 8042 3080 50  0000 L CNN
-F 2 "Capacitor_SMD:C_0805_2012Metric" H 7950 3125 50  0001 C CNN
+F 2 "Capacitor_SMD:C_0603_1608Metric" H 7950 3125 50  0001 C CNN
 F 3 "~" H 7950 3125 50  0001 C CNN
 	1    7950 3125
@@
 F 0 "C106" H 8042 4671 50  0000 L CNN
 F 1 "1uf" H 8042 4580 50  0000 L CNN
-F 2 "Capacitor_SMD:C_0805_2012Metric" H 7950 4625 50  0001 C CNN
+F 2 "Capacitor_SMD:C_0603_1608Metric" H 7950 4625 50  0001 C CNN
 F 3 "~" H 7950 4625 50  0001 C CNN
 	1    7950 4625
@@
 F 0 "C105" H 8042 4246 50  0000 L CNN
 F 1 "1uf" H 8042 4155 50  0000 L CNN
-F 2 "Capacitor_SMD:C_0805_2012Metric" H 7950 4200 50  0001 C CNN
+F 2 "Capacitor_SMD:C_0603_1608Metric" H 7950 4200 50  0001 C CNN
 F 3 "~" H 7950 4200 50  0001 C CNN
 	1    7950 4200
@@
 Text Label 4500 2775 0    50   ~ 0
 BST_4P
-Text Label 7500 875  0    50   ~ 0
+Text Label 7500 1600 0    50   ~ 0
 OUT_1M
-Text Label 7500 1600 0    50   ~ 0
+Text Label 7525 875  0    50   ~ 0
 OUT_1P
+Text Label 7500 1925 0    50   ~ 0
+OUT_2P
 Text Label 7500 2650 0    50   ~ 0
-OUT_2P
-Text Label 7500 1925 0    50   ~ 0
 OUT_2M
+Text Label 7500 3700 0    50   ~ 0
+OUT_3M
 Text Label 7500 2975 0    50   ~ 0
-OUT_3M
-Text Label 7500 3700 0    50   ~ 0
 OUT_3P
+Text Label 7500 4775 0    50   ~ 0
+OUT_4M
 Text Label 7500 4050 0    50   ~ 0
-OUT_4M
-Text Label 7500 4775 0    50   ~ 0
 OUT_4P
+Text Label 7500 1350 0    50   ~ 0
+BST_1M
 Text Label 7500 1125 0    50   ~ 0
-BST_1M
-Text Label 7500 1350 0    50   ~ 0
 BST_1P
+Text Label 7500 2400 0    50   ~ 0
+BST_2M
 Text Label 7500 2175 0    50   ~ 0
-BST_2M
-Text Label 7500 2400 0    50   ~ 0
 BST_2P
+Text Label 7500 3450 0    50   ~ 0
+BST_3M
 Text Label 7500 3225 0    50   ~ 0
-BST_3M
-Text Label 7500 3450 0    50   ~ 0
 BST_3P
+Text Label 7500 4525 0    50   ~ 0
+BST_4M
 Text Label 7500 4300 0    50   ~ 0
-BST_4M
-Text Label 7500 4525 0    50   ~ 0
 BST_4P
 Text HLabel 1100 2775 0    50   Input ~ 0
@@
 $EndComp
 $Comp
-L power:VCC #PWR086
-U 1 1 60674381
-P 725 4775
-F 0 "#PWR086" H 725 4625 50  0001 C CNN
-F 1 "VCC" H 742 4948 50  0000 C CNN
-F 2 "" H 725 4775 50  0001 C CNN
-F 3 "" H 725 4775 50  0001 C CNN
-	1    725  4775
-	1    0    0    -1
-$EndComp
-$Comp
 L Device:C_Small C84
 U 1 1 60675095
@@
 Wire Wire Line
 	1150 6700 1150 6500
-$Comp
-L power:VCC #PWR087
-U 1 1 607AB6F5
-P 1150 6500
-F 0 "#PWR087" H 1150 6350 50  0001 C CNN
-F 1 "VCC" H 1167 6673 50  0000 C CNN
-F 2 "" H 1150 6500 50  0001 C CNN
-F 3 "" H 1150 6500 50  0001 C CNN
-	1    1150 6500
-	1    0    0    -1
-$EndComp
 Connection ~ 725  5425
 Wire Wire Line
@@
 Wire Wire Line
 	1950 7000 1950 7150
+$Comp
+L Device:C_Small C32
+U 1 1 5FC64C70
+P 2325 6900
+F 0 "C32" H 2417 6946 50  0000 L CNN
+F 1 "100uf" H 2417 6855 50  0000 L CNN
+F 2 "Capacitor_SMD:C_1210_3225Metric" H 2325 6900 50  0001 C CNN
+F 3 "~" H 2325 6900 50  0001 C CNN
+	1    2325 6900
+	1    0    0    -1
+$EndComp
+Wire Wire Line
+	2325 6700 2325 6800
+Wire Wire Line
+	2325 7000 2325 7150
+$Comp
+L Device:C_Small C33
+U 1 1 5FC95E47
+P 2725 6900
+F 0 "C33" H 2817 6946 50  0000 L CNN
+F 1 "100uf" H 2817 6855 50  0000 L CNN
+F 2 "Capacitor_SMD:C_1210_3225Metric" H 2725 6900 50  0001 C CNN
+F 3 "~" H 2725 6900 50  0001 C CNN
+	1    2725 6900
+	1    0    0    -1
+$EndComp
+Wire Wire Line
+	2725 6700 2725 6800
+Wire Wire Line
+	2725 7000 2725 7150
+$Comp
+L Device:C_Small C34
+U 1 1 5FCA66DA
+P 3125 6900
+F 0 "C34" H 3217 6946 50  0000 L CNN
+F 1 "100uf" H 3217 6855 50  0000 L CNN
+F 2 "Capacitor_SMD:C_1210_3225Metric" H 3125 6900 50  0001 C CNN
+F 3 "~" H 3125 6900 50  0001 C CNN
+	1    3125 6900
+	1    0    0    -1
+$EndComp
+Wire Wire Line
+	3125 6700 3125 6800
+Wire Wire Line
+	3125 7000 3125 7150
+$Comp
+L Device:C_Small C35
+U 1 1 5FCB73A0
+P 3525 6900
+F 0 "C35" H 3617 6946 50  0000 L CNN
+F 1 "100uf" H 3617 6855 50  0000 L CNN
+F 2 "Capacitor_SMD:C_1210_3225Metric" H 3525 6900 50  0001 C CNN
+F 3 "~" H 3525 6900 50  0001 C CNN
+	1    3525 6900
+	1    0    0    -1
+$EndComp
+Wire Wire Line
+	3525 6700 3525 6800
+Wire Wire Line
+	3525 7000 3525 7150
+Wire Wire Line
+	1950 7150 2325 7150
+Connection ~ 1950 7150
+Wire Wire Line
+	2325 7150 2725 7150
+Connection ~ 2325 7150
+Wire Wire Line
+	2725 7150 3125 7150
+Connection ~ 2725 7150
+Wire Wire Line
+	3125 7150 3525 7150
+Connection ~ 3125 7150
+Wire Wire Line
+	3525 6700 3125 6700
+Wire Wire Line
+	3125 6700 2725 6700
+Connection ~ 3125 6700
+Wire Wire Line
+	2725 6700 2325 6700
+Connection ~ 2725 6700
+Wire Wire Line
+	2325 6700 1950 6700
+Connection ~ 2325 6700
+Connection ~ 1950 6700
+$Comp
+L power:VCCQ #PWR?
+U 1 1 5FCB3AB2
+P 725 4775
+AR Path="/5F16021E/5FCB3AB2" Ref="#PWR?"  Part="1"
+AR Path="/5FC5910D/5FCB3AB2" Ref="#PWR0108"  Part="1"
+F 0 "#PWR0108" H 725 4625 50  0001 C CNN
+F 1 "VCCQ" H 742 4948 50  0000 C CNN
+F 2 "" H 725 4775 50  0001 C CNN
+F 3 "" H 725 4775 50  0001 C CNN
+	1    725  4775
+	1    0    0    -1
+$EndComp
+$Comp
+L power:VCCQ #PWR?
+U 1 1 5FCC61D5
+P 1150 6500
+AR Path="/5F16021E/5FCC61D5" Ref="#PWR?"  Part="1"
+AR Path="/5FC5910D/5FCC61D5" Ref="#PWR0109"  Part="1"
+F 0 "#PWR0109" H 1150 6350 50  0001 C CNN
+F 1 "VCCQ" H 1167 6673 50  0000 C CNN
+F 2 "" H 1150 6500 50  0001 C CNN
+F 3 "" H 1150 6500 50  0001 C CNN
+	1    1150 6500
+	1    0    0    -1
+$EndComp
 $EndSCHEMATC
