File: mcu/digital-amplifier2/circuit/TPA6120A2.sch (KiCad schematic (older format))
At the start: 19 parts, among them J9 AudioJack3_Switch, U11 TPA6120A2DWP

Commit message: pcb ok
Parts:
- U11: symbol ti:TPA6120A2DWP -> digital-amplifier2-rescue:TPA6120A2DWP-ti-digital-amplifier2-rescue
Connections:
- wire segments 87 -> 93
Other:
- moved on the sheet: C79, C80, J9, R54, R55, R56, R57, R58, R59, R60, R61, R62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
