File: mcu/digital-amplifier2/circuit/digital-amplifier2.kicad_pcb (KiCad board)
At the start: 2 copper layers, 100 x 100 mm, 258 parts, among them J1 I2C_oled, J10 Audio outA, J11 Audio outB, J12 Audio outC, J13 Audio outD, J14 Conn_Coaxial, J2 encoder, J3 USB_B, J4 Conn_ARM_JTAG_SWD_20, J5 Barrel_Jack_Switch, J6 AudioJack3_Switch, J7 Conn_Coaxial, J8 Conn_Coaxial, J9 AudioJack3_Switch, Q1 S8550, U1 DLT11H0, U10 LT3094xMSE, U11 TPA6120A2DWP, U12 TAS6424QDKQRQ1, U13 SJR-BTM331, U2 STM32F446RETx, U3 TPS54360DDA, U4 AMS1117-3.3, U5 LT3045xMSE-1, U6 pcm1863, U7 PCM5242, U8 TPS54360DDA, U9 LT3045xMSE-1, Y1 5032 8m, Y2 3225

Commit message: pcb ok
Parts:
- removed C36, C37: 12pf, Capacitor_SMD:C_0805_2012Metric
- removed C38, C40, C43, C45: 10uf, Capacitor_SMD:C_0805_2012Metric
- removed C39, C41: 2.2uf, Capacitor_SMD:C_0805_2012Metric
- removed C42, C44: 100nf, Capacitor_SMD:C_0805_2012Metric
- removed D2: 10v 1A, Diode_SMD:D_SMB
- removed J14: Conn_Coaxial, Connector_Coaxial:U.FL_Molex_MCRF_73412-0110_Vertical
- removed J6: AudioJack3_Switch, Connector_Audio:Jack_3.5mm_Ledino_KB3SPRS_Horizontal
- removed J7, J8: Conn_Coaxial, connector:RCA_x1_3pin
- removed R17: 50Ω, Resistor_SMD:R_0805_2012Metric
- removed R31, R33: 2.2k, Resistor_SMD:R_0805_2012Metric
- removed R32: 10k, Resistor_SMD:R_0805_2012Metric
- removed R34: R_Small, Resistor_SMD:R_0805_2012Metric
- removed R35, R36, R37: 0Ω, Resistor_SMD:R_0805_2012Metric
- removed R72: 0Ω, Resistor_SMD:R_0603_1608Metric
- removed U6: pcm1863, Package_SO:TSSOP-30_4.4x7.8mm_P0.5mm
- removed Y2: 3225, Crystal:Crystal_SMD_3225-4Pin_3.2x2.5mm
- AE1: value Antenna -> Antenna_Shield; moved to B.Cu
- C1, C107, C108, C109, C114, C115, C116, C117, C118, C119, C120, C121, C122, C123, C124, C13, C14, C15, C16, C18, C19, C20, C21, C23, C24, C27, C28, C29, C3, C4, C46, C47, C5, C51, C52, C54, C55, C87, C88, C90, C91, C94, C96, C98, FB1, L1, L11, L2, L4, L7, L8, R14, R15, R18, R19, R20, R21, R38, R40, R41, R44, R45, R60, R69, U13, U3: moved to B.Cu
- C10, C11, C12, C8: footprint Capacitor_SMD:C_0805_2012Metric -> Capacitor_SMD:C_0603_1608Metric
- C100, C101, C102, C103, C104, C105, C106, C6, C7, C99: footprint Capacitor_SMD:C_0805_2012Metric -> Capacitor_SMD:C_0603_1608Metric; moved to B.Cu
- C17: value 5F/5v -> 100nf; footprint misc:Capacitor_5.5V_4F_H -> Resistor_SMD:R_0805_2012Metric; moved to B.Cu
- C25: value 470uf -> 100uf; footprint Capacitor_THT:CP_Radial_D10.0mm_P5.00mm -> Capacitor_SMD:C_1210_3225Metric; moved to B.Cu
- C32, C33, C34, C35: value 10uf -> 100uf; footprint Capacitor_SMD:C_0805_2012Metric -> Capacitor_SMD:C_1210_3225Metric; moved to B.Cu
- C58, C66: value 22uf -> 10uf
- C59, C67: footprint Capacitor_SMD:C_0805_2012Metric -> Capacitor_SMD:C_1210_3225Metric
- C62, C71: value 1uf -> 100nf
- D1: value 40v 5A -> 60v 3A; footprint Diode_SMD:D_SMB -> Diode_SMD:D_SMA; moved to B.Cu
- D3, D4, D5: footprint Diode_SMD:D_SMB -> Diode_SMD:D_SMA; moved to B.Cu
- D7, D8: value 50v 5A -> 60v 3A; footprint Diode_SMD:D_SMB -> Diode_SMD:D_SMA; moved to B.Cu
- L3: footprint Inductor_SMD:L_CommonMode_Wuerth_WE-SL2 -> misc:MSD1278
- Q1: footprint Package_TO_SOT_THT:TO-92_Inline -> Package_TO_SOT_SMD:SOT-23
- R5: footprint Resistor_SMD:R_0805_2012Metric -> Resistor_SMD:R_0603_1608Metric; moved to B.Cu
- TP1, TP2, TP3, TP4, TP5, TP6, TP7, TP8, TP9: footprint TestPoint:TestPoint_Pad_1.5x1.5mm -> TestPoint:TestPoint_Pad_1.0x1.0mm
- moved J10 129.0 mm to (139.2, 56.3)
- moved C34 127.9 mm to (109.1, 94.9), turned to 90 degrees
- moved C35 127.3 mm to (109.2, 87.2), turned to 270 degrees
- moved U9 123.6 mm to (103.3, 118.8), turned to 180 degrees
- moved R25 106.0 mm to (55.4, 133.0), turned to 270 degrees
- moved C33 104.4 mm to (138.3, 94.7), turned to 90 degrees
- moved J11 103.4 mm to (127.4, 56.3)
- moved J1 101.9 mm to (54.0, 105.2)
- moved J2 99.0 mm to (53.7, 126.5), turned to 180 degrees
- moved C76 98.8 mm to (95.9, 111.3), turned to 90 degrees
- moved C90 98.2 mm to (100.3, 85.6), turned to 270 degrees
- moved R3 97.9 mm to (58.0, 111.8)
- moved U11 97.4 mm to (114.1, 137.2), turned to 270 degrees
- moved C32 97.3 mm to (138.3, 87.5), turned to 270 degrees
- moved TP8 97.2 mm to (60.8, 121.7)
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Connections:
- AE1 pad 2: (no net) -> GND
- C100 pad 1: /TAS6424/BST_1P -> /TAS6424/BST_1M
- C100 pad 2: /TAS6424/OUT_1P -> /TAS6424/OUT_1M
- C101 pad 1: /TAS6424/OUT_2M -> /TAS6424/OUT_2P
- C101 pad 2: /TAS6424/BST_2M -> /TAS6424/BST_2P
- C102 pad 1: /TAS6424/BST_2P -> /TAS6424/BST_2M
- C102 pad 2: /TAS6424/OUT_2P -> /TAS6424/OUT_2M
- C103 pad 1: /TAS6424/OUT_3M -> /TAS6424/OUT_3P
- C103 pad 2: /TAS6424/BST_3M -> /TAS6424/BST_3P
- C104 pad 1: /TAS6424/BST_3P -> /TAS6424/BST_3M
- C104 pad 2: /TAS6424/OUT_3P -> /TAS6424/OUT_3M
- C105 pad 1: /TAS6424/OUT_4M -> /TAS6424/OUT_4P
- C105 pad 2: /TAS6424/BST_4M -> /TAS6424/BST_4P
- C106 pad 1: /TAS6424/BST_4P -> /TAS6424/BST_4M
- C106 pad 2: /TAS6424/OUT_4P -> /TAS6424/OUT_4M
- C17 pad 1: Net-(C17-Pad1) -> +3V3
- C18 pad 1: VCC -> /power/powin
- C20 pad 1: Net-(C20-Pad1) -> VCC
- C32 pad 1: /pcm1863/lin_l -> VCCQ
- C32 pad 2: Net-(C32-Pad2) -> GND
- C33 pad 1: /pcm1863/lin_r -> VCCQ
- C33 pad 2: Net-(C33-Pad2) -> GND
- C34 pad 1: /pcm1863/mic_l -> VCCQ
- C34 pad 2: Net-(C34-Pad2) -> GND
- C35 pad 1: /pcm1863/mic_r -> VCCQ
- C35 pad 2: Net-(C35-Pad2) -> GND
- C58 pad 1: Net-(C58-Pad1) -> +15V
- C59 pad 1: Net-(C58-Pad1) -> +15V
- C60 pad 1: Net-(C58-Pad1) -> +15V
- C62 pad 1: Net-(C58-Pad1) -> +15V
- C65 pad 1: Net-(C58-Pad1) -> +15V
- C69 pad 1: GND -> Net-(C69-Pad1)
- C72 pad 1: GND -> Net-(C69-Pad1)
- C81 pad 1: VCC -> VCCQ
- C82 pad 1: VCC -> VCCQ
- C83 pad 1: VCC -> VCCQ
- C84 pad 1: VCC -> VCCQ
- C85 pad 1: VCC -> VCCQ
- C86 pad 1: VCC -> VCCQ
- C89 pad 1: VCC -> VCCQ
- C92 pad 1: VCC -> VCCQ
- C99 pad 1: /TAS6424/OUT_1M -> /TAS6424/OUT_1P
- C99 pad 2: /TAS6424/BST_1M -> /TAS6424/BST_1P
- D3 pad 1: Net-(C20-Pad1) -> VCC
- D4 pad 1: Net-(C20-Pad1) -> VCC
- D7 pad 1: GND -> Net-(C69-Pad1)
- FB1 pad 1: VCC -> /power/powin
- FB1 pad 2: Net-(C20-Pad1) -> VCC
- L1 pad 1: Net-(C20-Pad1) -> VCC
- L10 pad 1: /TAS6424/OUT_3P -> /TAS6424/OUT_3M
- L11 pad 1: /TAS6424/OUT_4P -> /TAS6424/OUT_4M
- L4 pad 1: /TAS6424/OUT_1M -> /TAS6424/OUT_1P
- L5 pad 1: /TAS6424/OUT_2M -> /TAS6424/OUT_2P
- L6 pad 1: /TAS6424/OUT_3M -> /TAS6424/OUT_3P
- L7 pad 1: /TAS6424/OUT_4M -> /TAS6424/OUT_4P
- L8 pad 1: /TAS6424/OUT_1P -> /TAS6424/OUT_1M
- L9 pad 1: /TAS6424/OUT_2P -> /TAS6424/OUT_2M
- R18 pad 1: VCC -> /power/powin
- R44 pad 1: GND -> Net-(C69-Pad1)
- R46 pad 2: GND -> Net-(C69-Pad1)
- R56 pad 1: Net-(C80-Pad1) -> Net-(C80-Pad2)
- R56 pad 2: /Headphone/OUTLP -> /Headphone/OUTLN
- R57 pad 1: Net-(C80-Pad2) -> Net-(C80-Pad1)
- R57 pad 2: /Headphone/OUTLN -> /Headphone/OUTLP
- R58 pad 1: /Headphone/sheet5FF9330D/LOUT -> /Headphone/sheet5FF9330D/ROUT
- R59 pad 1: /Headphone/sheet5FF9330D/ROUT -> /Headphone/sheet5FF9330D/LOUT
- R61 pad 1: /Headphone/sheet5FF9330D/LOUT -> Net-(R61-Pad1)
- R61 pad 2: /Headphone/OUTLN -> /Headphone/sheet5FF9330D/ROUT
- R62 pad 1: /Headphone/sheet5FF9330D/ROUT -> Net-(R62-Pad1)
- R62 pad 2: /Headphone/OUTRN -> /Headphone/sheet5FF9330D/LOUT
- R63 pad 1: /Headphone/OUTRP -> Net-(R63-Pad1)
- R64 pad 1: /Headphone/OUTRN -> Net-(R62-Pad1)
- R65 pad 1: /Headphone/OUTLP -> Net-(R61-Pad1)
- R65 pad 2: Net-(C80-Pad1) -> Net-(C80-Pad2)
- R66 pad 1: /Headphone/OUTLN -> Net-(R66-Pad1)
- R66 pad 2: Net-(C80-Pad2) -> Net-(C80-Pad1)
- R67 pad 1: /Headphone/OUTRP -> Net-(R63-Pad1)
- R68 pad 1: /Headphone/OUTLP -> Net-(R66-Pad1)
- U11 pad 16: /Headphone/OUTLN -> Net-(R61-Pad1)
- U11 pad 17: /Headphone/OUTLP -> Net-(R66-Pad1)
- U11 pad 4: /Headphone/OUTRP -> Net-(R63-Pad1)
- U11 pad 5: /Headphone/OUTRN -> Net-(R62-Pad1)
- U13 pad 46: Net-(J14-Pad1) -> Net-(AE1-Pad1)
- U2 pad 1: /stm32/VBAT -> +3V3
- U2 pad 2: /pcm1863_gp3 -> /headphone_in
- U2 pad 52: /headphone_in -> Net-(U2-Pad52)
- U2 pad 53: /mic_in -> Net-(U2-Pad53)
- U3 pad 2: VCC -> /power/powin
Routing:
- net GND: track 0.00 -> 1819.4 mm, vias 0 -> 46
- net +3V3: track 0.00 -> 363.9 mm, vias 0 -> 10
- net VCCQ: track 0.00 -> 164.6 mm, vias 0 -> 12
- net /SCL: track 0.00 -> 162.7 mm, vias 0 -> 2
- net /SDA: track 0.00 -> 154.0 mm, vias 0 -> 2
- net VCC: track 0.00 -> 129.6 mm, vias 0 -> 1
- net +15V: track 0.00 -> 120.4 mm, vias 0 -> 10
- net /SAI1_SD: track 0.00 -> 117.1 mm, vias 0 -> 4
- net /BT_spdif: track 0.00 -> 114.3 mm, vias 0 -> 1
- net /SAI1_FS: track 0.00 -> 114.0 mm, vias 0 -> 4
- net -15V: track 0.00 -> 111.5 mm, vias 0 -> 2
- net /SAI1_CLK: track 0.00 -> 109.2 mm, vias 0 -> 4
- net +3.3VA: track 0.00 -> 98.3 mm, vias 0 -> 8
- net /BT_en: track 0.00 -> 96.5 mm, vias 0 -> 1
- net /SAI1_MCK: track 0.00 -> 92.3 mm, vias 0 -> 2
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Other:
- net class Default: clearance 0.2 -> 0.15; trace_width 0.25 -> 0.2; via_dia 0.8 -> 0.6; via_drill 0.4 -> 0.3
- net class p1A added: clearance 0.2, trace_width 0.3, via_dia 0.6, via_drill 0.3
- net class signal added: clearance 0.15, trace_width 0.15, via_dia 0.6, via_drill 0.3
- net class vcc added: clearance 0.2, trace_width 2.5, via_dia 0.6, via_drill 0.3
- rule trace_clearance: 0.2 -> 0.15
- rule trace_min: 0.2 -> 0.15
- rule via_min_size: 0.4 -> 0.6
