File: mcu/digital-amplifier2/circuit/digital-amplifier2.sch (KiCad schematic (older format))
At the start: 8 parts

Commit message: pcb ok
Parts:
- TP1, TP2, TP3, TP4, TP5, TP6, TP7, TP8: footprint TestPoint:TestPoint_Pad_1.5x1.5mm -> TestPoint:TestPoint_Pad_1.0x1.0mm
Connections:
- net labels removed: mic_in, pcm1863_gp3
- wire segments 68 -> 58
Changed lines of the file:
@@
 $Descr A4 11693 8268
 encoding utf-8
-Sheet 1 10
+Sheet 1 9
 Title ""
 Date ""
@@
 F18 "tas6424_warn" I R 2125 5175 50
 F19 "tas6424_fault" I R 2125 5275 50
-F20 "mic_in" I R 2125 5425 50
-F21 "headphone_in" I R 2125 4725 50
-F22 "headphone_en" I R 2125 4625 50
-F23 "pcm1863_gp3" I R 2125 5525 50
-F24 "BT_spdif" I R 2125 5775 50
-F25 "BT_state" I R 2125 5875 50
-F26 "BT_en" I R 2125 5975 50
-F27 "BT_bn" I R 2125 5675 50
+F20 "headphone_in" I R 2125 4725 50
+F21 "headphone_en" I R 2125 4625 50
+F22 "BT_spdif" I R 2125 5775 50
+F23 "BT_state" I R 2125 5875 50
+F24 "BT_en" I R 2125 5975 50
+F25 "BT_bn" I R 2125 5675 50
 $EndSheet
 $Sheet
@@
 F0 "power" 50
 F1 "power.sch" 50
-$EndSheet
-$Sheet
-S 8900 4675 1175 1150
-U 5F9D81B4
-F0 "pcm1863" 50
-F1 "pcm1863.sch" 50
-F2 "mic_in" I L 8900 4775 50
-F3 "MCLK" I L 8900 4900 50
-F4 "BCK" I L 8900 5000 50
-F5 "LRCK" I L 8900 5100 50
-F6 "DOUT" I L 8900 5200 50
-F7 "SCL" I L 8900 5325 50
-F8 "SDA" I L 8900 5425 50
-F9 "GP3" I L 8900 5725 50
 $EndSheet
 $Sheet
@@
 SAI1_SD
 Wire Wire Line
-	8900 4775 8275 4775
-Wire Wire Line
-	8900 4900 8275 4900
-Wire Wire Line
-	8900 5000 8275 5000
-Wire Wire Line
-	8900 5100 8275 5100
-Wire Wire Line
-	8900 5200 8275 5200
-Wire Wire Line
-	8900 5325 8275 5325
-Wire Wire Line
-	8900 5425 8275 5425
-Wire Wire Line
-	8900 5725 8275 5725
-Text Label 8350 5325 0    50   ~ 0
-SCL
-Text Label 8350 5425 0    50   ~ 0
-SDA
-Wire Wire Line
 	2125 3025 2900 3025
 Wire Wire Line
@@
 Text Label 2400 4000 0    50   ~ 0
 SAI2_SD
-Text Label 8350 5000 0    50   ~ 0
-SAI2_CLK
-Text Label 8350 5100 0    50   ~ 0
-SAI2_FS
-Text Label 8350 5200 0    50   ~ 0
-SAI2_SD
 Wire Wire Line
 	2125 4625 2900 4625
@@
 Wire Wire Line
 	2125 5275 2900 5275
-Wire Wire Line
-	2125 5425 2900 5425
-Wire Wire Line
-	2125 5525 2900 5525
-Text Label 2275 5525 0    50   ~ 0
-pcm1863_gp3
-Text Label 2275 5425 0    50   ~ 0
-mic_in
 Text Label 2275 5275 0    50   ~ 0
 tas6424_fault
@@
 Wire Wire Line
 	8250 2900 8950 2900
-Text Label 8350 4775 0    50   ~ 0
-mic_in
-Text Label 8325 5725 0    50   ~ 0
-pcm1863_gp3
 Text Label 5125 6775 0    50   ~ 0
 SAI1_CLK
@@
 I2S1_MCK
 $Sheet
-S 5475 3125 950  1325
+S 5575 950  950  1325
 U 5FD6457F
 F0 "Bluetooth" 50
 F1 "Bluetooth.sch" 50
-F2 "CLK" I L 5475 3450 50
-F3 "FS" I L 5475 3550 50
-F4 "SD" I L 5475 3650 50
-F5 "EN" I L 5475 3775 50
-F6 "button" I L 5475 3875 50
-F7 "state" I L 5475 3975 50
-F8 "SPDIF" I L 5475 3200 50
+F2 "CLK" I L 5575 1275 50
+F3 "FS" I L 5575 1375 50
+F4 "SD" I L 5575 1475 50
+F5 "EN" I L 5575 1600 50
+F6 "button" I L 5575 1700 50
+F7 "state" I L 5575 1800 50
+F8 "SPDIF" I L 5575 1025 50
 $EndSheet
 Wire Wire Line
-	5475 3450 5000 3450
-Wire Wire Line
-	5475 3550 5000 3550
-Wire Wire Line
-	5475 3650 5000 3650
-Wire Wire Line
-	5475 3775 5000 3775
-Wire Wire Line
-	5475 3875 5000 3875
-Wire Wire Line
-	5475 3975 5000 3975
-Wire Wire Line
-	5475 3200 5000 3200
+	5575 1275 5100 1275
+Wire Wire Line
+	5575 1375 5100 1375
+Wire Wire Line
+	5575 1475 5100 1475
+Wire Wire Line
+	5575 1600 5100 1600
+Wire Wire Line
+	5575 1700 5100 1700
+Wire Wire Line
+	5575 1800 5100 1800
+Wire Wire Line
+	5575 1025 5100 1025
 Text Label 2400 4275 0    50   ~ 0
 I2S1_SCK
@@
 Text Label 2400 4475 0    50   ~ 0
 I2S1_SD
-Text Label 5025 3450 0    50   ~ 0
+Text Label 5125 1275 0    50   ~ 0
 I2S1_SCK
-Text Label 5025 3550 0    50   ~ 0
+Text Label 5125 1375 0    50   ~ 0
 I2S1_FS
-Text Label 5025 3650 0    50   ~ 0
+Text Label 5125 1475 0    50   ~ 0
 I2S1_SD
-Text Label 5025 3775 0    50   ~ 0
+Text Label 5125 1600 0    50   ~ 0
 BT_en
-Text Label 5025 3875 0    50   ~ 0
+Text Label 5125 1700 0    50   ~ 0
 BT_bn
-Text Label 5025 3975 0    50   ~ 0
+Text Label 5125 1800 0    50   ~ 0
 BT_state
-Text Label 5025 3200 0    50   ~ 0
+Text Label 5125 1025 0    50   ~ 0
 BT_spdif
-Text Label 8350 4900 0    50   ~ 0
-I2S1_MCK
 Wire Wire Line
 	2125 5675 2900 5675
@@
 F 0 "TP1" V 5070 6524 50  0000 C CNN
 F 1 "TestPoint" V 4979 6524 50  0000 C CNN
-F 2 "TestPoint:TestPoint_Pad_1.5x1.5mm" H 5075 6450 50  0001 C CNN
+F 2 "TestPoint:TestPoint_Pad_1.0x1.0mm" H 5075 6450 50  0001 C CNN
 F 3 "~" H 5075 6450 50  0001 C CNN
 	1    4875 6450
@@
 F 0 "TP2" V 5070 6849 50  0000 C CNN
 F 1 "TestPoint" V 4979 6849 50  0000 C CNN
-F 2 "TestPoint:TestPoint_Pad_1.5x1.5mm" H 5075 6775 50  0001 C CNN
+F 2 "TestPoint:TestPoint_Pad_1.0x1.0mm" H 5075 6775 50  0001 C CNN
 F 3 "~" H 5075 6775 50  0001 C CNN
 	1    4875 6775
@@
 F 0 "TP3" V 5070 7149 50  0000 C CNN
 F 1 "TestPoint" V 4979 7149 50  0000 C CNN
-F 2 "TestPoint:TestPoint_Pad_1.5x1.5mm" H 5075 7075 50  0001 C CNN
+F 2 "TestPoint:TestPoint_Pad_1.0x1.0mm" H 5075 7075 50  0001 C CNN
 F 3 "~" H 5075 7075 50  0001 C CNN
 	1    4875 7075
@@
 F 0 "TP4" V 5070 7499 50  0000 C CNN
 F 1 "TestPoint" V 4979 7499 50  0000 C CNN
-F 2 "TestPoint:TestPoint_Pad_1.5x1.5mm" H 5075 7425 50  0001 C CNN
+F 2 "TestPoint:TestPoint_Pad_1.0x1.0mm" H 5075 7425 50  0001 C CNN
 F 3 "~" H 5075 7425 50  0001 C CNN
 	1    4875 7425
@@
 F 0 "TP5" V 6295 6524 50  0000 C CNN
 F 1 "TestPoint" V 6204 6524 50  0000 C CNN
-F 2 "TestPoint:TestPoint_Pad_1.5x1.5mm" H 6300 6450 50  0001 C CNN
+F 2 "TestPoint:TestPoint_Pad_1.0x1.0mm" H 6300 6450 50  0001 C CNN
 F 3 "~" H 6300 6450 50  0001 C CNN
 	1    6100 6450
@@
 F 0 "TP6" V 6295 6849 50  0000 C CNN
 F 1 "TestPoint" V 6204 6849 50  0000 C CNN
-F 2 "TestPoint:TestPoint_Pad_1.5x1.5mm" H 6300 6775 50  0001 C CNN
+F 2 "TestPoint:TestPoint_Pad_1.0x1.0mm" H 6300 6775 50  0001 C CNN
 F 3 "~" H 6300 6775 50  0001 C CNN
 	1    6100 6775
@@
 F 0 "TP7" V 6295 7149 50  0000 C CNN
 F 1 "TestPoint" V 6204 7149 50  0000 C CNN
-F 2 "TestPoint:TestPoint_Pad_1.5x1.5mm" H 6300 7075 50  0001 C CNN
+F 2 "TestPoint:TestPoint_Pad_1.0x1.0mm" H 6300 7075 50  0001 C CNN
 F 3 "~" H 6300 7075 50  0001 C CNN
 	1    6100 7075
@@
 F 0 "TP8" V 6295 7499 50  0000 C CNN
 F 1 "TestPoint" V 6204 7499 50  0000 C CNN
-F 2 "TestPoint:TestPoint_Pad_1.5x1.5mm" H 6300 7425 50  0001 C CNN
+F 2 "TestPoint:TestPoint_Pad_1.0x1.0mm" H 6300 7425 50  0001 C CNN
 F 3 "~" H 6300 7425 50  0001 C CNN
 	1    6100 7425
