File: mcu/digital-amplifier2/circuit/jtag_and_power.sch (KiCad schematic (older format))
At the start: 27 parts, among them J3 USB_B, J4 Conn_ARM_JTAG_SWD_20, Q1 S8550

Commit message: pcb ok
Parts:
- removed C17: 5F/5v, misc:Capacitor_5.5V_4F_H, symbol Device:CP_Small
- removed D2: 10v 1A, Diode_SMD:D_SMB, symbol Device:D_Small
- removed R17: 50Ω, Resistor_SMD:R_0805_2012Metric, symbol Device:R_Small
- added C17: 100nf, Resistor_SMD:R_0805_2012Metric, symbol Device:C_Small
- C10, C11, C12, C8: footprint Capacitor_SMD:C_0805_2012Metric -> Capacitor_SMD:C_0603_1608Metric
- D1: value 40v 5A -> 60v 3A; footprint Diode_SMD:D_SMB -> Diode_SMD:D_SMA
- Q1: footprint Package_TO_SOT_THT:TO-92_Inline -> Package_TO_SOT_SMD:SOT-23
Connections:
- net +3V3: now also C17.1
- net GND: now also C17.2
Changed lines of the file:
@@
 $Descr A4 11693 8268
 encoding utf-8
-Sheet 3 10
+Sheet 3 9
 Title ""
 Date ""
@@
 F 0 "C12" H 2917 6646 50  0000 L CNN
 F 1 "100nf/10v" H 2917 6555 50  0000 L CNN
-F 2 "Capacitor_SMD:C_0805_2012Metric" H 2825 6600 50  0001 C CNN
+F 2 "Capacitor_SMD:C_0603_1608Metric" H 2825 6600 50  0001 C CNN
 F 3 "~" H 2825 6600 50  0001 C CNN
 	1    2825 6600
@@
 F 0 "C11" H 2317 6596 50  0000 L CNN
 F 1 "100nf/10v" H 2317 6505 50  0000 L CNN
-F 2 "Capacitor_SMD:C_0805_2012Metric" H 2225 6550 50  0001 C CNN
+F 2 "Capacitor_SMD:C_0603_1608Metric" H 2225 6550 50  0001 C CNN
 F 3 "~" H 2225 6550 50  0001 C CNN
 	1    2225 6550
@@
 F 0 "C10" H 1717 6596 50  0000 L CNN
 F 1 "100nf/10v" H 1717 6505 50  0000 L CNN
-F 2 "Capacitor_SMD:C_0805_2012Metric" H 1625 6550 50  0001 C CNN
+F 2 "Capacitor_SMD:C_0603_1608Metric" H 1625 6550 50  0001 C CNN
 F 3 "~" H 1625 6550 50  0001 C CNN
 	1    1625 6550
@@
 F 0 "C8" H 1067 6596 50  0000 L CNN
 F 1 "100nf/10v" H 1067 6505 50  0000 L CNN
-F 2 "Capacitor_SMD:C_0805_2012Metric" H 975 6550 50  0001 C CNN
+F 2 "Capacitor_SMD:C_0603_1608Metric" H 975 6550 50  0001 C CNN
 F 3 "~" H 975 6550 50  0001 C CNN
 	1    975  6550
@@
 JTDI
 $Comp
-L Device:CP_Small C?
-U 1 1 5FD99DE8
-P 9075 5375
-AR Path="/5F047EA6/5FD99DE8" Ref="C?"  Part="1"
-AR Path="/5F047EA6/5FD62F96/5FD99DE8" Ref="C17"  Part="1"
-F 0 "C17" H 9163 5421 50  0000 L CNN
-F 1 "5F/5v" H 9163 5330 50  0000 L CNN
-F 2 "misc:Capacitor_5.5V_4F_H" H 9075 5375 50  0001 C CNN
-F 3 "~" H 9075 5375 50  0001 C CNN
-	1    9075 5375
-	1    0    0    -1
-$EndComp
-Wire Wire Line
-	9075 5725 9075 5475
-$Comp
-L Device:D_Small D?
-U 1 1 5FD99DF0
-P 9075 4575
-AR Path="/5F047EA6/5FD99DF0" Ref="D?"  Part="1"
-AR Path="/5F047EA6/5FD62F96/5FD99DF0" Ref="D2"  Part="1"
-F 0 "D2" H 9075 4780 50  0000 C CNN
-F 1 "10v 1A" H 9075 4689 50  0000 C CNN
-F 2 "Diode_SMD:D_SMB" V 9075 4575 50  0001 C CNN
-F 3 "~" V 9075 4575 50  0001 C CNN
-	1    9075 4575
-	0    -1   -1   0
-$EndComp
-$Comp
-L Device:R_Small R?
-U 1 1 5FD99DF7
-P 9075 4975
-AR Path="/5F047EA6/5FD99DF7" Ref="R?"  Part="1"
-AR Path="/5F047EA6/5FD62F96/5FD99DF7" Ref="R17"  Part="1"
-F 0 "R17" H 9134 5021 50  0000 L CNN
-F 1 "50Ω" H 9134 4930 50  0000 L CNN
-F 2 "Resistor_SMD:R_0805_2012Metric" H 9075 4975 50  0001 C CNN
-F 3 "~" H 9075 4975 50  0001 C CNN
-	1    9075 4975
-	1    0    0    -1
-$EndComp
-Wire Wire Line
-	9075 4875 9075 4775
-Wire Wire Line
-	9075 5075 9075 5275
-Wire Wire Line
-	9075 4775 9525 4775
-Connection ~ 9075 4775
-Wire Wire Line
-	9075 4775 9075 4675
-Wire Wire Line
-	9075 4175 9075 4475
-$Comp
 L power:GND #PWR?
 U 1 1 5FD99E05
-P 9075 5725
+P 9075 5100
 AR Path="/5F047EA6/5FD99E05" Ref="#PWR?"  Part="1"
 AR Path="/5F047EA6/5FD62F96/5FD99E05" Ref="#PWR035"  Part="1"
-F 0 "#PWR035" H 9075 5475 50  0001 C CNN
-F 1 "GND" H 9080 5552 50  0000 C CNN
-F 2 "" H 9075 5725 50  0001 C CNN
-F 3 "" H 9075 5725 50  0001 C CNN
-	1    9075 5725
+F 0 "#PWR035" H 9075 4850 50  0001 C CNN
+F 1 "GND" H 9080 4927 50  0000 C CNN
+F 2 "" H 9075 5100 50  0001 C CNN
+F 3 "" H 9075 5100 50  0001 C CNN
+	1    9075 5100
 	1    0    0    -1
 $EndComp
@@
 L power:+3.3V #PWR034
 U 1 1 5FD9AFB0
-P 9075 4175
-F 0 "#PWR034" H 9075 4025 50  0001 C CNN
-F 1 "+3.3V" H 9090 4348 50  0000 C CNN
-F 2 "" H 9075 4175 50  0001 C CNN
-F 3 "" H 9075 4175 50  0001 C CNN
-	1    9075 4175
+P 9075 4375
+F 0 "#PWR034" H 9075 4225 50  0001 C CNN
+F 1 "+3.3V" H 9090 4548 50  0000 C CNN
+F 2 "" H 9075 4375 50  0001 C CNN
+F 3 "" H 9075 4375 50  0001 C CNN
+	1    9075 4375
 	1    0    0    -1
 $EndComp
@@
 F 0 "Q1" H 2816 2629 50  0000 L CNN
 F 1 "S8550" H 2816 2720 50  0000 L CNN
-F 2 "Package_TO_SOT_THT:TO-92_Inline" H 2825 2600 50  0001 L CIN
+F 2 "Package_TO_SOT_SMD:SOT-23" H 2825 2600 50  0001 L CIN
 F 3 "http://www.unisonic.com.tw/datasheet/S8550.pdf" H 2625 2675 50  0001 L CNN
 	1    2625 2675
@@
 P 1975 1150
 F 0 "D1" H 1975 934 50  0000 C CNN
-F 1 "40v 5A" H 1975 1025 50  0000 C CNN
-F 2 "Diode_SMD:D_SMB" H 1975 1150 50  0001 C CNN
+F 1 "60v 3A" H 1975 1025 50  0000 C CNN
+F 2 "Diode_SMD:D_SMA" H 1975 1150 50  0001 C CNN
 F 3 "~" H 1975 1150 50  0001 C CNN
 	1    1975 1150
@@
 	1    0    0    -1
 $EndComp
-$Comp
-L power:PWR_FLAG #FLG03
-U 1 1 5FC1EA42
-P 9525 4475
-F 0 "#FLG03" H 9525 4550 50  0001 C CNN
-F 1 "PWR_FLAG" H 9525 4649 50  0000 C CNN
-F 2 "" H 9525 4475 50  0001 C CNN
-F 3 "~" H 9525 4475 50  0001 C CNN
-	1    9525 4475
-	1    0    0    -1
-$EndComp
-Wire Wire Line
-	9525 4475 9525 4775
-Connection ~ 9525 4775
-Wire Wire Line
-	9525 4775 9725 4775
 Wire Wire Line
 	5525 6225 5525 6025
@@
 Wire Wire Line
 	7550 1475 7550 1350
+$Comp
+L Device:C_Small C17
+U 1 1 5FC9F0DF
+P 9075 4875
+F 0 "C17" H 9167 4921 50  0000 L CNN
+F 1 "100nf" H 9167 4830 50  0000 L CNN
+F 2 "Resistor_SMD:R_0805_2012Metric" H 9075 4875 50  0001 C CNN
+F 3 "~" H 9075 4875 50  0001 C CNN
+	1    9075 4875
+	1    0    0    -1
+$EndComp
+Connection ~ 9075 4775
+Wire Wire Line
+	9075 5100 9075 4975
+Wire Wire Line
+	9075 4375 9075 4775
+Wire Wire Line
+	9075 4775 9725 4775
 $EndSCHEMATC
