File: mcu/digital-amplifier2/circuit/power.sch (KiCad schematic (older format))
At the start: 40 parts, among them J5 Barrel_Jack_Switch, U3 TPS54360DDA, U4 AMS1117-3.3, U5 LT3045xMSE-1

Commit message: pcb ok
Parts:
- removed C25: 470uf, Capacitor_THT:CP_Radial_D10.0mm_P5.00mm, symbol Device:CP_Small
- added C25: 100uf, Capacitor_SMD:C_1210_3225Metric, symbol Device:C_Small
- D3, D4, D5: footprint Diode_SMD:D_SMB -> Diode_SMD:D_SMA
Connections:
- net GND: now also C25.2
- net VCC: now also C20.1, D3.1 (K), D4.1 (K), FB1.2, L1.1; no longer C18.1, FB1.1, R18.1, U3.2 (VIN)
- net VCCQ: now also C25.1
- new net powin: C18.1, FB1.1, R18.1, U3.2 (VIN)
Changed lines of the file:
@@
 $Descr A4 11693 8268
 encoding utf-8
-Sheet 4 10
+Sheet 4 9
 Title ""
 Date ""
@@
 F 0 "D5" H 3325 2430 50  0000 C CNN
 F 1 "B560C" H 3325 2339 50  0000 C CNN
-F 2 "Diode_SMD:D_SMB" V 3325 2225 50  0001 C CNN
+F 2 "Diode_SMD:D_SMA" V 3325 2225 50  0001 C CNN
 F 3 "~" V 3325 2225 50  0001 C CNN
 	1    3325 2225
@@
 Wire Wire Line
 	1925 1500 2050 1500
-Wire Wire Line
-	1575 1300 1575 1925
 Connection ~ 1575 1300
 Wire Wire Line
@@
 L power:VCC #PWR043
 U 1 1 5FC6ED11
-P 3475 3900
-F 0 "#PWR043" H 3475 3750 50  0001 C CNN
-F 1 "VCC" H 3492 4073 50  0000 C CNN
-F 2 "" H 3475 3900 50  0001 C CNN
-F 3 "" H 3475 3900 50  0001 C CNN
-	1    3475 3900
+P 2500 3900
+F 0 "#PWR043" H 2500 3750 50  0001 C CNN
+F 1 "VCC" H 2517 4073 50  0000 C CNN
+F 2 "" H 2500 3900 50  0001 C CNN
+F 3 "" H 2500 3900 50  0001 C CNN
+	1    2500 3900
 	1    0    0    -1
 $EndComp
@@
 $EndComp
 Connection ~ 3225 4575
-$Comp
-L Device:CP_Small C25
-U 1 1 60853A00
-P 3225 4750
-F 0 "C25" H 3313 4796 50  0000 L CNN
-F 1 "470uf" H 3313 4705 50  0000 L CNN
-F 2 "Capacitor_THT:CP_Radial_D10.0mm_P5.00mm" H 3225 4750 50  0001 C CNN
-F 3 "~" H 3225 4750 50  0001 C CNN
-	1    3225 4750
-	1    0    0    -1
-$EndComp
 Wire Wire Line
 	3225 4650 3225 4575
@@
 F 0 "D3" H 1850 4359 50  0000 C CNN
 F 1 "40v 5A" H 1850 4450 50  0000 C CNN
-F 2 "Diode_SMD:D_SMB" H 1850 4575 50  0001 C CNN
+F 2 "Diode_SMD:D_SMA" H 1850 4575 50  0001 C CNN
 F 3 "~" H 1850 4575 50  0001 C CNN
 	1    1850 4575
@@
 $EndComp
 Connection ~ 4675 1500
-$Comp
-L power:PWR_FLAG #FLG05
-U 1 1 5FD58CFC
-P 3800 3900
-F 0 "#FLG05" H 3800 3975 50  0001 C CNN
-F 1 "PWR_FLAG" H 3800 4074 50  0000 C CNN
-F 2 "" H 3800 3900 50  0001 C CNN
-F 3 "~" H 3800 3900 50  0001 C CNN
-	1    3800 3900
-	1    0    0    -1
-$EndComp
 Wire Wire Line
 	3225 4575 3675 4575
-Wire Wire Line
-	3800 3900 3800 4200
 $Comp
 L power:PWR_FLAG #FLG04
@@
 $EndComp
 Wire Wire Line
-	1225 1300 1225 1025
-$Comp
-L power:VCC #PWR036
-U 1 1 5FC052DE
-P 1225 1025
-F 0 "#PWR036" H 1225 875 50  0001 C CNN
-F 1 "VCC" H 1242 1198 50  0000 C CNN
-F 2 "" H 1225 1025 50  0001 C CNN
-F 3 "" H 1225 1025 50  0001 C CNN
-	1    1225 1025
-	1    0    0    -1
-$EndComp
-Connection ~ 1225 1300
-Wire Wire Line
 	2975 1600 2975 2275
 Wire Wire Line
@@
 	2500 4200 2800 4200
 Wire Wire Line
-	3000 4200 3475 4200
-Wire Wire Line
-	3475 3900 3475 4200
+	2500 3900 2500 4200
 Wire Wire Line
 	2000 4575 2125 4575
-Wire Wire Line
-	3475 4200 3800 4200
-Connection ~ 3475 4200
 $Comp
 L Device:R_Small R30
@@
 F 0 "D4" H 2125 4559 50  0000 C CNN
 F 1 "40v 5A" H 2125 4650 50  0000 C CNN
-F 2 "Diode_SMD:D_SMB" H 2125 4775 50  0001 C CNN
+F 2 "Diode_SMD:D_SMA" H 2125 4775 50  0001 C CNN
 F 3 "~" H 2125 4775 50  0001 C CNN
 	1    2125 4775
@@
 Wire Wire Line
 	4550 4575 4625 4575
+$Comp
+L Device:C_Small C25
+U 1 1 5FC3FB60
+P 3225 4750
+F 0 "C25" H 3317 4796 50  0000 L CNN
+F 1 "100uf" H 3317 4705 50  0000 L CNN
+F 2 "Capacitor_SMD:C_1210_3225Metric" H 3225 4750 50  0001 C CNN
+F 3 "~" H 3225 4750 50  0001 C CNN
+	1    3225 4750
+	1    0    0    -1
+$EndComp
+Connection ~ 2500 4200
+Wire Wire Line
+	3000 4200 3800 4200
+Wire Wire Line
+	1575 1000 1575 1300
+$Comp
+L power:PWR_FLAG #FLG05
+U 1 1 5FD58CFC
+P 1575 1000
+F 0 "#FLG05" H 1575 1075 50  0001 C CNN
+F 1 "PWR_FLAG" H 1575 1174 50  0000 C CNN
+F 2 "" H 1575 1000 50  0001 C CNN
+F 3 "~" H 1575 1000 50  0001 C CNN
+	1    1575 1000
+	1    0    0    -1
+$EndComp
+Wire Wire Line
+	1575 1300 1575 1925
+Wire Wire Line
+	1225 1300 750  1300
+Connection ~ 1225 1300
+Text Label 850  1300 0    50   ~ 0
+powin
+Text Label 3525 4200 0    50   ~ 0
+powin
+Wire Wire Line
+	1925 3900 1925 4200
+$Comp
+L power:PWR_FLAG #FLG0101
+U 1 1 5FD2F2F0
+P 1925 3900
+F 0 "#FLG0101" H 1925 3975 50  0001 C CNN
+F 1 "PWR_FLAG" H 1925 4074 50  0000 C CNN
+F 2 "" H 1925 3900 50  0001 C CNN
+F 3 "~" H 1925 3900 50  0001 C CNN
+	1    1925 3900
+	1    0    0    -1
+$EndComp
+Wire Wire Line
+	1925 4200 2500 4200
 $EndSCHEMATC
