File: mcu/digital-amplifier2/circuit/stm32.sch (KiCad schematic (older format))
At the start: 17 parts, among them J1 I2C_oled, J2 encoder, U1 DLT11H0, U2 STM32F446RETx, Y1 5032 8m

Commit message: pcb ok
Parts:
- C6, C7: footprint Capacitor_SMD:C_0805_2012Metric -> Capacitor_SMD:C_0603_1608Metric
- R5: footprint Resistor_SMD:R_0805_2012Metric -> Resistor_SMD:R_0603_1608Metric
Connections:
- net labels removed: mic_in, pcm1863_gp3
- wire segments 121 -> 119
- no-connect marks 10 -> 12
Changed lines of the file:
@@
 $Descr A4 11693 8268
 encoding utf-8
-Sheet 2 10
+Sheet 2 9
 Title ""
 Date ""
@@
 F 0 "C7" H 6067 7346 50  0000 L CNN
 F 1 "12pf" H 6067 7255 50  0000 L CNN
-F 2 "Capacitor_SMD:C_0805_2012Metric" H 5975 7300 50  0001 C CNN
+F 2 "Capacitor_SMD:C_0603_1608Metric" H 5975 7300 50  0001 C CNN
 F 3 "~" H 5975 7300 50  0001 C CNN
 	1    5975 7300
@@
 F 0 "C6" H 5467 7346 50  0000 L CNN
 F 1 "12pf" H 5467 7255 50  0000 L CNN
-F 2 "Capacitor_SMD:C_0805_2012Metric" H 5375 7300 50  0001 C CNN
+F 2 "Capacitor_SMD:C_0603_1608Metric" H 5375 7300 50  0001 C CNN
 F 3 "~" H 5375 7300 50  0001 C CNN
 	1    5375 7300
@@
 F 0 "R5" V 5479 6850 50  0000 C CNN
 F 1 "1mΩ" V 5570 6850 50  0000 C CNN
-F 2 "Resistor_SMD:R_0805_2012Metric" H 5675 6850 50  0001 C CNN
+F 2 "Resistor_SMD:R_0603_1608Metric" H 5675 6850 50  0001 C CNN
 F 3 "~" H 5675 6850 50  0001 C CNN
 	1    5675 6850
@@
 Text HLabel 8200 3200 2    50   Input ~ 0
 headphone_en
-Text HLabel 5875 4100 0    50   Input ~ 0
+Text HLabel 5875 4300 0    50   Input ~ 0
 headphone_in
 Text HLabel 8200 3100 2    50   Input ~ 0
@@
 Text HLabel 5875 4400 0    50   Input ~ 0
 tas6424_fault
-Text HLabel 5875 4300 0    50   Input ~ 0
-pcm1863_gp3
 Wire Wire Line
 	7650 1400 8200 1400
@@
 encoder_b
 Wire Wire Line
-	6250 4100 5875 4100
+	6250 4300 5875 4300
 Wire Wire Line
 	6250 4400 5875 4400
 Wire Wire Line
 	6250 4000 5875 4000
-Wire Wire Line
-	6250 4300 5875 4300
-Wire Wire Line
-	6250 4200 5875 4200
 $Comp
 L power:+3.3V #PWR010
@@
 	5875 4500 6250 4500
 NoConn ~ 6250 3900
-Text HLabel 5875 4200 0    50   Input ~ 0
-mic_in
 Wire Wire Line
 	7650 4300 8175 4300
@@
 	1    0    0    -1
 $EndComp
+NoConn ~ 6250 4100
+NoConn ~ 6250 4200
 $EndSCHEMATC
