File: mcu/digital-amplifier2/circuit_main/TAS6424.sch (KiCad schematic (older format))
At the start: 57 parts, among them J10 Audio outA, J11 Audio outB, J12 Audio outC, J13 Audio outD, U12 TAS6424QDKQRQ1

Commit message: pcb ok
Parts:
- removed C107, C83, C84, C89, C92: 10uf, Capacitor_SMD:C_0805_2012Metric, symbol Device:C_Small
- removed C116, C85, C86: 100nf, Capacitor_SMD:C_0805_2012Metric, symbol Device:C_Small
- removed C32, C33, C34, C35: 100uf, Capacitor_SMD:C_1210_3225Metric, symbol Device:C_Small
- removed C81, C82: 100uf, Capacitor_SMD:C_0805_2012Metric, symbol Device:C_Small
- removed C94: 1uf, Capacitor_SMD:C_0805_2012Metric, symbol Device:C_Small
- removed C96, C98: 2.2uf, Capacitor_SMD:C_0805_2012Metric, symbol Device:C_Small
- removed R69: 0Ω, Resistor_SMD:R_0805_2012Metric, symbol Device:R_Small
- removed unit 2 of U12
Connections:
- net labels added: gnd_x, vcc_x
- net labels removed: +3.3V, GND, VCCQ, vdd
- wire segments 249 -> 147
