File: mcu/digital-amplifier2/circuit_main/stm32.sch (KiCad schematic (older format))
At the start: 17 parts, among them J1 I2C_oled, J2 encoder, U1 DLT11H0, U2 STM32F446RETx, Y1 5032 8m

Commit message: pcb ok
Parts:
- added C13: 10uf, Capacitor_SMD:C_0805_2012Metric, symbol Device:C_Small
- added C14: 100nf, Capacitor_SMD:C_0805_2012Metric, symbol Device:C_Small
- added R12: 0Ω, Resistor_SMD:R_0805_2012Metric, symbol Device:R_Small
- C6, C7: footprint Capacitor_SMD:C_0805_2012Metric -> Capacitor_SMD:C_0603_1608Metric
- R5: footprint Resistor_SMD:R_0805_2012Metric -> Resistor_SMD:R_0603_1608Metric
Connections:
- net labels added: +3.3VA, headphone_irq
- net labels removed: I2S1_MCK, SAI1_A_FS, SAI1_A_SCK
- wire segments 119 -> 128
- no-connect marks 12 -> 14
Changed lines of the file:
@@
 $Descr A4 11693 8268
 encoding utf-8
-Sheet 2 9
+Sheet 2 7
 Title ""
 Date ""
@@
 F 0 "C7" H 6067 7346 50  0000 L CNN
 F 1 "12pf" H 6067 7255 50  0000 L CNN
-F 2 "Capacitor_SMD:C_0805_2012Metric" H 5975 7300 50  0001 C CNN
+F 2 "Capacitor_SMD:C_0603_1608Metric" H 5975 7300 50  0001 C CNN
 F 3 "~" H 5975 7300 50  0001 C CNN
 	1    5975 7300
@@
 F 0 "C6" H 5467 7346 50  0000 L CNN
 F 1 "12pf" H 5467 7255 50  0000 L CNN
-F 2 "Capacitor_SMD:C_0805_2012Metric" H 5375 7300 50  0001 C CNN
+F 2 "Capacitor_SMD:C_0603_1608Metric" H 5375 7300 50  0001 C CNN
 F 3 "~" H 5375 7300 50  0001 C CNN
 	1    5375 7300
@@
 F 0 "R5" V 5479 6850 50  0000 C CNN
 F 1 "1mΩ" V 5570 6850 50  0000 C CNN
-F 2 "Resistor_SMD:R_0805_2012Metric" H 5675 6850 50  0001 C CNN
+F 2 "Resistor_SMD:R_0603_1608Metric" H 5675 6850 50  0001 C CNN
 F 3 "~" H 5675 6850 50  0001 C CNN
 	1    5675 6850
@@
 SPDIF_RX
 Wire Wire Line
-	6250 3400 5525 3400
-Wire Wire Line
 	7650 1800 8200 1800
 Wire Wire Line
@@
 Text HLabel 8200 2300 2    50   Input ~ 0
 SAI1_B_SD
-Text HLabel 8200 1700 2    50   Input ~ 0
-SAI1_A_FS
 Text HLabel 8175 4000 2    50   Input ~ 0
 SAI1_B_FS
-Text HLabel 8175 4100 2    50   Input ~ 0
-SAI1_A_SCK
 Wire Wire Line
 	7650 3700 8175 3700
@@
 Text HLabel 8175 3800 2    50   Input ~ 0
 I2C_SDA
-Wire Wire Line
-	7650 1700 8200 1700
 Wire Wire Line
 	7650 1900 8200 1900
@@
 F9 "JTDI" I R 1550 1700 50
 F10 "VBAT" I R 1550 1950 50
-F11 "AVDD" I R 1550 2075 50
-F12 "USB_CONNECT" I R 1550 1800 50
+F11 "USB_CONNECT" I R 1550 1800 50
 $EndSheet
 Text Label 1700 1000 0    50   ~ 0
@@
 	6950 1200 6950 850
 Wire Wire Line
-	1550 2075 2000 2075
-Text Label 1700 2075 0    50   ~ 0
-AVDD
-Wire Wire Line
 	7250 1200 7250 850
 Text Label 7250 950  0    50   ~ 0
@@
 Wire Wire Line
 	8175 4000 7650 4000
-Wire Wire Line
-	7650 4100 8175 4100
 Text HLabel 8200 1900 2    50   Input ~ 0
 I2S1_SCK
 Text HLabel 8200 2100 2    50   Input ~ 0
 I2S1_SD
-Text HLabel 5525 3400 0    50   Input ~ 0
-I2S1_MCK
 Wire Wire Line
 	5525 3100 6250 3100
@@
 $EndComp
 NoConn ~ 6250 4100
-NoConn ~ 6250 4200
+NoConn ~ 6250 3400
+NoConn ~ 7650 1700
+NoConn ~ 7650 4100
+Text HLabel 5875 4200 0    50   Input ~ 0
+headphone_irq
+Wire Wire Line
+	6250 4200 5875 4200
+$Comp
+L Device:C_Small C13
+U 1 1 5FD63401
+P 3825 1600
+AR Path="/5F047EA6/5FD63401" Ref="C13"  Part="1"
+AR Path="/5F047EA6/5FD62F96/5FD63401" Ref="C?"  Part="1"
+F 0 "C13" H 3917 1646 50  0000 L CNN
+F 1 "10uf" H 3917 1555 50  0000 L CNN
+F 2 "Capacitor_SMD:C_0805_2012Metric" H 3825 1600 50  0001 C CNN
+F 3 "~" H 3825 1600 50  0001 C CNN
+	1    3825 1600
+	1    0    0    -1
+$EndComp
+$Comp
+L power:GND #PWR027
+U 1 1 5FD63408
+P 3825 2150
+AR Path="/5F047EA6/5FD63408" Ref="#PWR027"  Part="1"
+AR Path="/5F047EA6/5FD62F96/5FD63408" Ref="#PWR?"  Part="1"
+F 0 "#PWR027" H 3825 1900 50  0001 C CNN
+F 1 "GND" H 3830 1977 50  0000 C CNN
+F 2 "" H 3825 2150 50  0001 C CNN
+F 3 "" H 3825 2150 50  0001 C CNN
+	1    3825 2150
+	1    0    0    -1
+$EndComp
+Wire Wire Line
+	3825 2150 3825 1900
+Wire Wire Line
+	3825 1500 3825 1275
+$Comp
+L Device:R_Small R?
+U 1 1 5FD63410
+P 3400 1275
+AR Path="/5F047EA6/5FD62F96/5FD63410" Ref="R?"  Part="1"
+AR Path="/5F047EA6/5FD63410" Ref="R12"  Part="1"
+F 0 "R12" V 3204 1275 50  0000 C CNN
+F 1 "0Ω" V 3295 1275 50  0000 C CNN
+F 2 "Resistor_SMD:R_0805_2012Metric" H 3400 1275 50  0001 C CNN
+F 3 "~" H 3400 1275 50  0001 C CNN
+	1    3400 1275
+	0    1    1    0
+$EndComp
+Wire Wire Line
+	3125 1275 3125 950
+Wire Wire Line
+	3500 1275 3825 1275
+Connection ~ 3825 1900
+Wire Wire Line
+	3825 1900 3825 1700
+Connection ~ 3825 1275
+$Comp
+L Device:C_Small C14
+U 1 1 5FD6341D
+P 4300 1600
+AR Path="/5F047EA6/5FD6341D" Ref="C14"  Part="1"
+AR Path="/5F047EA6/5FD62F96/5FD6341D" Ref="C?"  Part="1"
+F 0 "C14" H 4392 1646 50  0000 L CNN
+F 1 "100nf" H 4392 1555 50  0000 L CNN
+F 2 "Capacitor_SMD:C_0805_2012Metric" H 4300 1600 50  0001 C CNN
+F 3 "~" H 4300 1600 50  0001 C CNN
+	1    4300 1600
+	1    0    0    -1
+$EndComp
+Wire Wire Line
+	4300 1500 4300 1275
+Wire Wire Line
+	4300 1900 4300 1700
+Wire Wire Line
+	3825 1900 4300 1900
+Wire Wire Line
+	3825 1275 4300 1275
+Connection ~ 4300 1275
+Wire Wire Line
+	4300 1275 4625 1275
+$Comp
+L power:PWR_FLAG #FLG?
+U 1 1 5FD6342A
+P 4300 1075
+AR Path="/5F047EA6/5FD62F96/5FD6342A" Ref="#FLG?"  Part="1"
+AR Path="/5F047EA6/5FD6342A" Ref="#FLG02"  Part="1"
+F 0 "#FLG02" H 4300 1150 50  0001 C CNN
+F 1 "PWR_FLAG" H 4300 1249 50  0000 C CNN
+F 2 "" H 4300 1075 50  0001 C CNN
+F 3 "~" H 4300 1075 50  0001 C CNN
+	1    4300 1075
+	1    0    0    -1
+$EndComp
+Wire Wire Line
+	4300 1275 4300 1075
+$Comp
+L power:+3.3VA #PWR?
+U 1 1 5FD63431
+P 3125 950
+AR Path="/5F047EA6/5FD62F96/5FD63431" Ref="#PWR?"  Part="1"
+AR Path="/5F047EA6/5FD63431" Ref="#PWR026"  Part="1"
+F 0 "#PWR026" H 3125 800 50  0001 C CNN
+F 1 "+3.3VA" H 3140 1123 50  0000 C CNN
+F 2 "" H 3125 950 50  0001 C CNN
+F 3 "" H 3125 950 50  0001 C CNN
+	1    3125 950
+	1    0    0    -1
+$EndComp
+Wire Wire Line
+	3125 1275 3300 1275
+Text Label 4400 1275 0    50   ~ 0
+AVDD
 $EndSCHEMATC
