File: mcu/digital-amplifier2/circuit/main/AudioPower.sch (KiCad schematic (older format))
At the start: 41 parts, among them U10 LT3094xMSE, U8 TPS54360DDA, U9 LT3045xMSE-1

Commit message: headphone
Parts:
- removed C58, C60, C66, C68: 10uf, Capacitor_SMD:C_0805_2012Metric, symbol Device:C_Small
- removed C59, C67: 100uf, Capacitor_SMD:C_1210_3225Metric, symbol Device:C_Small
- removed C62, C65, C71, C74: 100nf, Capacitor_SMD:C_0805_2012Metric, symbol Device:C_Small
- removed R46, R48: 0Ω, Resistor_SMD:R_0805_2012Metric, symbol Device:R_Small
- removed R47, R49: test point, Resistor_SMD:R_0805_2012Metric, symbol Device:R_Small
- renumbered C56 to C35, C57 to C36, C61 to C40, C63 to C42, C64 to C43, C69 to C48, C70 to C49, C72 to C51, C73 to C52, C75 to C54, C76 to C55, C77 to C56, C78 to C57, D7 to D1, D8 to D2, L3 to L1, R42 to R31, R43 to R32, R44 to R33, R45 to R34, R50 to R35, R51 to R36, R52 to R37, R53 to R38, U8 to U6, U9 to U7, U10 to U8
Connections:
- net at U8.1 (IN), U8.13 (IN), U8.2 (IN)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: now also C36.2, C40.2, C43.2, C49.2, C52.2, D2.2 (A), R31.2, R34.2, U6.7 (GND), U6.9 (GNDPAD)
- net at C48.1, C51.1, D1.1 (K)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: now also U7.1 (IN), U7.2 (IN), U7.4 (EN/UV), U7.7 (PGFB)
- no-connect marks 0 -> 2
