File: mcu/digital-amplifier2/circuit/main/AudioPower.sch (KiCad schematic (older format))
At the start: 35 parts, among them U10 LT3094xMSE, U7 TPS54360DDA, U8 TPS54360DDA, U9 LT3045xMSE-1

Commit message: digital-amplifier2-v3
Parts:
- C37, C40: value 1.3pf -> 220pF
- C39, C42: value 1.2nf -> 4.3nF
- R26, R27: value 121k -> 97.6kOhm
- R28, R29: value 68.1k -> 18.7kOhm
Changed lines of the file:
@@
 AR Path="/6035C8F0/5FF87CA8/5FC86ACF" Ref="R27"  Part="1"
 F 0 "R27" H 1809 5646 50  0000 L CNN
-F 1 "121k" H 1809 5555 50  0000 L CNN
+F 1 "97.6kOhm" H 1809 5555 50  0000 L CNN
 F 2 "Resistor_SMD:R_0805_2012Metric" H 1750 5600 50  0001 C CNN
 F 3 "~" H 1750 5600 50  0001 C CNN
@@
 AR Path="/6035C8F0/5FF87CA8/5FC8921F" Ref="R29"  Part="1"
 F 0 "R29" H 3059 5696 50  0000 L CNN
-F 1 "68.1k" H 3059 5605 50  0000 L CNN
+F 1 "18.7kOhm" H 3059 5605 50  0000 L CNN
 F 2 "Resistor_SMD:R_0805_2012Metric" H 3000 5650 50  0001 C CNN
 F 3 "~" H 3000 5650 50  0001 C CNN
@@
 AR Path="/6035C8F0/5FF87CA8/5FC892F9" Ref="C42"  Part="1"
 F 0 "C42" H 3092 6021 50  0000 L CNN
-F 1 "1.2nf" H 3092 5930 50  0000 L CNN
+F 1 "4.3nF" H 3092 5930 50  0000 L CNN
 F 2 "Capacitor_SMD:C_0805_2012Metric" H 3000 5975 50  0001 C CNN
 F 3 "~" H 3000 5975 50  0001 C CNN
@@
 AR Path="/6035C8F0/5FF87CA8/5FC89457" Ref="C40"  Part="1"
 F 0 "C40" H 2742 5821 50  0000 L CNN
-F 1 "1.3pf" H 2742 5730 50  0000 L CNN
+F 1 "220pF" H 2742 5730 50  0000 L CNN
 F 2 "Capacitor_SMD:C_0805_2012Metric" H 2650 5775 50  0001 C CNN
 F 3 "~" H 2650 5775 50  0001 C CNN
@@
 AR Path="/6035C8F0/5FF87CA8/6068367B" Ref="R28"  Part="1"
 F 0 "R28" H 2509 2246 50  0000 L CNN
-F 1 "68.1k" H 2509 2155 50  0000 L CNN
+F 1 "18.7kOhm" H 2509 2155 50  0000 L CNN
 F 2 "Resistor_SMD:R_0805_2012Metric" H 2450 2200 50  0001 C CNN
 F 3 "~" H 2450 2200 50  0001 C CNN
@@
 AR Path="/6035C8F0/5FF87CA8/60683681" Ref="C39"  Part="1"
 F 0 "C39" H 2542 2571 50  0000 L CNN
-F 1 "1.2nf" H 2542 2480 50  0000 L CNN
+F 1 "4.3nF" H 2542 2480 50  0000 L CNN
 F 2 "Capacitor_SMD:C_0805_2012Metric" H 2450 2525 50  0001 C CNN
 F 3 "~" H 2450 2525 50  0001 C CNN
@@
 AR Path="/6035C8F0/5FF87CA8/60683687" Ref="C37"  Part="1"
 F 0 "C37" H 2192 2371 50  0000 L CNN
-F 1 "1.3pf" H 2192 2280 50  0000 L CNN
+F 1 "220pF" H 2192 2280 50  0000 L CNN
 F 2 "Capacitor_SMD:C_0805_2012Metric" H 2100 2325 50  0001 C CNN
 F 3 "~" H 2100 2325 50  0001 C CNN
@@
 AR Path="/6035C8F0/5FF87CA8/606D6645" Ref="R26"  Part="1"
 F 0 "R26" H 1309 2121 50  0000 L CNN
-F 1 "121k" H 1309 2030 50  0000 L CNN
+F 1 "97.6kOhm" H 1309 2030 50  0000 L CNN
 F 2 "Resistor_SMD:R_0805_2012Metric" H 1250 2075 50  0001 C CNN
 F 3 "~" H 1250 2075 50  0001 C CNN
@@
 Wire Wire Line
 	3425 6250 4075 6250
-Entry Wire Line
-	3350 6175 3450 6275
 $EndSCHEMATC
