File: mcu/digital-amplifier2/circuit/main/Bluetooth.sch (KiCad schematic (older format))
At the start: 9 parts, among them J7 Conn_Coaxial, U13 SJR-BTM331

Commit message: headphone
Parts:
- removed D10, D9: LED, LED_SMD:LED_0805_2012Metric, symbol Device:LED
- removed J7: Conn_Coaxial, Connector_Coaxial:U.FL_Hirose_U.FL-R-SMT-1_Vertical, symbol Connector:Conn_Coaxial
- removed R70, R71: 1k, Resistor_SMD:R_0805_2012Metric, symbol Device:R_Small
- added AE1: Antenna_Shield, RF_Antenna:Texas_SWRA117D_2.4GHz_Left, symbol Device:Antenna_Shield
Connections:
- net labels removed: SPDIF
- wire segments 52 -> 37
- no-connect marks 35 -> 38
Changed lines of the file:
@@
 $Descr A4 11693 8268
 encoding utf-8
-Sheet 7 7
+Sheet 5 8
 Title ""
 Date ""
@@
 Text HLabel 6175 5525 2    50   Input ~ 0
 state
-Text HLabel 3100 2025 0    50   Input ~ 0
-SPDIF
-Wire Wire Line
-	3550 2375 3550 2025
-Wire Wire Line
-	3550 2025 3100 2025
 NoConn ~ 2850 4025
 NoConn ~ 3550 6275
-$Comp
-L Device:R_Small R70
-U 1 1 5FD79927
-P 2275 5925
-F 0 "R70" H 2334 5971 50  0000 L CNN
-F 1 "1k" H 2334 5880 50  0000 L CNN
-F 2 "Resistor_SMD:R_0805_2012Metric" H 2275 5925 50  0001 C CNN
-F 3 "~" H 2275 5925 50  0001 C CNN
-	1    2275 5925
-	1    0    0    -1
-$EndComp
-$Comp
-L Device:R_Small R71
-U 1 1 5FD7999C
-P 2600 5925
-F 0 "R71" H 2659 5971 50  0000 L CNN
-F 1 "1k" H 2659 5880 50  0000 L CNN
-F 2 "Resistor_SMD:R_0805_2012Metric" H 2600 5925 50  0001 C CNN
-F 3 "~" H 2600 5925 50  0001 C CNN
-	1    2600 5925
-	1    0    0    -1
-$EndComp
-$Comp
-L Device:LED D9
-U 1 1 5FD79E0B
-P 2275 6300
-F 0 "D9" V 2220 6378 50  0000 L CNN
-F 1 "LED" V 2311 6378 50  0000 L CNN
-F 2 "LED_SMD:LED_0805_2012Metric" H 2275 6300 50  0001 C CNN
-F 3 "~" H 2275 6300 50  0001 C CNN
-	1    2275 6300
-	0    1    1    0
-$EndComp
-$Comp
-L Device:LED D10
-U 1 1 5FD79E88
-P 2600 6325
-F 0 "D10" V 2545 6403 50  0000 L CNN
-F 1 "LED" V 2636 6403 50  0000 L CNN
-F 2 "LED_SMD:LED_0805_2012Metric" H 2600 6325 50  0001 C CNN
-F 3 "~" H 2600 6325 50  0001 C CNN
-	1    2600 6325
-	0    1    1    0
-$EndComp
-Wire Wire Line
-	2600 5825 2600 5525
-Wire Wire Line
-	2600 5525 2850 5525
-Wire Wire Line
-	2850 5375 2275 5375
-Wire Wire Line
-	2275 5375 2275 5825
-Wire Wire Line
-	2275 6025 2275 6150
-Wire Wire Line
-	2600 6025 2600 6175
-Wire Wire Line
-	2600 6475 2600 6650
-Wire Wire Line
-	2600 6650 2450 6650
-Wire Wire Line
-	2275 6650 2275 6450
-Wire Wire Line
-	3025 6825 2450 6825
-Wire Wire Line
-	2450 6825 2450 6650
-Connection ~ 2450 6650
-Wire Wire Line
-	2450 6650 2275 6650
 NoConn ~ 4600 6275
 NoConn ~ 4750 6275
@@
 Wire Wire Line
 	9425 1100 9425 1425
-Text Label 2650 6825 0    50   ~ 0
-vdd_x
 Wire Wire Line
 	4600 2175 4900 2175
@@
 Connection ~ 4900 2175
 Wire Wire Line
-	4900 1800 4900 2175
-Wire Wire Line
 	4900 2175 4900 2375
 NoConn ~ 2850 3875
-$Comp
-L Connector:Conn_Coaxial J7
-U 1 1 6012EC07
-P 4950 1400
-F 0 "J7" H 5050 1400 50  0000 L CNN
-F 1 "Conn_Coaxial" H 5050 1300 50  0000 L CNN
-F 2 "Connector_Coaxial:U.FL_Hirose_U.FL-R-SMT-1_Vertical" H 4950 1400 50  0001 C CNN
-F 3 " ~" H 4950 1400 50  0001 C CNN
-	1    4950 1400
-	1    0    0    -1
-$EndComp
-Wire Wire Line
-	4750 1400 4750 2375
-Wire Wire Line
-	4950 1600 4950 1800
-Wire Wire Line
-	4950 1800 4900 1800
+NoConn ~ 3550 2375
+$Comp
+L Device:Antenna_Shield AE1
+U 1 1 6041BD6E
+P 4750 1530
+F 0 "AE1" H 4905 1595 50  0000 L CNN
+F 1 "Antenna_Shield" H 4905 1495 50  0000 L CNN
+F 2 "RF_Antenna:Texas_SWRA117D_2.4GHz_Left" H 4750 1630 50  0001 C CNN
+F 3 "~" H 4750 1630 50  0001 C CNN
+	1    4750 1530
+	1    0    0    -1
+$EndComp
+Wire Wire Line
+	4850 1730 4900 1730
+Wire Wire Line
+	4900 1730 4900 2175
+Wire Wire Line
+	4750 1730 4750 2375
+NoConn ~ 2850 5375
+NoConn ~ 2850 5525
 $EndSCHEMATC
