File: mcu/digital-amplifier2/circuit/main/Bluetooth.sch (KiCad schematic (older format))
At the start: 5 parts, among them U5 SJR-BTM331

Commit message: main_v4
Parts:
- renumbered C22 to C23, C23 to C24, R22 to R24, U5 to U6
Connections:
- net labels added: state2
- wire segments 37 -> 38
- no-connect marks 38 -> 37
Changed lines of the file:
@@
 $Descr A4 11693 8268
 encoding utf-8
-Sheet 5 10
+Sheet 6 10
 Title ""
 Date ""
@@
 	2100 4925 2850 4925
 $Comp
-L Device:C_Small C22
+L Device:C_Small C23
 U 1 1 5FD6F3D0
 P 1800 5450
-F 0 "C22" H 1892 5496 50  0000 L CNN
+F 0 "C23" H 1892 5496 50  0000 L CNN
 F 1 "22uf" H 1892 5405 50  0000 L CNN
 F 2 "Capacitor_SMD:C_0805_2012Metric" H 1800 5450 50  0001 C CNN
@@
 $EndComp
 $Comp
-L power:GND #PWR040
+L power:GND #PWR037
 U 1 1 5FD6FF1D
 P 1800 5925
-F 0 "#PWR040" H 1800 5675 50  0001 C CNN
+F 0 "#PWR037" H 1800 5675 50  0001 C CNN
 F 1 "GND" H 1805 5752 50  0000 C CNN
 F 2 "" H 1800 5925 50  0001 C CNN
@@
 	4450 6900 5050 6900
 $Comp
-L power:GND #PWR041
+L power:GND #PWR038
 U 1 1 5FD70E74
 P 4000 6725
-F 0 "#PWR041" H 4000 6475 50  0001 C CNN
+F 0 "#PWR038" H 4000 6475 50  0001 C CNN
 F 1 "GND" H 4005 6552 50  0000 C CNN
 F 2 "" H 4000 6725 50  0001 C CNN
@@
 	4000 6725 4000 6275
 $Comp
-L power:GND #PWR044
+L power:GND #PWR041
 U 1 1 5FD71A86
 P 6250 4325
-F 0 "#PWR044" H 6250 4075 50  0001 C CNN
+F 0 "#PWR041" H 6250 4075 50  0001 C CNN
 F 1 "GND" H 6255 4152 50  0000 C CNN
 F 2 "" H 6250 4325 50  0001 C CNN
@@
 	6250 4025 5600 4025
 $Comp
-L power:GND #PWR042
+L power:GND #PWR039
 U 1 1 5FD726D5
 P 5875 2425
-F 0 "#PWR042" H 5875 2175 50  0001 C CNN
+F 0 "#PWR039" H 5875 2175 50  0001 C CNN
 F 1 "GND" H 5880 2252 50  0000 C CNN
 F 2 "" H 5875 2425 50  0001 C CNN
@@
 Text HLabel 6175 5075 2    50   Input ~ 0
 button
-Text HLabel 6175 5525 2    50   Input ~ 0
+Text HLabel 6175 5525 2    50   Output ~ 0
 state
 NoConn ~ 2850 4025
@@
 NoConn ~ 4900 6275
 NoConn ~ 3850 6275
-NoConn ~ 2850 3275
-$Comp
-L power:GND #PWR043
+$Comp
+L power:GND #PWR040
 U 1 1 5FDC12A0
 P 6250 3300
-F 0 "#PWR043" H 6250 3050 50  0001 C CNN
+F 0 "#PWR040" H 6250 3050 50  0001 C CNN
 F 1 "GND" H 6255 3127 50  0000 C CNN
 F 2 "" H 6250 3300 50  0001 C CNN
@@
 	5600 3125 6250 3125
 $Comp
-L misc:SJR-BTM331 U5
+L misc:SJR-BTM331 U6
 U 1 1 5FD6BC07
 P 2950 2475
-F 0 "U5" H 4225 2753 50  0000 C CNN
+F 0 "U6" H 4225 2753 50  0000 C CNN
 F 1 "SJR-BTM331" H 4225 2662 50  0000 C CNN
 F 2 "misc:SJR-BTM331" H 3350 975 50  0001 C CNN
@@
 $EndComp
 $Comp
-L power:+3.3V #PWR045
+L power:+3.3V #PWR042
 U 1 1 5FE85C0D
 P 8875 1075
-F 0 "#PWR045" H 8875 925 50  0001 C CNN
+F 0 "#PWR042" H 8875 925 50  0001 C CNN
 F 1 "+3.3V" H 8890 1248 50  0000 C CNN
 F 2 "" H 8875 1075 50  0001 C CNN
@@
 $EndComp
 $Comp
-L Device:R_Small R22
+L Device:R_Small R24
 U 1 1 5FE85C5E
 P 9150 1425
-F 0 "R22" V 8954 1425 50  0000 C CNN
+F 0 "R24" V 8954 1425 50  0000 C CNN
 F 1 "0Ω" V 9045 1425 50  0000 C CNN
 F 2 "Resistor_SMD:R_0805_2012Metric" H 9150 1425 50  0001 C CNN
@@
 vdd_x
 $Comp
-L Device:C_Small C23
+L Device:C_Small C24
 U 1 1 5FE872FA
 P 9425 1625
-F 0 "C23" H 9517 1671 50  0000 L CNN
+F 0 "C24" H 9517 1671 50  0000 L CNN
 F 1 "10uf" H 9517 1580 50  0000 L CNN
 F 2 "Capacitor_SMD:C_0805_2012Metric" H 9425 1625 50  0001 C CNN
@@
 	9425 1725 9425 1900
 $Comp
-L power:GND #PWR046
+L power:GND #PWR043
 U 1 1 5FE88CAB
 P 9425 1900
-F 0 "#PWR046" H 9425 1650 50  0001 C CNN
+F 0 "#PWR043" H 9425 1650 50  0001 C CNN
 F 1 "GND" H 9430 1727 50  0000 C CNN
 F 2 "" H 9425 1900 50  0001 C CNN
@@
 NoConn ~ 2850 5375
 NoConn ~ 2850 5525
+Text HLabel 2100 3275 0    50   Output ~ 0
+state2
+Wire Wire Line
+	2100 3275 2850 3275
 $EndSCHEMATC

Commit message: v5
Parts:
- added TP6: SPDIF, TestPoint:TestPoint_Pad_1.0x1.0mm, symbol Connector:TestPoint
Connections:
- wire segments 38 -> 39
- no-connect marks 37 -> 36
Changed lines of the file:
@@
 $Descr A4 11693 8268
 encoding utf-8
-Sheet 6 10
+Sheet 6 12
 Title ""
 Date ""
@@
 	4900 2175 4900 2375
 NoConn ~ 2850 3875
-NoConn ~ 3550 2375
 $Comp
 L Device:Antenna_Shield AE1
@@
 Wire Wire Line
 	2100 3275 2850 3275
+Wire Wire Line
+	3550 2375 3550 2000
+$Comp
+L Connector:TestPoint TP6
+U 1 1 609C4FDA
+P 3550 2000
+F 0 "TP6" H 3650 2150 50  0000 L CNN
+F 1 "SPDIF" H 3650 2050 50  0000 L CNN
+F 2 "TestPoint:TestPoint_Pad_1.0x1.0mm" H 3750 2000 50  0001 C CNN
+F 3 "~" H 3750 2000 50  0001 C CNN
+	1    3550 2000
+	1    0    0    -1
+$EndComp
 $EndSCHEMATC
