File: mcu/digital-amplifier2/circuit/main/Bluetooth.sch (KiCad schematic (older format))
At the start: 9 parts, among them U4 LP2992AIM5-3.3_NOPB, U6 SJR-BTM331

Commit message: digital-amplifier2_v8
Parts:
- removed C45: 10uf, Capacitor_SMD:C_0805_2012Metric, symbol Device:C_Small
- removed C46: 10nf, Capacitor_SMD:C_0805_2012Metric, symbol Device:C_Small
- removed R8, R9: 9.53k, Resistor_SMD:R_0805_2012Metric, symbol Device:R_Small
- removed U4: LP2992AIM5-3.3_NOPB, Package_TO_SOT_SMD:TSOT-23-5, symbol ti:LP2992AIM5-3.3_NOPB
- added R30: 9.53k, Resistor_SMD:R_0805_2012Metric, symbol Device:R_Small
- added R31: 0, Resistor_SMD:R_0805_2012Metric, symbol Device:R_Small
- AE1: footprint RF_Antenna:Texas_SWRA117D_2.4GHz_Left -> Connector_Coaxial:SMA_Molex_73251-2200_Horizontal
- renumbered C23 to C55, C47 to C56, U6 to U7
Connections:
- net labels added: +3.3V, FS, SCK, SD
- net labels removed: +5V, music_state
- wire segments 56 -> 48
- no-connect marks 37 -> 35
Other:
- moved on the sheet: C56
