File: mcu/digital-amplifier2/circuit/main/TPA6120A2.sch (KiCad schematic (older format))
At the start: 19 parts, among them J9 AudioJack3_Switch, U11 TPA6120A2DWP

Commit message: headphone
Parts:
- added C37, C45: 100uf, Capacitor_SMD:C_1210_3225Metric, symbol Device:C_Small
- added C38, C39, C46, C47: 10uf, Capacitor_SMD:C_0805_2012Metric, symbol Device:C_Small
- added C41, C44, C50, C53: 100nf, Capacitor_SMD:C_0805_2012Metric, symbol Device:C_Small
- J7: renamed from J9; footprint Connector_Audio:Jack_6.35mm_Neutrik_NMJ6HFD2-AU_Horizontal -> Connector_Audio:Jack_6.35mm_Neutrik_NMJ6HFD2_Horizontal
- renumbered C79 to C58, C80 to C59, R54 to R40, R55 to R41, R56 to R42, R57 to R43, R60 to R44, R58 to R45, R59 to R46, R63 to R47, R64 to R48, R65 to R49, R66 to R50, R67 to R51, R68 to R52, R62 to R53, R61 to R54, U11 to U9
Connections:
- wire segments 93 -> 133
Other:
- moved on the sheet: J7, R44, R45, R46
