File: mcu/digital-amplifier2/circuit/main/TPA6120A2.sch (KiCad schematic (older format))
At the start: 29 parts, among them J6 AudioJack4, U11 TPA6120A2DWP

Commit message: main_v4
Parts:
- removed C51, C52: 1nf, Capacitor_SMD:C_0805_2012Metric, symbol Device:C_Small
- removed R38, R39, R40, R41: 402Ω, Resistor_SMD:R_0805_2012Metric, symbol Device:R_Small
- added J7: AudioJack3_Switch, Connector_Audio:Jack_6.35mm_Neutrik_NMJ6HFD2-AU_Horizontal, symbol Connector:AudioJack3_Switch
- added R55: 9.53k, Resistor_SMD:R_0805_2012Metric, symbol Device:R_Small
- R25: renamed from R42; value 402Ω -> 1k
- R26: renamed from R43; value 402Ω -> 1k
- R27: renamed from R44; value 402Ω -> 1k
- R28: renamed from R45; value 402Ω -> 1k
- R29: renamed from R46; value 806Ω -> 1k
- R30: renamed from R47; value 806Ω -> 1k
- R31: renamed from R48; value 806Ω -> 1k
- R32: renamed from R49; value 806Ω -> 1k
- R33: renamed from R50; value 9.53k -> 1m
- renumbered C49 to C25, C50 to C26, C53 to C27, C54 to C28, C55 to C29, C56 to C30, C57 to C31, C58 to C32, C59 to C33, C60 to C34, R51 to R34, R52 to R35, U11 to U7
Connections:
- net labels added: +3.3V
- wire segments 133 -> 129
- no-connect marks 0 -> 3
Other:
- moved on the sheet: J6, R25, R26, R27, R28, R29, R30, R31, R32, R33, R34, R35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

Commit message: v5
Parts:
- removed U7: TPA6120A2DWP, ti:TPA6120A2DWP, symbol digital-amplifier2-rescue:TPA6120A2DWP-ti-digital-amplifier2-rescue
- added U7: TPA6120A2, ti:TPA6120A2DWP, symbol ti:TPA6120A2
Changed lines of the file:
@@
 $Descr A4 11693 8268
 encoding utf-8
-Sheet 7 10
+Sheet 7 12
 Title ""
 Date ""
@@
 Wire Wire Line
 	4325 2575 4750 2575
-$Comp
-L digital-amplifier2-rescue:TPA6120A2DWP-ti-digital-amplifier2-rescue U?
-U 1 1 600C7C24
-P 4750 2575
-AR Path="/5F115848/600C7C24" Ref="U?"  Part="1"
-AR Path="/5F9D81B7/5FF93314/600C7C24" Ref="U?"  Part="1"
-AR Path="/600C7C24" Ref="U?"  Part="1"
-AR Path="/6035C8F0/5FF93314/600C7C24" Ref="U?"  Part="1"
-AR Path="/6079F77B/600C7C24" Ref="U7"  Part="1"
-F 0 "U7" H 5550 3062 60  0000 C CNN
-F 1 "TPA6120A2DWP" H 5550 2956 60  0000 C CNN
-F 2 "ti:TPA6120A2DWP" H 5550 2915 60  0001 C CNN
-F 3 "" H 4750 2575 60  0000 C CNN
-	1    4750 2575
-	1    0    0    -1
-$EndComp
-$Comp
-L digital-amplifier2-rescue:TPA6120A2DWP-ti-digital-amplifier2-rescue U?
-U 2 1 600CA436
-P 8850 4075
-AR Path="/5F115848/600CA436" Ref="U?"  Part="2"
-AR Path="/5F9D81B7/5FF93314/600CA436" Ref="U?"  Part="2"
-AR Path="/600CA436" Ref="U?"  Part="2"
-AR Path="/6035C8F0/5FF93314/600CA436" Ref="U?"  Part="2"
-AR Path="/6079F77B/600CA436" Ref="U7"  Part="2"
-F 0 "U7" H 10178 3378 60  0000 L CNN
-F 1 "TPA6120A2DWP" H 10178 3272 60  0000 L CNN
-F 2 "ti:TPA6120A2DWP" H 9650 4415 60  0001 C CNN
-F 3 "" H 8850 4075 60  0000 C CNN
-	2    8850 4075
-	1    0    0    -1
-$EndComp
 Wire Wire Line
 	8850 4075 8700 4075
@@
 Wire Wire Line
 	6350 1925 6350 2475
-Connection ~ 6350 2475
 Wire Wire Line
 	3875 1675 2700 1675
@@
 	1    0    0    -1
 $EndComp
+$Comp
+L ti:TPA6120A2 U7
+U 1 1 60C26CC9
+P 4750 2575
+F 0 "U7" H 5575 3100 60  0000 C CNN
+F 1 "TPA6120A2" H 5575 3000 60  0000 C CNN
+F 2 "ti:TPA6120A2DWP" H 5550 2915 60  0001 C CNN
+F 3 "" H 4750 2575 60  0000 C CNN
+	1    4750 2575
+	1    0    0    -1
+$EndComp
+Connection ~ 6350 2475
+$Comp
+L ti:TPA6120A2 U7
+U 2 1 60C2A547
+P 8850 4075
+F 0 "U7" H 10225 3400 60  0000 L CNN
+F 1 "TPA6120A2" H 10225 3300 60  0000 L CNN
+F 2 "ti:TPA6120A2DWP" H 9650 4415 60  0001 C CNN
+F 3 "" H 8850 4075 60  0000 C CNN
+	2    8850 4075
+	1    0    0    -1
+$EndComp
