File: mcu/digital-amplifier2/circuit/main/TPA6120A2.sch (KiCad schematic (older format))
At the start: 21 parts, among them U7 TPA6120A2

Commit message: digital-amplifier2_v8
Parts:
- added C23, C29: 100uf, Capacitor_SMD:C_1210_3225Metric, symbol Device:C_Small
- C27: renamed from C28; footprint Capacitor_SMD:C_0805_2012Metric -> Capacitor_SMD:C_0603_1608Metric
- C28: renamed from C29; footprint Capacitor_SMD:C_0805_2012Metric -> Capacitor_SMD:C_0603_1608Metric
- C33, C34: footprint Capacitor_SMD:C_0805_2012Metric -> Capacitor_SMD:C_0603_1608Metric
- R12: renamed from R25; footprint Resistor_SMD:R_0805_2012Metric -> Resistor_SMD:R_0603_1608Metric
- R13: renamed from R26; footprint Resistor_SMD:R_0805_2012Metric -> Resistor_SMD:R_0603_1608Metric
- R14: renamed from R27; footprint Resistor_SMD:R_0805_2012Metric -> Resistor_SMD:R_0603_1608Metric
- R15: renamed from R28; footprint Resistor_SMD:R_0805_2012Metric -> Resistor_SMD:R_0603_1608Metric
- R16: renamed from R29; footprint Resistor_SMD:R_0805_2012Metric -> Resistor_SMD:R_0603_1608Metric
- R17: renamed from R30; footprint Resistor_SMD:R_0805_2012Metric -> Resistor_SMD:R_0603_1608Metric
- R18: renamed from R31; footprint Resistor_SMD:R_0805_2012Metric -> Resistor_SMD:R_0603_1608Metric
- R19: renamed from R32; footprint Resistor_SMD:R_0805_2012Metric -> Resistor_SMD:R_0603_1608Metric
- renumbered C25 to C24, C26 to C25, C27 to C26, R34 to R20, R35 to R21, U7 to U4
Connections:
- net +12V: now also C23.1
- net -12V: now also C29.1
- net GND: now also C23.2, C29.2

Commit message: amplifier2_v9
Connections:
- net +12V renamed +15V
- net -12V renamed -15V
Changed lines of the file:
@@
 $Descr A4 11693 8268
 encoding utf-8
-Sheet 4 12
+Sheet 4 11
 Title ""
 Date ""
@@
 Wire Wire Line
 	4550 7000 4925 7000
-$Comp
-L power:+12V #PWR?
-U 1 1 608C4FC6
-P 975 6300
-AR Path="/6035C8F0/5FF93314/608C4FC6" Ref="#PWR?"  Part="1"
-AR Path="/6079F77B/608C4FC6" Ref="#PWR026"  Part="1"
-F 0 "#PWR026" H 975 6150 50  0001 C CNN
-F 1 "+12V" H 1025 6525 50  0000 C CNN
-F 2 "" H 975 6300 50  0001 C CNN
-F 3 "" H 975 6300 50  0001 C CNN
-	1    975  6300
-	1    0    0    -1
-$EndComp
-$Comp
-L power:-12V #PWR?
-U 1 1 608C55FE
-P 3725 6250
-AR Path="/6035C8F0/5FF93314/608C55FE" Ref="#PWR?"  Part="1"
-AR Path="/6079F77B/608C55FE" Ref="#PWR029"  Part="1"
-F 0 "#PWR029" H 3725 6350 50  0001 C CNN
-F 1 "-12V" H 3750 6475 50  0000 C CNN
-F 2 "" H 3725 6250 50  0001 C CNN
-F 3 "" H 3725 6250 50  0001 C CNN
-	1    3725 6250
-	1    0    0    -1
-$EndComp
 Wire Wire Line
 	1775 7025 2150 7025
@@
 	1    0    0    -1
 $EndComp
-$Comp
-L power:+12V #PWR?
-U 1 1 6090AD02
-P 8175 4825
-AR Path="/6035C8F0/5FF93314/6090AD02" Ref="#PWR?"  Part="1"
-AR Path="/6079F77B/6090AD02" Ref="#PWR032"  Part="1"
-F 0 "#PWR032" H 8175 4675 50  0001 C CNN
-F 1 "+12V" H 8225 5025 50  0000 C CNN
-F 2 "" H 8175 4825 50  0001 C CNN
-F 3 "" H 8175 4825 50  0001 C CNN
-	1    8175 4825
-	1    0    0    -1
-$EndComp
-$Comp
-L power:-12V #PWR?
-U 1 1 60910D15
-P 8450 5850
-AR Path="/6035C8F0/5FF93314/60910D15" Ref="#PWR?"  Part="1"
-AR Path="/6079F77B/60910D15" Ref="#PWR034"  Part="1"
-F 0 "#PWR034" H 8450 5950 50  0001 C CNN
-F 1 "-12V" H 8425 6075 50  0000 C CNN
-F 2 "" H 8450 5850 50  0001 C CNN
-F 3 "" H 8450 5850 50  0001 C CNN
-	1    8450 5850
-	-1   0    0    1
-$EndComp
 Wire Wire Line
 	2250 2950 2700 2950
@@
 Connection ~ 975  7025
 Connection ~ 975  6500
+$Comp
+L power:+15V #PWR025
+U 1 1 60F5A0E9
+P 8175 4825
+F 0 "#PWR025" H 8175 4675 50  0001 C CNN
+F 1 "+15V" H 8200 5025 50  0000 C CNN
+F 2 "" H 8175 4825 50  0001 C CNN
+F 3 "" H 8175 4825 50  0001 C CNN
+	1    8175 4825
+	1    0    0    -1
+$EndComp
+$Comp
+L power:-15V #PWR032
+U 1 1 60F5AE14
+P 8450 5850
+F 0 "#PWR032" H 8450 5950 50  0001 C CNN
+F 1 "-15V" H 8450 6075 50  0000 C CNN
+F 2 "" H 8450 5850 50  0001 C CNN
+F 3 "" H 8450 5850 50  0001 C CNN
+	1    8450 5850
+	-1   0    0    1
+$EndComp
+$Comp
+L power:-15V #PWR0127
+U 1 1 60F6C622
+P 3725 6250
+F 0 "#PWR0127" H 3725 6350 50  0001 C CNN
+F 1 "-15V" H 3725 6475 50  0000 C CNN
+F 2 "" H 3725 6250 50  0001 C CNN
+F 3 "" H 3725 6250 50  0001 C CNN
+	1    3725 6250
+	1    0    0    -1
+$EndComp
+$Comp
+L power:+15V #PWR0141
+U 1 1 60F7279D
+P 975 6300
+F 0 "#PWR0141" H 975 6150 50  0001 C CNN
+F 1 "+15V" H 1000 6500 50  0000 C CNN
+F 2 "" H 975 6300 50  0001 C CNN
+F 3 "" H 975 6300 50  0001 C CNN
+	1    975  6300
+	1    0    0    -1
+$EndComp
 $EndSCHEMATC

Commit message: digital-amplifier2_v10
Parts:
- C23, C24, C29, C30: value 100uf -> 47uf
