File: mcu/digital-amplifier2/circuit/main/digital-amplifier2.sch (KiCad schematic (older format))
At the start: 5 parts, among them J6 Conn_02x10_Odd_Even

Commit message: headphone
Parts:
- removed H1: m2_1, MountingHole:MountingHole_2.2mm_M2_ISO7380_Pad, symbol Mechanical:MountingHole
- removed H2: m2_2, MountingHole:MountingHole_2.2mm_M2_ISO7380_Pad, symbol Mechanical:MountingHole
- removed H3: m2_3, MountingHole:MountingHole_2.2mm_M2_ISO7380_Pad, symbol Mechanical:MountingHole
- removed H4: m2_4, MountingHole:MountingHole_2.2mm_M2_ISO7380_Pad, symbol Mechanical:MountingHole
- removed J6: Conn_02x10_Odd_Even, Connector_PinHeader_2.54mm:PinHeader_2x10_P2.54mm_Vertical, symbol Connector_Generic:Conn_02x10_Odd_Even
- added H1, H2, H3, H4: m3, MountingHole:MountingHole_3.2mm_M3_Pad, symbol Mechanical:MountingHole_Pad
- added J6: Conn_01x06, Connector_PinHeader_2.54mm:PinHeader_1x06_P2.54mm_Vertical, symbol Connector_Generic:Conn_01x06
Connections:
- net labels removed: BT_spdif, GND, SAI1_A_SD, SAI1_B_MCK, VCC, headphone_irq, headphone_mute, tas6424_fault, tas6424_mute, tas6424_warn
- wire segments 68 -> 33
- no-connect marks 0 -> 4
