File: mcu/digital-amplifier2/circuit/main/digital-amplifier2.sch (KiCad schematic (older format))
At the start: 6 parts

Commit message: digital-amplifier2-v3
Changed lines of the file:
@@
 F8 "JackIN" O L 5490 1135 50
 $EndSheet
-Text Label 4865 1795 0    50   ~ 0
+Text Label 4880 1890 0    50   ~ 0
 SCL
-Text Label 4865 1890 0    50   ~ 0
+Text Label 4875 1795 0    50   ~ 0
 SDA
 Wire Wire Line

Commit message: main_v4
Parts:
- removed H5, H6: m3, MountingHole:MountingHole_3.2mm_M3_Pad, symbol Mechanical:MountingHole_Pad
Connections:
- net labels added: BT_state2, I2S1_MCK, SAI1_A_FS, SAI1_A_SCK, SAI1_A_SD
- net labels removed: GND, SAI1_B_CLK, SAI1_B_FS, SAI1_B_SD, tas6424_en
- wire segments 35 -> 38

Commit message: v5
Connections:
- net labels added: dac_power_en
- net labels removed: headphone_en
Changed lines of the file:
@@
 $Descr A4 11693 8268
 encoding utf-8
-Sheet 1 10
+Sheet 1 12
 Title ""
 Date ""
@@
 $EndSheet
 $Sheet
-S 2540 6415 1300 975
+S 4350 6525 1300 975
 U 6074FC63
 F0 "headphone_power" 50
@@
 F6 "LRCK" I L 7675 1350 50
 F7 "DATA" I L 7675 1450 50
-F8 "RST" I L 7675 1625 50
-F9 "OUTLP" O R 8525 1175 50
-F10 "OUTLN" O R 8525 1300 50
-F11 "OUTRP" O R 8525 925 50
-F12 "OUTRN" O R 8525 1050 50
+F8 "OUTLP" O R 8525 1175 50
+F9 "OUTLN" O R 8525 1300 50
+F10 "OUTRP" O R 8525 925 50
+F11 "OUTRN" O R 8525 1050 50
 $EndSheet
 $Sheet
@@
 SAI1_A_FS
 Wire Wire Line
-	6910 1625 7675 1625
-Wire Wire Line
 	8710 3375 9475 3375
 Wire Wire Line
@@
 SAI1_A_SCK
 Text Label 2200 1725 0    50   ~ 0
-headphone_en
-Text Label 7050 1625 0    50   ~ 0
-headphone_en
+dac_power_en
 Text Label 10425 1650 0    50   ~ 0
 headphone_in
@@
 Text Label 2195 2755 0    50   ~ 0
 BT_state2
+$Sheet
+S 7600 5050 1000 950
+U 60973CA0
+F0 "power7v" 50
+F1 "power7v.sch" 50
+F2 "EN" I L 7600 5325 50
+$EndSheet
+$Sheet
+S 2725 6500 1125 950
+U 6099BEE5
+F0 "power±15v" 50
+F1 "power±15v.sch" 50
+$EndSheet
+Wire Wire Line
+	6835 5325 7600 5325
+Text Label 6950 5325 0    50   ~ 0
+dac_power_en
 $EndSCHEMATC
