File: mcu/digital-amplifier2/circuit/main/digital-amplifier2.sch (KiCad schematic (older format))
At the start: 0 parts

Commit message: digital-amplifier2_v8
Connections:
- net labels added: 5805_en, USB_EN, oled_en, out_a+, out_a-, out_b+, out_b-
- net labels removed: BT_music, USB_CO, ext_en, ext_irq
- wire segments 77 -> 88

Commit message: amplifier2_v9
Changed lines of the file:
@@
 $Descr A4 11693 8268
 encoding utf-8
-Sheet 1 12
+Sheet 1 11
 Title ""
 Date ""
@@
 F2 "SCL" I L 7675 875 50
 F3 "SDA" I L 7675 975 50
-F4 "SCK" I L 7675 1150 50
-F5 "BCK" I L 7675 1250 50
+F4 "MCK" I L 7675 1150 50
+F5 "SCK" I L 7675 1250 50
 F6 "LRCK" I L 7675 1350 50
 F7 "DATA" I L 7675 1450 50
@@
 Wire Wire Line
 	7125 875  7675 875
-$Sheet
-S 9600 2275 800  725
-U 60C533A9
-F0 "hp_ldo" 50
-F1 "hp_ldo.sch" 50
-$EndSheet
 Wire Wire Line
 	7675 1575 7125 1575
 Text Label 7275 1575 0    50   ~ 0
 hp_en
+Text Label 7275 1150 0    50   ~ 0
+SAI_MCK
 Text Label 7275 1450 0    50   ~ 0
-SAI_MCK
-Text Label 7275 1150 0    50   ~ 0
 SAI_SD
+Text Label 7275 1350 0    50   ~ 0
+SAI_FS
 Text Label 7275 1250 0    50   ~ 0
-SAI_FS
-Text Label 7275 1350 0    50   ~ 0
 SAI_SCK
 Wire Wire Line

Commit message: digital-amplifier2_v10
Connections:
- net labels added: adr1, adr2
- wire segments 88 -> 92
Changed lines of the file:
@@
 F30 "HP_EN" O R 3325 1225 50
 F31 "OLED_EN" O R 3325 2600 50
+F32 "ADR1" I R 3325 2800 50
+F33 "ADR2" I R 3325 2900 50
 $EndSheet
 $Sheet
@@
 F10 "OUT_B-" O R 6500 4425 50
 F11 "SD" I L 5375 4525 50
+F12 "ADR1" I R 6500 4525 50
+F13 "ADR2" I R 6500 4625 50
 $EndSheet
 Wire Wire Line
@@
 Text Label 3525 2600 0    50   ~ 0
 oled_en
+Wire Wire Line
+	6500 4525 6950 4525
+Wire Wire Line
+	6500 4625 6950 4625
+Text Label 6625 4525 0    50   ~ 0
+adr1
+Text Label 6625 4625 0    50   ~ 0
+adr2
+Wire Wire Line
+	3325 2800 4100 2800
+Wire Wire Line
+	3325 2900 4100 2900
+Text Label 3525 2800 0    50   ~ 0
+adr1
+Text Label 3525 2900 0    50   ~ 0
+adr2
 $EndSCHEMATC
