File: mcu/digital-amplifier2/circuit/main/jtag_and_power.sch (KiCad schematic (older format))
At the start: 19 parts, among them J1 i2c, J2 USB_B, J3 encoder, J4 swd, Q1 s8550, U2 DLT11H0

Commit message: main_v4
Parts:
- removed J1: i2c, Connector_PinHeader_2.54mm:PinHeader_1x04_P2.54mm_Vertical, symbol Connector_Generic:Conn_01x04
- removed J4: swd, Connector_PinHeader_2.54mm:PinHeader_1x04_P2.54mm_Vertical, symbol Connector_Generic:Conn_01x04
- removed R5, R7: 4.7k, Resistor_SMD:R_0805_2012Metric, symbol Device:R_Small
- added D1, D2: 40v 5A, Diode_SMD:D_SMA, symbol Device:D
- added H5, H6, H7, H8: m3, MountingHole:MountingHole_3.2mm_M3_Pad, symbol Mechanical:MountingHole_Pad
- added J3: Barrel_Jack_Switch, connector:DC-044A_5.5-2.1, symbol Connector:Barrel_Jack_Switch
- renumbered J3 to J4, R6 to R7
Connections:
- net GND: now also H6.1, H8.1, J3.2
- new net: D1.2 (A), D2.2 (A), J3.1
- new net VCC: D1.1 (K), D2.1 (K), H5.1, H7.1
- no-connect marks 2 -> 3
Other:
- moved on the sheet: C12, C13, C14, J4, R12, R13, R14, U2

Commit message: v5
Parts:
- removed D1, D2: 40v 5A, Diode_SMD:D_SMA, symbol Device:D
- added D4: 2a, Diode_SMD:D_SMA, symbol Device:D_Schottky_Small
Connections:
- net VCC: now also J3.1
- net at J2.1 (VBUS): now also D4.2 (A)
- new net +5V: D4.1 (K)
- no-connect marks 3 -> 2
Other:
- moved on the sheet: J2, Q1, R10, R11, R7
Changed lines of the file:
@@
 $Descr A4 11693 8268
 encoding utf-8
-Sheet 3 10
+Sheet 3 12
 Title ""
 Date ""
@@
 Comment4 ""
 $EndDescr
-Text HLabel 2865 2330 2    50   Input ~ 0
+Text HLabel 2850 2325 2    50   Input ~ 0
 USBD+
-Text HLabel 2865 2530 2    50   Input ~ 0
+Text HLabel 2850 2525 2    50   Input ~ 0
 USBD-
 $Comp
 L Device:R_Small R9
 U 1 1 607B112A
-P 2440 2530
-F 0 "R9" V 2365 2530 50  0000 C CNN
-F 1 "12Ω" V 2515 2530 50  0000 C CNN
-F 2 "Resistor_SMD:R_0805_2012Metric" H 2440 2530 50  0001 C CNN
-F 3 "~" H 2440 2530 50  0001 C CNN
-	1    2440 2530
+P 2425 2525
+F 0 "R9" V 2350 2525 50  0000 C CNN
+F 1 "12Ω" V 2500 2525 50  0000 C CNN
+F 2 "Resistor_SMD:R_0805_2012Metric" H 2425 2525 50  0001 C CNN
+F 3 "~" H 2425 2525 50  0001 C CNN
+	1    2425 2525
 	0    1    1    0
 $EndComp
@@
 L Device:R_Small R8
 U 1 1 607B112B
-P 2440 2330
-F 0 "R8" V 2244 2330 50  0000 C CNN
-F 1 "12Ω" V 2335 2330 50  0000 C CNN
-F 2 "Resistor_SMD:R_0805_2012Metric" H 2440 2330 50  0001 C CNN
-F 3 "~" H 2440 2330 50  0001 C CNN
-	1    2440 2330
+P 2425 2325
+F 0 "R8" V 2229 2325 50  0000 C CNN
+F 1 "12Ω" V 2320 2325 50  0000 C CNN
+F 2 "Resistor_SMD:R_0805_2012Metric" H 2425 2325 50  0001 C CNN
+F 3 "~" H 2425 2325 50  0001 C CNN
+	1    2425 2325
 	0    1    1    0
 $EndComp
-Wire Wire Line
-	2540 2530 2865 2530
-Wire Wire Line
-	2540 2330 2865 2330
 $Comp
 L Device:R_Small R7
 U 1 1 5FE10838
-P 2040 1840
-F 0 "R7" H 2099 1886 50  0000 L CNN
-F 1 "1.5k" H 2099 1795 50  0000 L CNN
-F 2 "Resistor_SMD:R_0805_2012Metric" H 2040 1840 50  0001 C CNN
-F 3 "~" H 2040 1840 50  0001 C CNN
-	1    2040 1840
+P 2025 1900
+F 0 "R7" H 2084 1946 50  0000 L CNN
+F 1 "1.5k" H 2084 1855 50  0000 L CNN
+F 2 "Resistor_SMD:R_0805_2012Metric" H 2025 1900 50  0001 C CNN
+F 3 "~" H 2025 1900 50  0001 C CNN
+	1    2025 1900
 	1    0    0    -1
 $EndComp
@@
 L power:+3.3V #PWR016
 U 1 1 5FE16E8B
-P 2040 890
-F 0 "#PWR016" H 2040 740 50  0001 C CNN
-F 1 "+3.3V" H 2055 1063 50  0000 C CNN
-F 2 "" H 2040 890 50  0001 C CNN
-F 3 "" H 2040 890 50  0001 C CNN
-	1    2040 890
-	1    0    0    -1
-$EndComp
-Wire Wire Line
-	2040 1740 2040 1640
+P 2025 1000
+F 0 "#PWR016" H 2025 850 50  0001 C CNN
+F 1 "+3.3V" H 2040 1173 50  0000 C CNN
+F 2 "" H 2025 1000 50  0001 C CNN
+F 3 "" H 2025 1000 50  0001 C CNN
+	1    2025 1000
+	1    0    0    -1
+$EndComp
 $Comp
 L Device:R_Small R11
 U 1 1 607B112E
-P 2550 1440
-F 0 "R11" V 2450 1280 50  0000 C CNN
-F 1 "5.1k" V 2450 1540 50  0000 C CNN
-F 2 "Resistor_SMD:R_0805_2012Metric" H 2550 1440 50  0001 C CNN
-F 3 "~" H 2550 1440 50  0001 C CNN
-	1    2550 1440
+P 2575 1475
+F 0 "R11" V 2475 1315 50  0000 C CNN
+F 1 "5.1k" V 2475 1575 50  0000 C CNN
+F 2 "Resistor_SMD:R_0805_2012Metric" H 2575 1475 50  0001 C CNN
+F 3 "~" H 2575 1475 50  0001 C CNN
+	1    2575 1475
 	0    1    1    0
 $EndComp
-Wire Wire Line
-	2340 1440 2450 1440
 $Comp
 L Device:R_Small R10
 U 1 1 607B112F
-P 2550 1180
-F 0 "R10" V 2640 1240 50  0000 L CNN
-F 1 "22k" V 2630 1060 50  0000 L CNN
-F 2 "Resistor_SMD:R_0805_2012Metric" H 2550 1180 50  0001 C CNN
-F 3 "~" H 2550 1180 50  0001 C CNN
-	1    2550 1180
+P 2575 1225
+F 0 "R10" V 2665 1285 50  0000 L CNN
+F 1 "22k" V 2655 1105 50  0000 L CNN
+F 2 "Resistor_SMD:R_0805_2012Metric" H 2575 1225 50  0001 C CNN
+F 3 "~" H 2575 1225 50  0001 C CNN
+	1    2575 1225
 	0    -1   -1   0
 $EndComp
-Text HLabel 3465 1440 2    50   Input ~ 0
+Text HLabel 3100 1475 2    50   Input ~ 0
 USB_CONNECT
 $Comp
 L Device:Q_PNP_BEC Q1
 U 1 1 601B7316
-P 2140 1440
-F 0 "Q1" H 2340 1390 50  0000 L CNN
-F 1 "s8550" H 2340 1440 50  0000 L CNN
-F 2 "Package_TO_SOT_SMD:SOT-23" H 2340 1540 50  0001 C CNN
-F 3 "~" H 2140 1440 50  0001 C CNN
-	1    2140 1440
+P 2125 1475
+F 0 "Q1" H 2325 1425 50  0000 L CNN
+F 1 "s8550" H 2325 1475 50  0000 L CNN
+F 2 "Package_TO_SOT_SMD:SOT-23" H 2325 1575 50  0001 C CNN
+F 3 "~" H 2125 1475 50  0001 C CNN
+	1    2125 1475
 	-1   0    0    1
 $EndComp
-Wire Wire Line
-	1365 2430 1540 2430
-Wire Wire Line
-	1540 2430 1540 2530
-NoConn ~ 965  2730
-NoConn ~ 1365 2130
-Wire Wire Line
-	1540 2530 2340 2530
+NoConn ~ 900  2725
 $Comp
 L power:+3.3V #PWR?
@@
 Wire Wire Line
 	8960 4595 8960 4435
-Wire Wire Line
-	2040 890  2040 1180
-Wire Wire Line
-	2450 1180 2040 1180
-Connection ~ 2040 1180
-Wire Wire Line
-	2040 1180 2040 1240
-Wire Wire Line
-	2650 1180 2820 1180
-Wire Wire Line
-	2820 1180 2820 1440
-Connection ~ 2820 1440
-Wire Wire Line
-	2650 1440 2820 1440
-Wire Wire Line
-	2820 1440 3465 1440
-Wire Wire Line
-	2040 1940 2040 2330
-Wire Wire Line
-	1365 2330 2040 2330
-Connection ~ 2040 2330
-Wire Wire Line
-	2040 2330 2340 2330
 $Comp
 L power:VCC #PWR?
@@
 	1    0    0    -1
 $EndComp
-$Comp
-L Device:D D?
-U 1 1 6072E8B2
-P 5025 6250
-AR Path="/5F16021E/6072E8B2" Ref="D?"  Part="1"
-AR Path="/5F047EA6/5FD62F96/6072E8B2" Ref="D1"  Part="1"
-F 0 "D1" H 5025 6034 50  0000 C CNN
-F 1 "40v 5A" H 5025 6125 50  0000 C CNN
-F 2 "Diode_SMD:D_SMA" H 5025 6250 50  0001 C CNN
-F 3 "~" H 5025 6250 50  0001 C CNN
-	1    5025 6250
-	-1   0    0    1
-$EndComp
-Wire Wire Line
-	4675 6250 4850 6250
 Wire Wire Line
 	5675 6250 5675 5875
 Wire Wire Line
 	5675 5575 5675 5875
-Wire Wire Line
-	5175 6250 5300 6250
-$Comp
-L Device:D D?
-U 1 1 6072E8BC
-P 5025 6600
-AR Path="/5F16021E/6072E8BC" Ref="D?"  Part="1"
-AR Path="/5F047EA6/5FD62F96/6072E8BC" Ref="D2"  Part="1"
-F 0 "D2" H 5025 6384 50  0000 C CNN
-F 1 "40v 5A" H 5025 6475 50  0000 C CNN
-F 2 "Diode_SMD:D_SMA" H 5025 6600 50  0001 C CNN
-F 3 "~" H 5025 6600 50  0001 C CNN
-	1    5025 6600
-	-1   0    0    1
-$EndComp
-Connection ~ 5300 6250
 $Comp
 L Connector:Barrel_Jack_Switch J?
@@
 Wire Wire Line
 	4675 6450 4675 6850
-Wire Wire Line
-	4850 6250 4850 6600
-Wire Wire Line
-	4850 6600 4875 6600
-Connection ~ 4850 6250
-Wire Wire Line
-	4850 6250 4875 6250
-Wire Wire Line
-	5175 6600 5300 6600
-Wire Wire Line
-	5300 6250 5300 6600
 $Comp
 L Connector:USB_B J2
 U 1 1 6058E78E
-P 1065 2330
-F 0 "J2" H 1122 2797 50  0000 C CNN
-F 1 "USB_B" H 1122 2706 50  0000 C CNN
-F 2 "Connector_USB:USB_B_OST_USB-B1HSxx_Horizontal" H 1215 2280 50  0001 C CNN
-F 3 " ~" H 1215 2280 50  0001 C CNN
-	1    1065 2330
+P 1000 2325
+F 0 "J2" H 1057 2792 50  0000 C CNN
+F 1 "USB_B" H 1057 2701 50  0000 C CNN
+F 2 "Connector_USB:USB_B_OST_USB-B1HSxx_Horizontal" H 1150 2275 50  0001 C CNN
+F 3 " ~" H 1150 2275 50  0001 C CNN
+	1    1000 2325
 	1    0    0    -1
 $EndComp
@@
 L power:GND #PWR013
 U 1 1 60C54D24
-P 1065 2905
-F 0 "#PWR013" H 1065 2655 50  0001 C CNN
-F 1 "GND" H 1090 2680 50  0000 C CNN
-F 2 "" H 1065 2905 50  0001 C CNN
-F 3 "" H 1065 2905 50  0001 C CNN
-	1    1065 2905
-	1    0    0    -1
-$EndComp
-Wire Wire Line
-	1065 2905 1065 2730
+P 1000 2850
+F 0 "#PWR013" H 1000 2600 50  0001 C CNN
+F 1 "GND" H 1025 2625 50  0000 C CNN
+F 2 "" H 1000 2850 50  0001 C CNN
+F 3 "" H 1000 2850 50  0001 C CNN
+	1    1000 2850
+	1    0    0    -1
+$EndComp
 $Comp
 L power:GND #PWR?
@@
 Wire Wire Line
 	6150 6100 6150 6250
-Wire Wire Line
-	5300 6250 5675 6250
 Connection ~ 5675 6250
 Wire Wire Line
@@
 	6600 6850 6150 6850
 Connection ~ 6150 6850
+$Comp
+L Device:D_Schottky_Small D4
+U 1 1 60DBB743
+P 1525 1925
+F 0 "D4" V 1450 2000 50  0000 L CNN
+F 1 "2a" V 1550 2000 50  0000 L CNN
+F 2 "Diode_SMD:D_SMA" V 1525 1925 50  0001 C CNN
+F 3 "~" V 1525 1925 50  0001 C CNN
+	1    1525 1925
+	0    1    1    0
+$EndComp
+$Comp
+L power:+5V #PWR0101
+U 1 1 60DBDF20
+P 1525 1600
+F 0 "#PWR0101" H 1525 1450 50  0001 C CNN
+F 1 "+5V" H 1550 1800 50  0000 C CNN
+F 2 "" H 1525 1600 50  0001 C CNN
+F 3 "" H 1525 1600 50  0001 C CNN
+	1    1525 1600
+	1    0    0    -1
+$EndComp
+Wire Wire Line
+	2475 1225 2025 1225
+Wire Wire Line
+	2025 1225 2025 1275
+Wire Wire Line
+	2025 1000 2025 1225
+Connection ~ 2025 1225
+Wire Wire Line
+	2475 1475 2325 1475
+Wire Wire Line
+	2675 1225 2875 1225
+Wire Wire Line
+	2875 1225 2875 1475
+Wire Wire Line
+	2875 1475 2675 1475
+Wire Wire Line
+	2875 1475 3100 1475
+Connection ~ 2875 1475
+Wire Wire Line
+	2025 1675 2025 1800
+Wire Wire Line
+	2025 2000 2025 2325
+Wire Wire Line
+	2025 2325 2325 2325
+Wire Wire Line
+	2025 2325 1300 2325
+Connection ~ 2025 2325
+Wire Wire Line
+	1300 2425 2025 2425
+Wire Wire Line
+	2025 2425 2025 2525
+Wire Wire Line
+	2025 2525 2325 2525
+Wire Wire Line
+	2525 2325 2850 2325
+Wire Wire Line
+	2850 2525 2525 2525
+Wire Wire Line
+	1525 2025 1525 2125
+Wire Wire Line
+	1525 2125 1300 2125
+Wire Wire Line
+	1525 1825 1525 1600
+Wire Wire Line
+	1000 2850 1000 2725
+Wire Wire Line
+	4675 6250 5675 6250
 $EndSCHEMATC
