File: mcu/digital-amplifier2/circuit/main/power.sch (KiCad schematic (older format))
At the start: 21 parts, among them J5 Barrel_Jack_Switch, U3 TPS54360DDA, U4 AMS1117-3.3

Commit message: main_v4
Parts:
- removed C20: 47uf, Capacitor_SMD:C_0805_2012Metric, symbol Device:C_Small
- removed D2, D3: 40v 5A, Diode_SMD:D_SMA, symbol Device:D
- removed J5: Barrel_Jack_Switch, connector:DC-044A_5.5-2.1, symbol Connector:Barrel_Jack_Switch
- removed R15: 523k, Resistor_SMD:R_0805_2012Metric, symbol Device:R_Small
- removed R16: 84.5k, Resistor_SMD:R_0805_2012Metric, symbol Device:R_Small
- added C22: 10uf, Capacitor_SMD:C_0805_2012Metric, symbol Device:C_Small
- added C72, C73: 100nf, Capacitor_SMD:C_0805_2012Metric, symbol Device:C_Small
- added R23: 0Ω, Resistor_SMD:R_0805_2012Metric, symbol Device:R_Small
- added U5: AMS1117-5.0, Package_TO_SOT_SMD:SOT-223-3_TabPin2, symbol Regulator_Linear:AMS1117-5.0
- renumbered C15 to C16, C16 to C17, C17 to C18, C18 to C19, C19 to C20, D1 to D3, R17 to R18, R18 to R19, R19 to R20, R20 to R21, R21 to R22
Connections:
- net labels added: +5V, +7.5V
- net labels removed: VDD
- wire segments 85 -> 79
Other:
- moved on the sheet: C21, R22, U4

Commit message: ciruit_save
Parts:
- R20: value 53.6k -> 75k
- R21: value 10.2k -> 9.53k
Changed lines of the file:
@@
 P 5625 2075
 F 0 "R20" H 5684 2121 50  0000 L CNN
-F 1 "53.6k" H 5684 2030 50  0000 L CNN
+F 1 "75k" H 5684 2030 50  0000 L CNN
 F 2 "Resistor_SMD:R_0805_2012Metric" H 5625 2075 50  0001 C CNN
 F 3 "~" H 5625 2075 50  0001 C CNN
@@
 P 5625 2475
 F 0 "R21" H 5684 2521 50  0000 L CNN
-F 1 "10.2k" H 5684 2430 50  0000 L CNN
+F 1 "9.53k" H 5684 2430 50  0000 L CNN
 F 2 "Resistor_SMD:R_0805_2012Metric" H 5625 2475 50  0001 C CNN
 F 3 "~" H 5625 2475 50  0001 C CNN

Commit message: pcb
Parts:
- C17: value 6.8nf -> 5.1nF
- C18: value 39pf -> 750pF
- R18: value 162k -> 49.9kOhm
- R19: value 13k -> 15.4k
Changed lines of the file:
@@
 P 2875 2300
 F 0 "R18" H 2934 2346 50  0000 L CNN
-F 1 "162k" H 2934 2255 50  0000 L CNN
+F 1 "49.9kOhm" H 2934 2255 50  0000 L CNN
 F 2 "Resistor_SMD:R_0805_2012Metric" H 2875 2300 50  0001 C CNN
 F 3 "~" H 2875 2300 50  0001 C CNN
@@
 P 3600 2800
 F 0 "R19" H 3659 2846 50  0000 L CNN
-F 1 "13k" H 3659 2755 50  0000 L CNN
+F 1 "15.4k" H 3659 2755 50  0000 L CNN
 F 2 "Resistor_SMD:R_0805_2012Metric" H 3600 2800 50  0001 C CNN
 F 3 "~" H 3600 2800 50  0001 C CNN
@@
 P 3925 2800
 F 0 "C18" H 4017 2846 50  0000 L CNN
-F 1 "39pf" H 4017 2755 50  0000 L CNN
+F 1 "750pF" H 4017 2755 50  0000 L CNN
 F 2 "Capacitor_SMD:C_0805_2012Metric" H 3925 2800 50  0001 C CNN
 F 3 "~" H 3925 2800 50  0001 C CNN
@@
 P 3600 3075
 F 0 "C17" H 3692 3121 50  0000 L CNN
-F 1 "6.8nf" H 3692 3030 50  0000 L CNN
+F 1 "5.1nF" H 3692 3030 50  0000 L CNN
 F 2 "Capacitor_SMD:C_0805_2012Metric" H 3600 3075 50  0001 C CNN
 F 3 "~" H 3600 3075 50  0001 C CNN

Commit message: v5
Parts:
- removed C73: 100nf, Capacitor_SMD:C_0805_2012Metric, symbol Device:C_Small
- removed R23: 0Ω, Resistor_SMD:R_0805_2012Metric, symbol Device:R_Small
- removed U5: AMS1117-5.0, Package_TO_SOT_SMD:SOT-223-3_TabPin2, symbol Regulator_Linear:AMS1117-5.0
- added C15: 1uf, Capacitor_SMD:C_0805_2012Metric, symbol Device:C_Small
- added C37: 10uf, Capacitor_SMD:C_0805_2012Metric, symbol Device:C_Small
- added C38, C41: 22uf, Capacitor_SMD:C_0805_2012Metric, symbol Device:C_Small
- added C46: 10nf, Capacitor_SMD:C_0805_2012Metric, symbol Device:C_Small
- added D1: 40v 3A, Diode_SMD:D_SMA, symbol Device:D
- added L2: 3.3uh, Inductor_SMD:L_1210_3225Metric, symbol Device:L_Small
- added R42: 0Ω, Resistor_SMD:R_0805_2012Metric, symbol Device:R_Small
- added U5: LP2992, Package_TO_SOT_SMD:TSOT-23-5, symbol ti:LP2992
- C22: value 10uf -> 1uf
- C72: value 100nf -> 10uf
Connections:
- net +5V: now also C15.1, C41.1, L2.1, U5.1 (IN), U5.3 (EN); no longer C22.1
- net GND: now also C15.2, C37.2, C38.2, C41.2, C46.2, U5.2 (GND)
- net VCC: now also D1.2 (A); no longer C16.1, U3.2 (VIN)
- net +7.5V: no longer names the net of C20.1, L1.2, R20.1
- net +7.5V: now also C38.1, L2.2
- new net: C16.1, D1.1 (K), U3.2 (VIN)
- new net: C22.1, R42.2, U5.5 (OUT)
- new net: C46.1, U5.4 (BYPASS)
- new net +3.3VA: C37.1, R42.1
Other:
- moved on the sheet: C16, C17, C18, C19, C20, C21, C72, D3, L1, R18, R19, R20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

Commit message: save
Parts:
- C17: value 5.1nF -> 2.7nf
- C18: value 750pF -> 10pf
- L1: value 8.2uh -> 15uh
- R18: value 49.9kOhm -> 10nf
- R19: value 15.4k -> 10.7k
- R20: value 75k -> 10.2k
- R21: value 9.53k -> 1.96k
Changed lines of the file:
@@
 P 2000 2025
 F 0 "R18" H 2059 2071 50  0000 L CNN
-F 1 "49.9kOhm" H 2059 1980 50  0000 L CNN
+F 1 "10nf" H 2059 1980 50  0000 L CNN
 F 2 "Resistor_SMD:R_0805_2012Metric" H 2000 2025 50  0001 C CNN
 F 3 "~" H 2000 2025 50  0001 C CNN
@@
 P 3700 1500
 F 0 "L1" V 3905 1500 50  0000 C CNN
-F 1 "8.2uh" V 3814 1500 50  0000 C CNN
+F 1 "15uh" V 3814 1500 50  0000 C CNN
 F 2 "Inductor_SMD:L_6.3x6.3_H3" H 3700 1500 50  0001 C CNN
 F 3 "~" H 3700 1500 50  0001 C CNN
@@
 P 2725 2525
 F 0 "R19" H 2784 2571 50  0000 L CNN
-F 1 "15.4k" H 2784 2480 50  0000 L CNN
+F 1 "10.7k" H 2784 2480 50  0000 L CNN
 F 2 "Resistor_SMD:R_0805_2012Metric" H 2725 2525 50  0001 C CNN
 F 3 "~" H 2725 2525 50  0001 C CNN
@@
 P 3050 2525
 F 0 "C18" H 3142 2571 50  0000 L CNN
-F 1 "750pF" H 3142 2480 50  0000 L CNN
+F 1 "10pf" H 3142 2480 50  0000 L CNN
 F 2 "Capacitor_SMD:C_0805_2012Metric" H 3050 2525 50  0001 C CNN
 F 3 "~" H 3050 2525 50  0001 C CNN
@@
 P 2725 2800
 F 0 "C17" H 2817 2846 50  0000 L CNN
-F 1 "5.1nF" H 2817 2755 50  0000 L CNN
+F 1 "2.7nf" H 2817 2755 50  0000 L CNN
 F 2 "Capacitor_SMD:C_0805_2012Metric" H 2725 2800 50  0001 C CNN
 F 3 "~" H 2725 2800 50  0001 C CNN
@@
 P 4750 1800
 F 0 "R20" H 4809 1846 50  0000 L CNN
-F 1 "75k" H 4809 1755 50  0000 L CNN
+F 1 "10.2k" H 4809 1755 50  0000 L CNN
 F 2 "Resistor_SMD:R_0805_2012Metric" H 4750 1800 50  0001 C CNN
 F 3 "~" H 4750 1800 50  0001 C CNN
@@
 P 4750 2200
 F 0 "R21" H 4809 2246 50  0000 L CNN
-F 1 "9.53k" H 4809 2155 50  0000 L CNN
+F 1 "1.96k" H 4809 2155 50  0000 L CNN
 F 2 "Resistor_SMD:R_0805_2012Metric" H 4750 2200 50  0001 C CNN
 F 3 "~" H 4750 2200 50  0001 C CNN
