File: mcu/digital-amplifier2/circuit/main/power.sch (KiCad schematic (older format))
At the start: 31 parts, among them T1 Transformer_diy_01, U2 LP2992AIM5-3.3_NOPB, U3 TPS55340

Commit message: digital-amplifier2_v8
Parts:
- removed C15: 47nf, Capacitor_SMD:C_0805_2012Metric, symbol Device:C_Small
- removed C17: NC, Capacitor_SMD:C_0805_2012Metric, symbol Device:C_Small
- removed C19, C20, C37, C38, C41: 22uf, Capacitor_SMD:C_0805_2012Metric, symbol Device:C_Small
- removed C24: 10nf, Capacitor_SMD:C_0805_2012Metric, symbol Device:C_Small
- removed C43: 100nf, Capacitor_SMD:C_0805_2012Metric, symbol Device:C_Small
- removed D1, D2, D5, D6, D7: ss34, Diode_SMD:D_SMA, symbol Device:D_Small
- removed R15: 80k, Resistor_SMD:R_0805_2012Metric, symbol Device:R_Small
- removed R16: 2.37k, Resistor_SMD:R_0805_2012Metric, symbol Device:R_Small
- removed R17: 2k, Resistor_SMD:R_0805_2012Metric, symbol Device:R_Small
- removed R18: 6.1367k, Resistor_SMD:R_0805_2012Metric, symbol Device:R_Small
- removed T1: Transformer_diy_01, misc:Transformer_diy_01, symbol misc:Transformer_diy_01
- removed U2: LP2992AIM5-3.3_NOPB, Package_TO_SOT_SMD:TSOT-23-5, symbol ti:LP2992AIM5-3.3_NOPB
- removed U3: TPS55340, Package_SO:HTSSOP-14-1EP_4.4x5mm_P0.65mm_EP3.4x5mm_Mask3x3.1mm_ThermalVias, symbol ti:TPS55340
- added C14: 100nf, Capacitor_SMD:C_0603_1608Metric, symbol Device:C_Small
- added C22: 22uf, Capacitor_SMD:C_0805_2012Metric, symbol Device:C_Small
- added C60: 1uf, Capacitor_SMD:C_0805_2012Metric, symbol Device:C_Small
- added C99: NC, Capacitor_SMD:C_0603_1608Metric, symbol Device:C_Small
- added L1, L2: 22uh / 0630, Inductor_SMD:L_6.3x6.3_H3, symbol Device:L_Small
- added L3: 2.2uh / 0805, Inductor_SMD:L_0805_2012Metric, symbol Device:L_Small
- added R10: 1k, Resistor_SMD:R_0603_1608Metric, symbol Device:R_Small
- added R11: 5k, Resistor_SMD:R_0603_1608Metric, symbol Device:R_Small
- added R46: 0Ω, Resistor_SMD:R_0603_1608Metric, symbol Device:R_Small
- added R7: 43k, Resistor_SMD:R_0603_1608Metric, symbol Device:R_Small
- added R8: 2.37k, Resistor_SMD:R_0603_1608Metric, symbol Device:R_Small
- added U2: TPS55340, Package_SO:HTSSOP-14-1EP_4.4x5mm_P0.65mm_EP3.4x5mm_Mask3x3.1mm_ThermalVias, symbol ti:TPS55340
- added U3: AMS1117-3.3, Package_TO_SOT_SMD:SOT-223-3_TabPin2, symbol Regulator_Linear:AMS1117-3.3
- added U9: AMS1117-5.0, Package_TO_SOT_SMD:SOT-223-3_TabPin2, symbol Regulator_Linear:AMS1117-5.0
- C13: value NC -> 47nf; footprint Capacitor_SMD:C_0805_2012Metric -> Capacitor_SMD:C_0603_1608Metric
- C16: value 100nf -> 2.2uf; footprint Capacitor_SMD:C_0805_2012Metric -> Capacitor_SMD:C_1206_3216Metric
- C17: renamed from C44; value 10uf -> 1uf
- C20: renamed from C42; value 22uf -> 100nf
- renumbered C14 to C15, C22 to C19
Connections:
- net labels added: FB1
- net labels removed: +15V, -15V, FB, SW, VBUS, t1a, t1b, t2a, t2b, t2c, t3a, t3b, vcc1
- wire segments 130 -> 92
Other:
- moved on the sheet: C15, C17, C18, C19, C20, D3
