File: mcu/digital-amplifier2/circuit/main/PCM1792.sch (KiCad schematic (older format))
At the start: 16 parts, among them U12 PCM1792A

Commit message: digital-amplifier2_v8
Parts:
- added R22: 0Ω, Resistor_SMD:R_0603_1608Metric, symbol Device:R_Small
- C35: renamed from C50; footprint Capacitor_SMD:C_0805_2012Metric -> Capacitor_SMD:C_0603_1608Metric
- C36: renamed from C51; footprint Capacitor_SMD:C_0805_2012Metric -> Capacitor_SMD:C_0603_1608Metric
- C37: renamed from C60; footprint Capacitor_SMD:C_0805_2012Metric -> Capacitor_SMD:C_0603_1608Metric
- C38: renamed from C61; footprint Capacitor_SMD:C_0805_2012Metric -> Capacitor_SMD:C_0603_1608Metric
- C39: renamed from C52; footprint Capacitor_SMD:C_0805_2012Metric -> Capacitor_SMD:C_0603_1608Metric
- C40: renamed from C53; footprint Capacitor_SMD:C_0805_2012Metric -> Capacitor_SMD:C_0603_1608Metric
- C41: renamed from C54; footprint Capacitor_SMD:C_0805_2012Metric -> Capacitor_SMD:C_0603_1608Metric
- C42: renamed from C55; footprint Capacitor_SMD:C_0805_2012Metric -> Capacitor_SMD:C_0603_1608Metric
- C43: renamed from C56; footprint Capacitor_SMD:C_0805_2012Metric -> Capacitor_SMD:C_0603_1608Metric
- C44: renamed from C57; footprint Capacitor_SMD:C_0805_2012Metric -> Capacitor_SMD:C_0603_1608Metric
- C45: renamed from C58; footprint Capacitor_SMD:C_0805_2012Metric -> Capacitor_SMD:C_0603_1608Metric
- C46: renamed from C59; footprint Capacitor_SMD:C_0805_2012Metric -> Capacitor_SMD:C_0603_1608Metric
- R23: renamed from R7; footprint Resistor_SMD:R_0805_2012Metric -> Resistor_SMD:R_0603_1608Metric
- R24: renamed from R50; footprint Resistor_SMD:R_0805_2012Metric -> Resistor_SMD:R_0603_1608Metric
- R25: renamed from R43; footprint Resistor_SMD:R_0805_2012Metric -> Resistor_SMD:R_0603_1608Metric
- renumbered U12 to U5
Connections:
- net labels added: +3.3V, +5V, EN
- net labels removed: +5VA
- wire segments 97 -> 102
Other:
- moved on the sheet: C35, C36, R23

Commit message: amplifier2_v9
Connections:
- net labels added: MCK
- net labels removed: BCK
Changed lines of the file:
@@
 $Descr A4 11693 8268
 encoding utf-8
-Sheet 5 12
+Sheet 5 11
 Title ""
 Date ""
@@
 	2675 4775 1975 4775
 Text HLabel 1975 4475 0    50   Input ~ 0
+MCK
+Text HLabel 1975 4575 0    50   Input ~ 0
 SCK
-Text HLabel 1975 4575 0    50   Input ~ 0
-BCK
 Text HLabel 1975 4675 0    50   Input ~ 0
 LRCK
