File: mcu/digital-amplifier2/circuit/main/headphone_power.sch (KiCad schematic (older format))
At the start: 41 parts, among them U10 LM317_SOT-223, U11 LM337_SOT223, U8 TPS54360DDA, U9 TPS54360DDA

Commit message: ciruit_save
Parts:
- R40, R42: value 215k -> 180k
- R41, R43: value 12.1k -> 9.53k
- R47: value 10k -> 7.5
- R57: value 10k -> 7.5k
Changed lines of the file:
@@
 AR Path="/6074FC63/5FC96B2B" Ref="R42"  Part="1"
 F 0 "R42" H 4774 6431 50  0000 L CNN
-F 1 "215k" H 4774 6340 50  0000 L CNN
+F 1 "180k" H 4774 6340 50  0000 L CNN
 F 2 "Resistor_SMD:R_0805_2012Metric" H 4715 6385 50  0001 C CNN
 F 3 "~" H 4715 6385 50  0001 C CNN
@@
 AR Path="/6074FC63/5FC96BA3" Ref="R43"  Part="1"
 F 0 "R43" H 4774 6781 50  0000 L CNN
-F 1 "12.1k" H 4774 6690 50  0000 L CNN
+F 1 "9.53k" H 4774 6690 50  0000 L CNN
 F 2 "Resistor_SMD:R_0805_2012Metric" H 4715 6735 50  0001 C CNN
 F 3 "~" H 4715 6735 50  0001 C CNN
@@
 AR Path="/6074FC63/606A5313" Ref="R40"  Part="1"
 F 0 "R40" H 4284 1796 50  0000 L CNN
-F 1 "215k" H 4284 1705 50  0000 L CNN
+F 1 "180k" H 4284 1705 50  0000 L CNN
 F 2 "Resistor_SMD:R_0805_2012Metric" H 4225 1750 50  0001 C CNN
 F 3 "~" H 4225 1750 50  0001 C CNN
@@
 AR Path="/6074FC63/606A5319" Ref="R41"  Part="1"
 F 0 "R41" H 4284 2146 50  0000 L CNN
-F 1 "12.1k" H 4284 2055 50  0000 L CNN
+F 1 "9.53k" H 4284 2055 50  0000 L CNN
 F 2 "Resistor_SMD:R_0805_2012Metric" H 4225 2100 50  0001 C CNN
 F 3 "~" H 4225 2100 50  0001 C CNN
@@
 P 8750 2600
 F 0 "R47" H 8650 2550 50  0000 R CNN
-F 1 "10k" H 8650 2600 50  0000 R CNN
+F 1 "7.5" H 8650 2635 50  0000 R CNN
 F 2 "Resistor_SMD:R_0805_2012Metric" H 8750 2600 50  0001 C CNN
 F 3 "~" H 8750 2600 50  0001 C CNN
@@
 $EndComp
 $Comp
-L Device:R_Small R56
-U 1 1 6078B5B2
-P 8750 2900
-F 0 "R56" H 8850 2950 50  0000 L CNN
-F 1 "1k" H 8850 2900 50  0000 L CNN
-F 2 "Resistor_SMD:R_0805_2012Metric" H 8750 2900 50  0001 C CNN
-F 3 "~" H 8750 2900 50  0001 C CNN
-	1    8750 2900
-	1    0    0    -1
-$EndComp
-$Comp
 L Device:R_Small R57
 U 1 1 6078ABD8
 P 8750 3200
 F 0 "R57" H 8850 3250 50  0000 L CNN
-F 1 "10k" H 8850 3200 50  0000 L CNN
+F 1 "7.5k" H 8850 3200 50  0000 L CNN
 F 2 "Resistor_SMD:R_0805_2012Metric" H 8750 3200 50  0001 C CNN
 F 3 "~" H 8750 3200 50  0001 C CNN
@@
 	-1   0    0    1
 $EndComp
+$Comp
+L Device:R_Small R56
+U 1 1 6078B5B2
+P 8750 2900
+F 0 "R56" H 8850 2950 50  0000 L CNN
+F 1 "1k" H 8845 2880 50  0000 L CNN
+F 2 "Resistor_SMD:R_0805_2012Metric" H 8750 2900 50  0001 C CNN
+F 3 "~" H 8750 2900 50  0001 C CNN
+	1    8750 2900
+	1    0    0    -1
+$EndComp
 $EndSCHEMATC

Commit message: pcb
Parts:
- C38: value 220pF -> 750pF
- C40: value 4.3nF -> 5.1nF
- R36: value 97.6kOhm -> 49.9kOhm
- R38: value 18.7kOhm -> 15.4kOhm
- R40, R42: value 180k -> 160k
- R56: value 1k -> 7.5k
- R57: value 7.5k -> 1k
Changed lines of the file:
@@
 AR Path="/6074FC63/5FC96B2B" Ref="R42"  Part="1"
 F 0 "R42" H 4774 6431 50  0000 L CNN
-F 1 "180k" H 4774 6340 50  0000 L CNN
+F 1 "160k" H 4774 6340 50  0000 L CNN
 F 2 "Resistor_SMD:R_0805_2012Metric" H 4715 6385 50  0001 C CNN
 F 3 "~" H 4715 6385 50  0001 C CNN
@@
 AR Path="/6074FC63/6068367B" Ref="R38"  Part="1"
 F 0 "R38" H 2509 2246 50  0000 L CNN
-F 1 "18.7kOhm" H 2509 2155 50  0000 L CNN
+F 1 "15.4kOhm" H 2509 2155 50  0000 L CNN
 F 2 "Resistor_SMD:R_0805_2012Metric" H 2450 2200 50  0001 C CNN
 F 3 "~" H 2450 2200 50  0001 C CNN
@@
 AR Path="/6074FC63/60683681" Ref="C40"  Part="1"
 F 0 "C40" H 2542 2571 50  0000 L CNN
-F 1 "4.3nF" H 2542 2480 50  0000 L CNN
+F 1 "5.1nF" H 2542 2480 50  0000 L CNN
 F 2 "Capacitor_SMD:C_0805_2012Metric" H 2450 2525 50  0001 C CNN
 F 3 "~" H 2450 2525 50  0001 C CNN
@@
 AR Path="/6074FC63/60683687" Ref="C38"  Part="1"
 F 0 "C38" H 2192 2371 50  0000 L CNN
-F 1 "220pF" H 2192 2280 50  0000 L CNN
+F 1 "750pF" H 2192 2280 50  0000 L CNN
 F 2 "Capacitor_SMD:C_0805_2012Metric" H 2100 2325 50  0001 C CNN
 F 3 "~" H 2100 2325 50  0001 C CNN
@@
 AR Path="/6074FC63/606A5313" Ref="R40"  Part="1"
 F 0 "R40" H 4284 1796 50  0000 L CNN
-F 1 "180k" H 4284 1705 50  0000 L CNN
+F 1 "160k" H 4284 1705 50  0000 L CNN
 F 2 "Resistor_SMD:R_0805_2012Metric" H 4225 1750 50  0001 C CNN
 F 3 "~" H 4225 1750 50  0001 C CNN
@@
 	1    0    0    -1
 $EndComp
-$Comp
-L Device:R_Small R?
-U 1 1 606D6645
-P 1250 2075
-AR Path="/5F115848/5FEDDDE8/606D6645" Ref="R?"  Part="1"
-AR Path="/5FBB5CE4/606D6645" Ref="R?"  Part="1"
-AR Path="/5F9D81B7/5FF87CA8/606D6645" Ref="R?"  Part="1"
-AR Path="/6035C8F0/5FF87CA8/606D6645" Ref="R?"  Part="1"
-AR Path="/6074FC63/606D6645" Ref="R36"  Part="1"
-F 0 "R36" H 1309 2121 50  0000 L CNN
-F 1 "97.6kOhm" H 1309 2030 50  0000 L CNN
-F 2 "Resistor_SMD:R_0805_2012Metric" H 1250 2075 50  0001 C CNN
-F 3 "~" H 1250 2075 50  0001 C CNN
-	1    1250 2075
-	1    0    0    -1
-$EndComp
 Wire Wire Line
 	1250 1975 1250 1450
@@
 P 8750 3200
 F 0 "R57" H 8850 3250 50  0000 L CNN
-F 1 "7.5k" H 8850 3200 50  0000 L CNN
+F 1 "1k" H 8850 3200 50  0000 L CNN
 F 2 "Resistor_SMD:R_0805_2012Metric" H 8750 3200 50  0001 C CNN
 F 3 "~" H 8750 3200 50  0001 C CNN
@@
 P 8750 2900
 F 0 "R56" H 8850 2950 50  0000 L CNN
-F 1 "1k" H 8845 2880 50  0000 L CNN
+F 1 "7.5k" H 8845 2880 50  0000 L CNN
 F 2 "Resistor_SMD:R_0805_2012Metric" H 8750 2900 50  0001 C CNN
 F 3 "~" H 8750 2900 50  0001 C CNN
@@
 	1    0    0    -1
 $EndComp
+$Comp
+L Device:R_Small R?
+U 1 1 606D6645
+P 1250 2075
+AR Path="/5F115848/5FEDDDE8/606D6645" Ref="R?"  Part="1"
+AR Path="/5FBB5CE4/606D6645" Ref="R?"  Part="1"
+AR Path="/5F9D81B7/5FF87CA8/606D6645" Ref="R?"  Part="1"
+AR Path="/6035C8F0/5FF87CA8/606D6645" Ref="R?"  Part="1"
+AR Path="/6074FC63/606D6645" Ref="R36"  Part="1"
+F 0 "R36" H 1309 2121 50  0000 L CNN
+F 1 "49.9kOhm" H 1309 2030 50  0000 L CNN
+F 2 "Resistor_SMD:R_0805_2012Metric" H 1250 2075 50  0001 C CNN
+F 3 "~" H 1250 2075 50  0001 C CNN
+	1    1250 2075
+	1    0    0    -1
+$EndComp

Commit message: v5
Parts:
- removed C37: 2.2uf, Capacitor_SMD:C_0805_2012Metric, symbol Device:C_Small
- removed C38: 750pF, Capacitor_SMD:C_0805_2012Metric, symbol Device:C_Small
- removed C41: 220pF, Capacitor_SMD:C_0805_2012Metric, symbol Device:C_Small
- removed C42, C48, C49: 100nf, Capacitor_SMD:C_0805_2012Metric, symbol Device:C_Small
- removed C43: 4.3nF, Capacitor_SMD:C_0805_2012Metric, symbol Device:C_Small
- removed C44, C45: 22uf, Capacitor_SMD:C_0805_2012Metric, symbol Device:C_Small
- removed C46, C47, C70, C71: 10uf, Capacitor_SMD:C_0805_2012Metric, symbol Device:C_Small
- removed D4: 60v/3A, Diode_SMD:D_SMA, symbol Device:D_Small
- removed D5: 60v 3A, Diode_SMD:D_SMA, symbol Device:D
- removed L2, L3: 22uh, Inductor_SMD:L_6.3x6.3_H3, symbol Device:L_Small
- removed R37: 97.6kOhm, Resistor_SMD:R_0805_2012Metric, symbol Device:R_Small
- removed R38: 15.4kOhm, Resistor_SMD:R_0805_2012Metric, symbol Device:R_Small
- removed R41, R43: 9.53k, Resistor_SMD:R_0805_2012Metric, symbol Device:R_Small
- removed R42: 160k, Resistor_SMD:R_0805_2012Metric, symbol Device:R_Small
- removed R44, R45, R58, R59: 0Ω, Resistor_SMD:R_0805_2012Metric, symbol Device:R_Small
- removed R46, R57: 1k, Resistor_SMD:R_0805_2012Metric, symbol Device:R_Small
- removed R47: 7.5, Resistor_SMD:R_0805_2012Metric, symbol Device:R_Small
- removed R56: 7.5k, Resistor_SMD:R_0805_2012Metric, symbol Device:R_Small
- removed U10: LM317_SOT-223, Package_TO_SOT_SMD:SOT-223-3_TabPin2, symbol Regulator_Linear:LM317_SOT-223
- removed U11: LM337_SOT223, Package_TO_SOT_SMD:SOT-223-3_TabPin2, symbol Regulator_Linear:LM337_SOT223
- removed U8, U9: TPS54360DDA, Package_SO:TI_SO-PowerPAD-8_ThermalVias, symbol Regulator_Switching:TPS54360DDA
- added R23: 0Ω, Resistor_SMD:R_0805_2012Metric, symbol Device:R_Small
- added TP1, TP2: TestPoint, TestPoint:TestPoint_Pad_1.0x1.0mm, symbol Connector:TestPoint
- added U8: LT3045xMSE-1, Package_SO:MSOP-12-1EP_3x4mm_P0.65mm_EP1.65x2.85mm, symbol misc:LT3045xMSE-1
- added U9: LT3094xMSE, Package_SO:MSOP-12-1EP_3x4mm_P0.65mm_EP1.65x2.85mm, symbol Regulator_Linear:LT3094xMSE
- C35, C36: value 2.2uf -> 4.7uf
- C39: value 100nf -> 10uf
- C40: value 5.1nF -> 10uf
- R36: value 49.9kOhm -> 0Ω
- R39: value 18.7kOhm -> 150k
- R40: value 160k -> 150k
Connections:
- net labels removed: FB1, FB2, VCC
- wire segments 152 -> 67
