File: mcu/digital-amplifier2/circuit/main/digital-amplifier2.kicad_pcb (KiCad board)
At the start: 2 copper layers, 94.5 x 100 mm, 166 parts, among them J1 I2C_oled, J10 Audio outA, J11 Audio outB, J12 Audio outC, J13 Audio outD, J2 encoder, J3 USB_C_Receptacle, J4 Conn_ARM_JTAG_SWD_20, J5 Barrel_Jack_Switch, J6 Conn_02x10_Odd_Even, J7 Conn_Coaxial, Q1 S8550, Q2 S8050, Q3 S8550, Q4 Q_NMOS_GDS, U1 DLT11H0, U12 TAS6424QDKQRQ1, U13 SJR-BTM331, U2 STM32F446RETx, U3 TPS54360DDA, U4 AMS1117-3.3, U5 LT3045xMSE-1, Y1 5032 8m

Commit message: headphone
Parts:
- removed C100, C101, C102, C103, C104, C105, C106, C99: 1uf, Capacitor_SMD:C_0603_1608Metric
- removed C108, C109, C110, C111, C112, C113, C114, C115, C87, C88: 1uf, Capacitor_SMD:C_0805_2012Metric
- removed C117, C118, C119, C120, C121, C122, C123, C124: 1nf, Capacitor_SMD:C_0805_2012Metric
- removed C9: 1nF/1KV, Capacitor_SMD:C_0805_2012Metric
- removed D10, D9: LED, LED_SMD:LED_0805_2012Metric
- removed FB1, FB2, FB3: 300 ohm @100MHz 3.1A, Inductor_SMD:L_1210_3225Metric
- removed J1: I2C_oled, Connector_PinHeader_2.54mm:PinHeader_1x04_P2.54mm_Vertical
- removed J10: Audio outA, Connector_JST:JST_NV_B02P-NV_1x02_P5.00mm_Vertical
- removed J11: Audio outB, Connector_JST:JST_NV_B02P-NV_1x02_P5.00mm_Vertical
- removed J12: Audio outC, Connector_JST:JST_NV_B02P-NV_1x02_P5.00mm_Vertical
- removed J13: Audio outD, Connector_JST:JST_NV_B02P-NV_1x02_P5.00mm_Vertical
- removed L10, L11, L4, L5, L6, L7, L8, L9: 3.3uh, Inductor_SMD:L_6.3x6.3_H3
- removed Q2: S8050, Package_TO_SOT_SMD:SOT-23
- removed Q3: S8550, Package_TO_SOT_SMD:SOT-23
- removed Q4: Q_NMOS_GDS, Package_TO_SOT_SMD:TO-252-2
- removed R6: 1m, Resistor_SMD:R_0805_2012Metric
- removed R70, R71: 1k, Resistor_SMD:R_0805_2012Metric
- removed U12: TAS6424QDKQRQ1, ti:TAS6424QDKQRQ1
- added AE1: Antenna_Shield, RF_Antenna:Texas_SWRA117D_2.4GHz_Left, B.Cu at (135.8, 143.9)
- added C33: 100nf, Capacitor_SMD:C_0805_2012Metric, B.Cu at (98.9, 109.9)
- added C51: 22uf, Capacitor_SMD:C_0805_2012Metric, F.Cu at (78.4, 97.8)
- added C52: 22uf, Capacitor_SMD:C_0805_2012Metric, F.Cu at (73.7, 97.8)
- added C53: 100nf, Capacitor_SMD:C_0805_2012Metric, F.Cu at (78.5, 122.6)
- added C54: 4.7uf, Capacitor_SMD:C_0805_2012Metric, F.Cu at (92.6, 98.9)
- added C55: 4.7uf, Capacitor_SMD:C_0805_2012Metric, F.Cu at (58.9, 99.6)
- added C56: 10uf, Capacitor_SMD:C_0805_2012Metric, F.Cu at (93.9, 101.3)
- added C57: 10uf, Capacitor_SMD:C_0805_2012Metric, F.Cu at (62.9, 99.6)
- added C58: 100pf, Capacitor_SMD:C_0805_2012Metric, F.Cu at (87.8, 112.4)
- added C59: 100pf, Capacitor_SMD:C_0805_2012Metric, F.Cu at (87.8, 116.7)
- added J8: Conn_01x02, Connector_JST:JST_VH_S2P-VH_1x02_P3.96mm_Horizontal, F.Cu at (75.3, 62.9)
- added L1: 150uh, misc:MSD1278, F.Cu at (79.4, 84.1)
- added R40: 402Ω, Resistor_SMD:R_0805_2012Metric, F.Cu at (90.6, 111.4)
- added R41: 402Ω, Resistor_SMD:R_0805_2012Metric, F.Cu at (90.6, 113.5)
- added R42: 402Ω, Resistor_SMD:R_0805_2012Metric, F.Cu at (90.6, 115.7)
- added R43: 402Ω, Resistor_SMD:R_0805_2012Metric, F.Cu at (90.6, 117.9)
- added R44: 10k, Resistor_SMD:R_0805_2012Metric, B.Cu at (64.5, 144.5)
- added R45: 39.2Ω, Resistor_SMD:R_0805_2012Metric, F.Cu at (86.4, 126.0)
- added R46: 39.2Ω, Resistor_SMD:R_0805_2012Metric, F.Cu at (84.1, 126.0)
- added R47: 402Ω, Resistor_SMD:R_0805_2012Metric, F.Cu at (84.8, 111.4)
- added R48: 402Ω, Resistor_SMD:R_0805_2012Metric, F.Cu at (84.8, 113.5)
- added R49: 402Ω, Resistor_SMD:R_0805_2012Metric, F.Cu at (84.8, 115.7)
- added R50: 402Ω, Resistor_SMD:R_0805_2012Metric, F.Cu at (84.8, 117.9)
- added R51: 806Ω, Resistor_SMD:R_0805_2012Metric, F.Cu at (84.1, 108.5)
- added R52: 806Ω, Resistor_SMD:R_0805_2012Metric, F.Cu at (84.1, 120.8)
- added R53: 806Ω, Resistor_SMD:R_0805_2012Metric, F.Cu at (86.4, 108.5)
- added R54: 806Ω, Resistor_SMD:R_0805_2012Metric, F.Cu at (86.4, 120.8)
- added U6: TPS54360DDA, Package_SO:TI_SO-PowerPAD-8_ThermalVias, F.Cu at (76.6, 72.4)
- added U7: LT3045xMSE-1, Package_SO:MSOP-12-1EP_3x4mm_P0.65mm_EP1.65x2.85mm, F.Cu at (93.9, 92.5)
- added U8: LT3094xMSE, Package_SO:MSOP-12-1EP_3x4mm_P0.65mm_EP1.65x2.85mm, F.Cu at (60.3, 93.1)
- added U9: TPA6120A2DWP, ti:TPA6120A2DWP, F.Cu at (73.3, 114.6)
- C1, C13, C14, C17, C34, C41, C50, D1, D3, D4: moved to F.Cu
- C19, C31: value 10uf -> 100nf
- C2: value 10pf -> 10uf
- C22: value 100nf -> 0.1uf
- C25: value 100uf -> 1uf; footprint Capacitor_SMD:C_1210_3225Metric -> Capacitor_SMD:C_0805_2012Metric
- C27: value 10uf -> 2.2uf/25v; moved to F.Cu
- C30: value 4.7uf -> 10uf
- C32: value 100uf -> 2.2uF/25V; footprint Capacitor_SMD:C_1210_3225Metric -> Capacitor_SMD:C_0805_2012Metric
- C36: value 10uf -> 1uf
- C37: value 100nf -> 100uf; footprint Capacitor_SMD:C_0805_2012Metric -> Capacitor_SMD:C_1210_3225Metric; moved to F.Cu
- C38: value 100nf -> 10uf; moved to B.Cu
- C40: value 100nf -> 750pf
- C42: value 100uf -> 0.1uf; footprint Capacitor_SMD:C_1210_3225Metric -> Capacitor_SMD:C_0805_2012Metric
- C43: value 100uf -> 5.1nf; footprint Capacitor_SMD:C_1210_3225Metric -> Capacitor_SMD:C_0805_2012Metric
- C44: value 100uf -> 100nf; footprint Capacitor_SMD:C_1210_3225Metric -> Capacitor_SMD:C_0805_2012Metric
- C45: value 100nf -> 100uf; footprint Capacitor_SMD:C_0805_2012Metric -> Capacitor_SMD:C_1210_3225Metric
- C46: value 1uf -> 10uf; moved to B.Cu
- C47: value 2.2uf -> 10uf; moved to B.Cu
- C48: value 2.2uf -> 22uf
- C49: value 1uf -> 22uf
- D2: value 10v -> 60v 3A; moved to F.Cu
- H1: value m2_1 -> m3; footprint MountingHole:MountingHole_2.2mm_M2_ISO7380_Pad -> MountingHole:MountingHole_3.2mm_M3_Pad
- H2: value m2_2 -> m3; footprint MountingHole:MountingHole_2.2mm_M2_ISO7380_Pad -> MountingHole:MountingHole_3.2mm_M3_Pad
- H3: value m2_3 -> m3; footprint MountingHole:MountingHole_2.2mm_M2_ISO7380_Pad -> MountingHole:MountingHole_3.2mm_M3_Pad
- H4: value m2_4 -> m3; footprint MountingHole:MountingHole_2.2mm_M2_ISO7380_Pad -> MountingHole:MountingHole_3.2mm_M3_Pad
- J3: footprint connector:usb_c_24p_smd -> Connector_USB:USB_C_Receptacle_Amphenol_12401548E4-2A
- J5: footprint Connector_BarrelJack:BarrelJack_Horizontal -> connector:DC-044A_5.5-2.1
- J6: value Conn_02x10_Odd_Even -> Conn_01x06; footprint Connector_PinHeader_2.54mm:PinHeader_2x10_P2.54mm_Vertical -> Connector_PinHeader_2.54mm:PinHeader_1x06_P2.54mm_Vertical
- J7: value Conn_Coaxial -> AudioJack3_Switch; footprint Connector_Coaxial:U.FL_Hirose_U.FL-R-SMT-1_Vertical -> Connector_Audio:Jack_6.35mm_Neutrik_NMJ6HFD2_Horizontal
- Q1: value S8550 -> s8550
- R1: moved to B.Cu
- R2: value 49.9Ω -> 9.53k; moved to B.Cu
- R26: value test point -> 9.53k; moved to B.Cu
- R27: value 33.2k -> 9.53k; moved to B.Cu
- R29: value 200k -> 0Ω
- R31: value 0Ω -> 49.9k
- R32: value 10k -> 15.4k
- R33: value 10k -> 215k
- R34: value 10k -> 12.1k
- R35: value 10k -> 200k
- R36: value 10kΩ -> 200k
- R37, R38: value 10k -> 150k; moved to F.Cu
- U5: value LT3045xMSE-1 -> PCM5242; footprint Package_SO:MSOP-12-1EP_3x4mm_P0.65mm_EP1.65x2.85mm -> ti:PCM5242RHBR
- moved J5 79.0 mm to (57.3, 53.1), turned to 0 degrees
- moved R2 77.0 mm to (111.6, 142.6)
- moved D3 71.2 mm to (57.4, 68.2), turned to 90 degrees
- moved D4 67.3 mm to (61.2, 68.2), turned to 90 degrees
- moved R36 67.1 mm to (59.1, 88.8), turned to 0 degrees
- moved C20 66.2 mm to (70.6, 60.6), turned to 270 degrees
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Connections:
- C18 pad 1: Net-(C18-Pad1) -> VCC
- C19 pad 1: VDD -> /Sheet6035C8EF/CPVDD
- C2 pad 1: /stm32/SPDIF_RX -> /Sheet6035C8EF/CPVDD
- C25 pad 1: /TAS6424/vcc_x -> GND
- C25 pad 2: /TAS6424/gnd_x -> Net-(C25-Pad2)
- C27 pad 1: /TAS6424/vcc_x -> Net-(C27-Pad1)
- C27 pad 2: /TAS6424/gnd_x -> Net-(C27-Pad2)
- C30 pad 1: Net-(C30-Pad1) -> /Sheet6035C8EF/AVDD
- C31 pad 1: +3.3VA -> /Sheet6035C8EF/AVDD
- C32 pad 1: /TAS6424/vcc_x -> Net-(C32-Pad1)
- C32 pad 2: /TAS6424/gnd_x -> GND
- C34 pad 1: /TAS6424/vcc_x -> /Sheet6035C8EF/DVDD
- C34 pad 2: /TAS6424/gnd_x -> GND
- C35 pad 1: /TAS6424/vcc_x -> VCC
- C35 pad 2: /TAS6424/gnd_x -> GND
- C36 pad 1: /TAS6424/tas6424_power/vdd_33 -> VCC
- C36 pad 2: /TAS6424/gnd_x -> Net-(C36-Pad2)
- C37 pad 1: /TAS6424/vcc_x -> +15V
- C37 pad 2: /TAS6424/gnd_x -> GND
- C38 pad 1: /TAS6424/vcc_x -> +15V
- C38 pad 2: /TAS6424/gnd_x -> GND
- C39 pad 1: /TAS6424/vcc_x -> +15V
- C39 pad 2: /TAS6424/gnd_x -> GND
- C40 pad 1: /TAS6424/tas6424_power/vdd_33 -> Net-(C40-Pad1)
- C40 pad 2: /TAS6424/gnd_x -> Net-(C36-Pad2)
- C41 pad 1: /TAS6424/vcc_x -> +15V
- C41 pad 2: /TAS6424/gnd_x -> GND
- C42 pad 1: /TAS6424/vcc_x -> Net-(C42-Pad1)
- C42 pad 2: /TAS6424/gnd_x -> Net-(C42-Pad2)
- C43 pad 1: /TAS6424/vcc_x -> Net-(C43-Pad1)
- C43 pad 2: /TAS6424/gnd_x -> Net-(C36-Pad2)
- C44 pad 1: /TAS6424/vcc_x -> +15V
- C44 pad 2: /TAS6424/gnd_x -> GND
- C45 pad 1: /TAS6424/vcc_x -> -15V
- C45 pad 2: /TAS6424/gnd_x -> GND
- C46 pad 1: Net-(C46-Pad1) -> -15V
- C46 pad 2: Net-(C46-Pad2) -> GND
- C47 pad 1: Net-(C47-Pad1) -> -15V
- C47 pad 2: /TAS6424/gnd_x -> GND
- C48 pad 2: /TAS6424/gnd_x -> GND
- C49 pad 1: /TAS6424/vcc_x -> GND
- C49 pad 2: /TAS6424/gnd_x -> Net-(C36-Pad2)
- C50 pad 1: /TAS6424/vcc_x -> -15V
- C50 pad 2: /TAS6424/gnd_x -> GND
- D1 pad 1: VCC -> Net-(C48-Pad1)
- D2 pad 1: Net-(D2-Pad1) -> Net-(C42-Pad1)
- D2 pad 2: GND -> Net-(C36-Pad2)
- H1 pad 1: (no net) -> Net-(H1-Pad1)
- H2 pad 1: (no net) -> Net-(H2-Pad1)
- H3 pad 1: (no net) -> Net-(H3-Pad1)
- H4 pad 1: (no net) -> Net-(H4-Pad1)
- J2 pad 1: /stm32/encoder_b -> GND
- J2 pad 2: /stm32/encoder_a -> /stm32/encoder_b
- J2 pad 3: /stm32/encoder_sw -> /stm32/encoder_a
- J2 pad 4: +3V3 -> /stm32/encoder_sw
- J3 pad A4: Net-(D1-Pad2) -> Net-(J3-PadA4)
- J3 pad A9: Net-(D1-Pad2) -> Net-(J3-PadA4)
- J3 pad B4: Net-(D1-Pad2) -> Net-(J3-PadA4)
- J3 pad B9: Net-(D1-Pad2) -> Net-(J3-PadA4)
- J6 pad 2: GND -> /SDA
- J6 pad 3: /SDA -> /SAI1_B_CLK
- J6 pad 4: GND -> /SAI1_B_FS
- J6 pad 5: /SAI1_B_MCK -> /SAI1_B_SD
- J6 pad 6: GND -> /tas6424_en
- Q1 pad 1: +3V3 -> Net-(Q1-Pad1)
- Q1 pad 2: Net-(Q1-Pad2) -> +3V3
- R10 pad 2: Net-(Q1-Pad2) -> Net-(Q1-Pad1)
- R12 pad 2: +3.3VA -> +3V3
- R18 pad 1: Net-(C18-Pad1) -> VCC
- R2 pad 1: /stm32/SPDIF_RX -> +3V3
- R2 pad 2: Net-(R2-Pad2) -> /stm32/encoder_sw
- R22 pad 2: Net-(C22-Pad1) -> Net-(R22-Pad2)
- R26 pad 1: Net-(R26-Pad1) -> +3V3
- R26 pad 2: Net-(R23-Pad2) -> /stm32/encoder_a
- R27 pad 1: Net-(R27-Pad1) -> +3V3
- R27 pad 2: GND -> /stm32/encoder_b
- R28 pad 1: Net-(C30-Pad1) -> /Sheet6035C8EF/CPVDD
- R28 pad 2: Net-(R27-Pad1) -> +3V3
- R29 pad 1: Net-(R29-Pad1) -> /Sheet6035C8EF/AVDD
- R29 pad 2: VDD -> +3V3
- R30 pad 1: GND -> /Sheet6035C8EF/DVDD
- R30 pad 2: Net-(R30-Pad2) -> +3V3
- R31 pad 1: /TAS6424/tas6424_power/vdd_33 -> Net-(R31-Pad1)
- R31 pad 2: +3V3 -> Net-(C36-Pad2)
- R32 pad 1: /tas6424_en -> Net-(C40-Pad1)
- R32 pad 2: GND -> Net-(C43-Pad1)
- R33 pad 1: Net-(Q2-Pad2) -> Net-(C48-Pad1)
- R33 pad 2: /tas6424_en -> Net-(R33-Pad2)
- R34 pad 1: Net-(Q3-Pad1) -> Net-(R33-Pad2)
- R34 pad 2: Net-(Q2-Pad3) -> Net-(C36-Pad2)
- R35 pad 2: Net-(Q2-Pad3) -> GND
- R36 pad 1: VCC -> GND
- R36 pad 2: Net-(Q3-Pad1) -> Net-(R36-Pad2)
- R37 pad 1: Net-(D2-Pad1) -> Net-(C54-Pad1)
- R38 pad 1: Net-(Q4-Pad1) -> GND
- R38 pad 2: Net-(D2-Pad1) -> Net-(C55-Pad2)
- R39 pad 1: Net-(D1-Pad2) -> Net-(J3-PadA4)
- U1 pad 1: Net-(R2-Pad2) -> /stm32/SPDIF_RX
- U13 pad 46: Net-(J7-Pad1) -> Net-(AE1-Pad1)
- U13 pad 54: /BT_spdif -> Net-(U13-Pad54)
- U2 pad 26: /headphone_mute -> Net-(U2-Pad26)
- U2 pad 3: /tas6424_fault -> Net-(U2-Pad3)
- U2 pad 38: /BT_spdif -> Net-(U2-Pad38)
- U2 pad 4: /tas6424_warn -> Net-(U2-Pad4)
- U2 pad 51: /tas6424_mute -> Net-(U2-Pad51)
- U2 pad 53: /headphone_irq -> Net-(U2-Pad53)
- U2 pad 8: /SAI1_B_MCK -> Net-(U2-Pad8)
- U2 pad 9: /SAI1_A_SD -> Net-(U2-Pad9)
- U3 pad 2: Net-(C18-Pad1) -> VCC
- U4 pad 2: Net-(C22-Pad1) -> Net-(R22-Pad2)
- U5 pad 1: VDD -> /Sheet6035C8EF/DVDD
- U5 pad 10: +3.3VA -> /Sheet6035C8EF/OUTLP
- U5 pad 11: +3.3VA -> /Sheet6035C8EF/OUTLN
- U5 pad 12: +3.3VA -> /Sheet6035C8EF/OUTRP
- U5 pad 13: +3.3VA -> /Sheet6035C8EF/OUTRN
- U5 pad 2: VDD -> Net-(C22-Pad1)
- U5 pad 3: Net-(R26-Pad1) -> GND
- U5 pad 4: VDD -> /Sheet6035C8EF/DVDD
- U5 pad 5: Net-(R29-Pad1) -> /Sheet6035C8EF/CPVDD
- U5 pad 6: Net-(R30-Pad2) -> Net-(C27-Pad2)
- U5 pad 7: VDD -> GND
- U5 pad 8: Net-(C30-Pad1) -> Net-(C27-Pad1)
- U5 pad 9: GND -> Net-(C32-Pad1)
Routing:
- net /TAS6424/gnd_x: track 463.3 -> 0.00 mm, vias 17 -> 0
- net GND: track 676.5 -> 1003.8 mm
- net /TAS6424/vcc_x: track 242.0 -> 0.00 mm, vias 8 -> 0
- net Net-(C36-Pad2): track 0.00 -> 106.3 mm, vias 0 -> 2
- net /tas6424_warn: track 74.8 -> 0.00 mm, vias 3 -> 0
- net /tas6424_fault: track 71.2 -> 0.00 mm, vias 3 -> 0
- net /headphone_in: track 55.6 -> 123.9 mm, vias 0 -> 3
- net /tas6424_en: track 135.6 -> 67.3 mm, vias 4 -> 2
- net /stm32/NRST: track 46.0 -> 114.2 mm, vias 0 -> 3
- net +15V: track 0.00 -> 67.7 mm, vias 0 -> 3
- net /headphone_mute: track 67.0 -> 0.00 mm, vias 2 -> 0
- net VCC: track 183.2 -> 117.8 mm, vias 6 -> 0
- net /SAI1_B_MCK: track 62.4 -> 0.00 mm, vias 1 -> 0
- net /tas6424_mute: track 57.0 -> 0.00 mm, vias 3 -> 0
- net -15V: track 0.00 -> 56.9 mm, vias 0 -> 3
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Other:
- outline, holes or cut-outs redrawn
- net class Default: clearance 0.15 -> 0.2
- rule trace_clearance: 0.15 -> 0.2

Commit message: v3
Parts:
- removed C125: 22uf, Capacitor_SMD:C_0805_2012Metric
- removed C126: 10uf, Capacitor_SMD:C_0805_2012Metric
- removed the C22 at (102.5, 109.9)
- removed the C25 at (96.1, 120.3)
- removed the C27 at (95.4, 109.9)
- removed the C32 at (95.4, 107.8)
- removed the C42 at (81.3, 72.3)
- removed the C43 at (72.1, 72.8)
- removed the C44 at (74.9, 122.6)
- removed the C47 at (78.4, 124.2)
- removed the C53 at (78.5, 122.6)
- removed the C58 at (87.8, 112.4)
- removed J8: Conn_01x02, Connector_JST:JST_VH_S2P-VH_1x02_P3.96mm_Horizontal
- removed the R27 at (116.8, 142.6)
- removed the R40 at (90.6, 111.4)
- removed the R41 at (90.6, 113.5)
- removed the R42 at (90.6, 115.7)
- removed the R43 at (90.6, 117.9)
- removed the R49 at (84.8, 115.7)
- removed the R50 at (84.8, 117.9)
- removed R73: 0Ω, Resistor_SMD:R_0805_2012Metric
- added C100: 100nf, Capacitor_SMD:C_0805_2012Metric, F.Cu at (97.3, 87.1)
- added C101: 1uf, Capacitor_SMD:C_0805_2012Metric, B.Cu at (80.5, 104.2)
- added C102: 2.2uf, Capacitor_SMD:C_0805_2012Metric, F.Cu at (84.8, 104.1)
- added C103: 2.2uf, Capacitor_SMD:C_0805_2012Metric, B.Cu at (86.9, 104.1)
- added C105: 100uf, Capacitor_SMD:C_1210_3225Metric, F.Cu at (100.6, 80.8)
- added C24: 10uf, Capacitor_SMD:C_0805_2012Metric, F.Cu at (88.6, 115.3)
- added C26: 0.1uf, Capacitor_SMD:C_0805_2012Metric, F.Cu at (92.7, 115.3)
- added C29: 10uf, Capacitor_SMD:C_0805_2012Metric, F.Cu at (80.5, 129.0)
- added C35: 2.2uf, Capacitor_SMD:C_0805_2012Metric, F.Cu at (115.9, 70.9)
- added C38: 100nf, Capacitor_SMD:C_0805_2012Metric, F.Cu at (120.4, 76.7)
- added C39: 1.2nf, Capacitor_SMD:C_0805_2012Metric, F.Cu at (113.8, 86.4)
- added C40: 1.3pf, Capacitor_SMD:C_0805_2012Metric, F.Cu at (128.0, 78.2)
- added C45: 4.7uf, Capacitor_SMD:C_0805_2012Metric, F.Cu at (61.2, 105.4)
- added C48: 10uf, Capacitor_SMD:C_0805_2012Metric, F.Cu at (85.6, 134.6)
- added C54: 100nf, Capacitor_SMD:C_0805_2012Metric, F.Cu at (64.3, 131.1)
- added C60: 100nf, Capacitor_SMD:C_0805_2012Metric, F.Cu at (72.6, 131.1)
- added C61: 1uf, Capacitor_SMD:C_0805_2012Metric, F.Cu at (82.8, 104.1)
- added C62: 1uf, Capacitor_SMD:C_0805_2012Metric, F.Cu at (80.8, 104.1)
- added C63: 10uf, Capacitor_SMD:C_0805_2012Metric, F.Cu at (78.2, 104.1)
- added C64: 1uf, Capacitor_SMD:C_0603_1608Metric, B.Cu at (91.5, 94.5)
- added C65: 1uf, Capacitor_SMD:C_0603_1608Metric, B.Cu at (93.5, 94.5)
- added C66: 1uf, Capacitor_SMD:C_0603_1608Metric, B.Cu at (87.6, 94.5)
- added C67: 1uf, Capacitor_SMD:C_0603_1608Metric, B.Cu at (89.8, 94.5)
- added C68: 1uf, Capacitor_SMD:C_0603_1608Metric, B.Cu at (83.2, 94.5)
- added C69: 1uf, Capacitor_SMD:C_0603_1608Metric, B.Cu at (85.1, 94.5)
- added C70: 1uf, Capacitor_SMD:C_0603_1608Metric, B.Cu at (79.2, 94.5)
- added C71: 1uf, Capacitor_SMD:C_0603_1608Metric, B.Cu at (81.4, 94.5)
- added C72: 1uf, Capacitor_SMD:C_0805_2012Metric, B.Cu at (86.4, 62.0)
- added C73: 1uf, Capacitor_SMD:C_0805_2012Metric, B.Cu at (82.3, 62.0)
- added C74: 1uf, Capacitor_SMD:C_0805_2012Metric, B.Cu at (78.2, 62.0)
- added C75: 1uf, Capacitor_SMD:C_0805_2012Metric, B.Cu at (74.2, 62.0)
- added C76: 1uf, Capacitor_SMD:C_0805_2012Metric, B.Cu at (70.1, 62.0)
- added C77: 1uf, Capacitor_SMD:C_0805_2012Metric, B.Cu at (66.0, 62.0)
- added C78: 1uf, Capacitor_SMD:C_0805_2012Metric, B.Cu at (62.0, 62.0)
- added C79: 1uf, Capacitor_SMD:C_0805_2012Metric, B.Cu at (57.9, 62.0)
- added C80: 1nf, Capacitor_SMD:C_0805_2012Metric, B.Cu at (88.4, 62.0)
- added C81: 1nf, Capacitor_SMD:C_0805_2012Metric, B.Cu at (84.3, 62.0)
- added C82: 1nf, Capacitor_SMD:C_0805_2012Metric, B.Cu at (80.3, 62.0)
- added C83: 1nf, Capacitor_SMD:C_0805_2012Metric, B.Cu at (76.2, 62.0)
- added C84: 1nf, Capacitor_SMD:C_0805_2012Metric, B.Cu at (72.1, 62.0)
- added C85: 1nf, Capacitor_SMD:C_0805_2012Metric, B.Cu at (68.1, 62.0)
- added C86: 1nf, Capacitor_SMD:C_0805_2012Metric, B.Cu at (64.0, 62.0)
- added C87: 1nf, Capacitor_SMD:C_0805_2012Metric, B.Cu at (59.9, 62.0)
- added C88: 100uf, Capacitor_SMD:C_1210_3225Metric, B.Cu at (74.2, 101.6)
- added C89: 10uf, Capacitor_SMD:C_0805_2012Metric, F.Cu at (73.8, 101.1)
- added C9: 12pf, Capacitor_SMD:C_0805_2012Metric, F.Cu at (108.7, 134.1)
- added C90: 10uf, Capacitor_SMD:C_0805_2012Metric, B.Cu at (72.1, 86.9)
- added C91: 10uf, Capacitor_SMD:C_0805_2012Metric, F.Cu at (99.8, 100.6)
- added C92: 100nf, Capacitor_SMD:C_0805_2012Metric, F.Cu at (76.2, 101.1)
- added C93: 100nf, Capacitor_SMD:C_0805_2012Metric, F.Cu at (75.7, 90.9)
- added C94: 100nf, Capacitor_SMD:C_0805_2012Metric, F.Cu at (90.9, 104.1)
- added C95: 100uf, Capacitor_SMD:C_1210_3225Metric, B.Cu at (96.0, 87.9)
- added C96: 100uf, Capacitor_SMD:C_1210_3225Metric, B.Cu at (69.1, 86.4)
- added C97: 10uf, Capacitor_SMD:C_0805_2012Metric, F.Cu at (97.3, 85.1)
- added C98: 10uf, Capacitor_SMD:C_0805_2012Metric, B.Cu at (93.0, 88.4)
- added C99: 100nf, Capacitor_SMD:C_0805_2012Metric, B.Cu at (90.9, 88.4)
- added H5: m3, MountingHole:MountingHole_3.2mm_M3_Pad, F.Cu at (68.7, 94.9)
- added H6: m3, MountingHole:MountingHole_3.2mm_M3_Pad, F.Cu at (106.8, 94.9)
- added J1: i2c, Connector_PinHeader_2.54mm:PinHeader_1x04_P2.54mm_Vertical, F.Cu at (98.6, 147.3)
- added L10: 3.3uh, Inductor_SMD:L_6.3x6.3_H3, F.Cu at (70.0, 67.6)
- added L11: 3.3uh, Inductor_SMD:L_6.3x6.3_H3, F.Cu at (63.0, 67.6)
- added L12: 4.7uh, Inductor_SMD:L_6.3x6.3_H3, F.Cu at (96.6, 73.9)
- added L3: 22uh, Inductor_SMD:L_6.3x6.3_H3, F.Cu at (132.3, 86.0)
- added L4: 3.3uh, Inductor_SMD:L_6.3x6.3_H3, F.Cu at (87.1, 75.2)
- added L5: 3.3uh, Inductor_SMD:L_6.3x6.3_H3, F.Cu at (80.1, 75.2)
- added L6: 3.3uh, Inductor_SMD:L_6.3x6.3_H3, F.Cu at (73.2, 75.2)
- added L7: 3.3uh, Inductor_SMD:L_6.3x6.3_H3, F.Cu at (66.2, 75.2)
- added L8: 3.3uh, Inductor_SMD:L_6.3x6.3_H3, F.Cu at (83.9, 67.6)
- added L9: 3.3uh, Inductor_SMD:L_6.3x6.3_H3, F.Cu at (77.0, 67.6)
- added R26: 121k, Resistor_SMD:R_0805_2012Metric, F.Cu at (112.3, 74.7)
- added R28: 68.1k, Resistor_SMD:R_0805_2012Metric, F.Cu at (114.8, 83.3)
- added R30: 215k, Resistor_SMD:R_0805_2012Metric, F.Cu at (111.3, 79.8)
- added R31: 12.1k, Resistor_SMD:R_0805_2012Metric, F.Cu at (111.3, 77.7)
- added R33: 12.1k, Resistor_SMD:R_0805_2012Metric, F.Cu at (124.0, 78.2)
- added R45: 402Ω, Resistor_SMD:R_0805_2012Metric, F.Cu at (75.4, 122.9)
- added R46: 806Ω, Resistor_SMD:R_0805_2012Metric, F.Cu at (75.4, 116.8)
- added R55: 0Ω, Resistor_SMD:R_0805_2012Metric, F.Cu at (54.4, 86.9)
- added R56: 0Ω, Resistor_SMD:R_0805_2012Metric, F.Cu at (99.8, 102.6)
- added R6: 1.5k, Resistor_SMD:R_0805_2012Metric, F.Cu at (117.3, 97.8)
- added U11: TPA6120A2DWP, ti:TPA6120A2DWP, F.Cu at (64.0, 121.9)
- added U12: TAS6424QDKQRQ1, ti:TAS6424QDKQRQ1, F.Cu at (87.1, 94.9)
- added U7: TPS54360DDA, Package_SO:TI_SO-PowerPAD-8_ThermalVias, F.Cu at (116.3, 76.7)
- C10: value 100nf/10v -> 100nf; footprint Capacitor_SMD:C_0603_1608Metric -> Resistor_SMD:R_0805_2012Metric
- C11: value 100nf/10v -> 100nf; footprint Capacitor_SMD:C_0603_1608Metric -> Capacitor_SMD:C_0805_2012Metric
- C12: value 100nf/10v -> 100nf; footprint Capacitor_SMD:C_0603_1608Metric -> Capacitor_SMD:C_0805_2012Metric; moved to B.Cu
- C13: value 10uf -> 100nf; moved to B.Cu
- C14: moved to B.Cu
- C15: value 100nf -> 4.7uf; moved to F.Cu
- C16: value 100nf -> 6.8nf; moved to F.Cu
- C17: value 100nf -> 39pf; footprint Resistor_SMD:R_0805_2012Metric -> Capacitor_SMD:C_0805_2012Metric
- C18: value 4.7uf -> 100nf
- C19: value 100nf -> 47uf
- C2: value 10uf -> 100nf/10v
- C20: value 4.7uf -> 47uf
- C21: value 6.8nf -> 10uf
- C22: renamed from C23; value 39pf -> 22uf
- C23: renamed from C24; value 100nf -> 10uf
- C25: renamed from C26; value 10uf -> 100nf
- C27: renamed from C28; value 47uf -> 1uf
- C28: renamed from C29; value 47uf -> 2.2uf/25v
- C3, C4: value 100nf -> 100nf/10v; moved to F.Cu
- C30: value 10uf -> 100nf
- C31: value 100nf -> 2.2uF/25V
- C32: renamed from C33; moved to F.Cu
- C34: renamed from C35; value 10uf -> 2.2uf
- C36: value 1uf -> 2.2uf
- C37: value 100uf -> 1.3pf; footprint Capacitor_SMD:C_1210_3225Metric -> Capacitor_SMD:C_0805_2012Metric
- C41: renamed from C38; value 10uf -> 100nf; moved to F.Cu
- C42: renamed from C39; value 10uf -> 1.2nf; moved to F.Cu
- C43: renamed from C40; value 750pf -> 22uf
- C44: renamed from C41; value 100nf -> 22uf
- C46: renamed from C45; value 100uf -> 4.7uf; footprint Capacitor_SMD:C_1210_3225Metric -> Capacitor_SMD:C_0805_2012Metric
- C47: renamed from C46; moved to F.Cu
- C49: renamed from C48; value 22uf -> 100uf; footprint Capacitor_SMD:C_0805_2012Metric -> Capacitor_SMD:C_1210_3225Metric
- C5: value 100nf -> 10uf; moved to F.Cu
- C50: renamed from C49; value 22uf -> 10uf
- C51: renamed from C50; value 100nf -> 1nf
- C52: renamed from C51; value 22uf -> 1nf
- C53: renamed from C52; value 22uf -> 10uf
- C55: renamed from C54; value 4.7uf -> 100nf
- C56: renamed from C55; value 4.7uf -> 100uf; footprint Capacitor_SMD:C_0805_2012Metric -> Capacitor_SMD:C_1210_3225Metric
- C59: value 100pf -> 100nf
- C6: value 12pf -> 100nf; footprint Capacitor_SMD:C_0603_1608Metric -> Capacitor_SMD:C_0805_2012Metric
- C7: value 12pf -> 100nf/10v; footprint Capacitor_SMD:C_0603_1608Metric -> Capacitor_SMD:C_0805_2012Metric
- C8: value 100nf/10v -> 12pf; footprint Capacitor_SMD:C_0603_1608Metric -> Capacitor_SMD:C_0805_2012Metric
- D1: value 60v 3A -> B560C
- D2: value 60v 3A -> 40v 5A
- D4: value 40v 5A -> 60v/3A
- D5: value B560C -> 60v 3A
- D6: value 0805 -> D; footprint LED_SMD:LED_0805_2012Metric -> Diode_SMD:D_SMA
- J2: value encoder -> USB_B; footprint Connector_PinHeader_2.54mm:PinHeader_1x04_P2.54mm_Vertical -> Connector_USB:USB_B_OST_USB-B1HSxx_Horizontal
- J3: value USB_C_Receptacle -> encoder; footprint Connector_USB:USB_C_Receptacle_Amphenol_12401548E4-2A -> Connector_PinHeader_2.54mm:PinHeader_1x04_P2.54mm_Vertical
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- renumbered C34 to C33, C56 to C57, C57 to C58
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Connections:
- C11 pad 1: +3V3 -> /stm32/NRST
- C12 pad 1: +3V3 -> /stm32/encoder_sw
- C13 pad 1: /stm32/AVDD -> /stm32/encoder_a
- C14 pad 1: /stm32/AVDD -> /stm32/encoder_b
- C15 pad 1: +3V3 -> VCC
- C16 pad 1: /stm32/NRST -> Net-(C16-Pad1)
- C17 pad 1: +3V3 -> Net-(C17-Pad1)
- C18 pad 1: VCC -> Net-(C18-Pad1)
- C18 pad 2: GND -> Net-(C18-Pad2)
- C19 pad 1: /Sheet6035C8EF/CPVDD -> VDD
- C2 pad 1: /Sheet6035C8EF/CPVDD -> +3V3
- C20 pad 1: VCC -> VDD
- C21 pad 1: Net-(C21-Pad1) -> +3V3
- C22 pad 1: Net-(C23-Pad1) -> /Bluetooth/vdd_x
- C23 pad 1: Net-(C24-Pad1) -> /Bluetooth/vdd_x
- C23 pad 2: Net-(C24-Pad2) -> GND
- C25 pad 1: +3V3 -> /Sheet6035C8EF/CPVDD
- C27 pad 1: VDD -> GND
- C27 pad 2: GND -> Net-(C27-Pad2)
- C28 pad 1: VDD -> Net-(C28-Pad1)
- C28 pad 2: GND -> Net-(C28-Pad2)
- C3 pad 1: /stm32/encoder_sw -> +3V3
- C31 pad 1: /Sheet6035C8EF/AVDD -> Net-(C31-Pad1)
- C36 pad 2: Net-(C36-Pad2) -> -15V
- C37 pad 1: +15V -> Net-(C37-Pad1)
- C4 pad 1: /stm32/encoder_a -> +3V3
- C41 pad 1: +15V -> Net-(C41-Pad1)
- C41 pad 2: GND -> Net-(C41-Pad2)
- C42 pad 1: +15V -> Net-(C42-Pad1)
- C42 pad 2: GND -> -15V
- C43 pad 1: Net-(C40-Pad1) -> +15V
- C43 pad 2: Net-(C36-Pad2) -> GND
- C44 pad 1: +15V -> GND
- C44 pad 2: GND -> -15V
- C46 pad 1: -15V -> GND
- C46 pad 2: GND -> Net-(C46-Pad2)
- C47 pad 1: -15V -> +12V
- C49 pad 1: Net-(C48-Pad1) -> +12V
- C5 pad 1: /stm32/encoder_b -> /stm32/AVDD
- C50 pad 1: GND -> +12V
- C50 pad 2: Net-(C36-Pad2) -> GND
- C51 pad 1: -15V -> Net-(C51-Pad1)
- C51 pad 2: GND -> Net-(C51-Pad2)
- C52 pad 1: Net-(C48-Pad1) -> Net-(C52-Pad1)
- C52 pad 2: GND -> Net-(C52-Pad2)
- C53 pad 1: GND -> +12V
- C53 pad 2: Net-(C36-Pad2) -> GND
- C55 pad 1: Net-(C54-Pad1) -> +12V
- C56 pad 1: GND -> -12V
- C56 pad 2: Net-(C55-Pad2) -> GND
- C57 pad 1: +15V -> -12V
- C58 pad 1: GND -> -12V
- C58 pad 2: -15V -> GND
- C59 pad 1: Net-(C59-Pad1) -> -12V
- C59 pad 2: Net-(C59-Pad2) -> GND
- C6 pad 1: /stm32/OSC_IN -> /stm32/AVDD
- C7 pad 1: /stm32/OSC_OUT -> +3V3
- C8 pad 1: +3V3 -> /stm32/OSC_IN
- D1 pad 1: Net-(C48-Pad1) -> Net-(C18-Pad1)
- D1 pad 2: Net-(D1-Pad2) -> GND
- D2 pad 1: Net-(C42-Pad1) -> VCC
- D2 pad 2: Net-(C36-Pad2) -> Net-(D2-Pad2)
- D3 pad 2: Net-(D3-Pad2) -> Net-(D2-Pad2)
- D4 pad 1: VCC -> Net-(C38-Pad2)
- D4 pad 2: Net-(D3-Pad2) -> GND
- D5 pad 1: Net-(C24-Pad1) -> Net-(C41-Pad1)
- D5 pad 2: GND -> -15V
- D6 pad 1: Net-(D6-Pad1) -> VCC
- H1 pad 1: Net-(H1-Pad1) -> (no net)
- H2 pad 1: Net-(H2-Pad1) -> (no net)
- H3 pad 1: Net-(H3-Pad1) -> (no net)
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Routing:
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Other:
- net class signal: clearance 0.15 -> 0.2; trace_width 0.15 -> 0.2
- rule trace_min: 0.15 -> 0.2
- rule via_min_size: 0.6 -> 0.5

Commit message: digital-amplifier2-v3
Parts:
- C37, C40: value 1.3pf -> 220pF
- C39, C42: value 1.2nf -> 4.3nF
- R26, R27: value 121k -> 97.6kOhm
- R28, R29: value 68.1k -> 18.7kOhm

Commit message: main_v4
Parts:
- removed C100, C92, C93, C94, C99: 100nf, Capacitor_SMD:C_0805_2012Metric
- removed C101, C74, C75, C76, C77, C78, C79: 1uf, Capacitor_SMD:C_0805_2012Metric
- removed C102, C103: 2.2uf, Capacitor_SMD:C_0805_2012Metric
- removed C105, C88, C95, C96: 100uf, Capacitor_SMD:C_1210_3225Metric
- removed C80, C81, C82, C83, C84, C85, C86, C87: 1nf, Capacitor_SMD:C_0805_2012Metric
- removed C89, C90, C91, C97, C98: 10uf, Capacitor_SMD:C_0805_2012Metric
- removed D6: D, Diode_SMD:D_SMA
- removed L10, L11, L4, L5, L6, L7, L8, L9: 3.3uh, Inductor_SMD:L_6.3x6.3_H3
- removed L12: 4.7uh, Inductor_SMD:L_6.3x6.3_H3
- added H7: m3, MountingHole:MountingHole_3.2mm_M3_Pad, F.Cu at (55.0, 115.0)
- added H8: m3, MountingHole:MountingHole_3.2mm_M3_Pad, F.Cu at (145.0, 115.0)
- added R57: 10k, Resistor_SMD:R_0805_2012Metric, F.Cu at (83.8, 104.8)
- added R58: 0Ω, Resistor_SMD:R_0805_2012Metric, F.Cu at (92.1, 99.7)
- added R59: 0Ω, Resistor_SMD:R_0805_2012Metric, F.Cu at (87.0, 111.6)
- AE1: moved to F.Cu
- C1: value 4.7uf/10v -> 4.7uf
- C10: value 100nf -> 12pf; footprint Resistor_SMD:R_0805_2012Metric -> Capacitor_SMD:C_0805_2012Metric
- C11: value 100nf -> 12pf
- C15: value 4.7uf -> 100nf; moved to B.Cu
- C16: value 6.8nf -> 4.7uf
- C17: value 39pf -> 6.8nf
- C18: value 100nf -> 39pf
- C19: value 47uf -> 100nf
- C2, C3, C4: value 100nf/10v -> 100nf
- C22: value 22uf -> 10uf
- C23: value 10uf -> 22uf
- C25, C30: value 100nf -> 100uf; footprint Capacitor_SMD:C_0805_2012Metric -> Capacitor_SMD:C_1210_3225Metric
- C26: value 0.1uf -> 10uf
- C27: value 1uf -> 10uf
- C28: value 2.2uf/25v -> 100nf
- C29, C33, C48, C53, C57: value 10uf -> 100nf
- C31: value 2.2uF/25V -> 10uf
- C32, C54: value 100nf -> 10uf
- C34: value 2.2uf -> 100nf
- C37: value 220pF -> 2.2uf
- C38, C41: value 100nf -> 220pF
- C39, C42: value 4.3nF -> 100nf
- C40: value 220pF -> 4.3nF
- C43: value 22uf -> 4.3nF
- C45: value 4.7uf -> 22uf
- C46: value 4.7uf -> 10uf
- C49: value 100uf -> 100nf; footprint Capacitor_SMD:C_1210_3225Metric -> Capacitor_SMD:C_0805_2012Metric
- C51: value 1nf -> 100nf
- C52: value 1nf -> 10uf
- C56: value 100uf -> 10uf; footprint Capacitor_SMD:C_1210_3225Metric -> Capacitor_SMD:C_0805_2012Metric
- C58: moved to B.Cu
- C60: value 100nf -> 47uf
- C61: value 1uf -> 47uf
- C62: value 1uf -> 2.7nf
- C63: value 10uf -> 2.7nf
- C64, C65: value 1uf -> 2.7nf; footprint Capacitor_SMD:C_0603_1608Metric -> Capacitor_SMD:C_0805_2012Metric; moved to F.Cu
- C66, C68, C70, C71: value 1uf -> 10uf; footprint Capacitor_SMD:C_0603_1608Metric -> Capacitor_SMD:C_0805_2012Metric; moved to F.Cu
- C67, C69: value 1uf -> 100nf; footprint Capacitor_SMD:C_0603_1608Metric -> Capacitor_SMD:C_0805_2012Metric; moved to F.Cu
- C7: value 100nf/10v -> 100nf; footprint Capacitor_SMD:C_0805_2012Metric -> Resistor_SMD:R_0805_2012Metric
- C72, C73: value 1uf -> 100nf; moved to F.Cu
- C8, C9: value 12pf -> 100nf
- D1: value B560C -> 40v 5A
- D3: value 40v 5A -> B560C
- J1: value i2c -> Conn_01x10_Female; footprint Connector_PinHeader_2.54mm:PinHeader_1x04_P2.54mm_Vertical -> Connector_PinHeader_2.54mm:PinHeader_1x10_P2.54mm_Vertical
- J3: value encoder -> Barrel_Jack_Switch; footprint Connector_PinHeader_2.54mm:PinHeader_1x04_P2.54mm_Vertical -> connector:DC-044A_5.5-2.1
- J4: value swd -> encoder
- J5: value Barrel_Jack_Switch -> Conn_ARM_JTAG_SWD_20; footprint connector:DC-044A_5.5-2.1 -> Connector_PinHeader_2.54mm:PinHeader_2x10_P2.54mm_Vertical
- J7: value Conn_01x08 -> AudioJack3_Switch; footprint Connector_JST:JST_VH_B8P-VH-B_1x08_P3.96mm_Vertical -> Connector_Audio:Jack_6.35mm_Neutrik_NMJ6HFD2-AU_Horizontal
- R15: value 523k -> 9.53k; moved to B.Cu
- R16: value 84.5k -> 9.53k; moved to B.Cu
- R17: value 162k -> 9.53k; moved to B.Cu
- R18: value 13k -> 162k
- R19: value 53.6k -> 13k
- R20: value 10.2k -> 53.6k
- R21: value 0Ω -> 10.2k
- R25, R56: value 0Ω -> 1k
- R26, R27: value 97.6kOhm -> 1k
- R28, R29: value 18.7kOhm -> 1k
- R3: value 1mΩ -> 4.7k; footprint Resistor_SMD:R_0603_1608Metric -> Resistor_SMD:R_0805_2012Metric
- R30, R32: value 215k -> 1k
- R31: value 12.1k -> 1k
- R33: value 12.1k -> 1m
- R34: value 200k -> 39.2Ω
- R35: value 150k -> 39.2Ω
- R36: value 200k -> 97.6kOhm
- R37: value 150k -> 97.6kOhm
- R38, R39: value 402Ω -> 18.7kOhm
- R4: value 9.53k -> 4.7k
- R40, R42: value 402Ω -> 215k
- R41, R43: value 402Ω -> 12.1k
- R44, R45: value 402Ω -> 0Ω
- R46: value 806Ω -> 1k
- R47: value 806Ω -> 10k
- R48, R49: value 806Ω -> 0Ω
- R5: value 4.7k -> 9.53k; moved to F.Cu
- R50: value 9.53k -> 10k
- R51, R52: value 39.2Ω -> 1k
- R53: value 9.53k -> 1k
- R55: value 0Ω -> 9.53k
- R6: value 1.5k -> 1mΩ; footprint Resistor_SMD:R_0805_2012Metric -> Resistor_SMD:R_0603_1608Metric
- R7: value 4.7k -> 1.5k; moved to F.Cu
- U10: value LT3094xMSE -> LM317_SOT-223; footprint Package_SO:MSOP-12-1EP_3x4mm_P0.65mm_EP1.65x2.85mm -> Package_TO_SOT_SMD:SOT-223-3_TabPin2
- U11: value TPA6120A2DWP -> LM337_SOT223; footprint ti:TPA6120A2DWP -> Package_TO_SOT_SMD:SOT-223-3_TabPin2
- U12: value TAS6424QDKQRQ1 -> PCM1792A; footprint ti:TAS6424QDKQRQ1 -> Package_SO:SSOP-28_5.3x10.2mm_P0.65mm
- U13: value LM317_SOT-223 -> OPA4134; footprint Package_TO_SOT_SMD:SOT-223-3_TabPin2 -> Package_SO:SOIC-14_3.9x8.7mm_P1.27mm
- U5: value SJR-BTM331 -> AMS1117-5.0; footprint misc:SJR-BTM331 -> Package_TO_SOT_SMD:SOT-223-3_TabPin2; moved to F.Cu
- U6: value PCM5242 -> SJR-BTM331; footprint ti:PCM5242RHBR -> misc:SJR-BTM331
- U7: value TPS54360DDA -> TPA6120A2DWP; footprint Package_SO:TI_SO-PowerPAD-8_ThermalVias -> ti:TPA6120A2DWP
- U9: value LT3045xMSE-1 -> TPS54360DDA; footprint Package_SO:MSOP-12-1EP_3x4mm_P0.65mm_EP1.65x2.85mm -> Package_SO:TI_SO-PowerPAD-8_ThermalVias
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Connections:
- C10 pad 1: +3V3 -> /stm32/OSC_IN
- C11 pad 1: /stm32/NRST -> /stm32/OSC_OUT
- C15 pad 1: VCC -> +3V3
- C16 pad 1: Net-(C16-Pad1) -> VCC
- C18 pad 2: Net-(C18-Pad2) -> GND
- C19 pad 1: VDD -> Net-(C19-Pad1)
- C19 pad 2: GND -> Net-(C19-Pad2)
- C2 pad 1: +3V3 -> /stm32/vdd1
- C20 pad 1: VDD -> +7.5V
- C22 pad 1: /Bluetooth/vdd_x -> +5V
- C24 pad 1: /Sheet6035C8EF/CPVDD -> /Bluetooth/vdd_x
- C25 pad 1: /Sheet6035C8EF/CPVDD -> +12V
- C26 pad 1: Net-(C26-Pad1) -> +12V
- C27 pad 1: GND -> +12V
- C27 pad 2: Net-(C27-Pad2) -> GND
- C28 pad 1: Net-(C28-Pad1) -> +12V
- C28 pad 2: Net-(C28-Pad2) -> GND
- C29 pad 1: /Sheet6035C8EF/AVDD -> +12V
- C3 pad 1: +3V3 -> /stm32/vdd1
- C30 pad 1: /Sheet6035C8EF/AVDD -> -12V
- C31 pad 1: Net-(C31-Pad1) -> -12V
- C32 pad 1: /Sheet6035C8EF/DVDD -> -12V
- C33 pad 1: /Sheet6035C8EF/DVDD -> -12V
- C34 pad 1: VCC -> -12V
- C36 pad 2: -15V -> GND
- C37 pad 1: Net-(C37-Pad1) -> VCC
- C37 pad 2: GND -> -15V
- C38 pad 2: Net-(C38-Pad2) -> GND
- C39 pad 2: GND -> Net-(C39-Pad2)
- C4 pad 1: +3V3 -> /stm32/vdd1
- C40 pad 2: -15V -> GND
- C41 pad 2: Net-(C41-Pad2) -> -15V
- C42 pad 2: -15V -> Net-(C42-Pad2)
- C43 pad 1: +15V -> Net-(C43-Pad1)
- C43 pad 2: GND -> -15V
- C44 pad 1: GND -> +15V
- C44 pad 2: -15V -> GND
- C45 pad 1: Net-(C45-Pad1) -> GND
- C45 pad 2: GND -> -15V
- C46 pad 1: GND -> Net-(C46-Pad1)
- C46 pad 2: Net-(C46-Pad2) -> GND
- C47 pad 1: +12V -> GND
- C47 pad 2: GND -> Net-(C47-Pad2)
- C48 pad 1: GND -> Net-(C46-Pad1)
- C48 pad 2: -12V -> GND
- C49 pad 1: +12V -> GND
- C49 pad 2: GND -> Net-(C47-Pad2)
- C5 pad 1: /stm32/AVDD -> /stm32/vdd1
- C50 pad 1: +12V -> /PCM1792/vdd1
- C51 pad 1: Net-(C51-Pad1) -> /PCM1792/vdd1
- C51 pad 2: Net-(C51-Pad2) -> GND
- C52 pad 1: Net-(C52-Pad1) -> /PCM1792/vdd2
- C52 pad 2: Net-(C52-Pad2) -> GND
- C53 pad 1: +12V -> /PCM1792/vdd2
- C54 pad 1: +12V -> /PCM1792/vdd2
- C55 pad 1: +12V -> /PCM1792/vdd2
- C56 pad 1: -12V -> /PCM1792/vdd2
- C57 pad 1: -12V -> /PCM1792/vdd2
- C58 pad 1: -12V -> /PCM1792/vdd2
- C59 pad 1: -12V -> /PCM1792/vdd2
- C6 pad 1: /stm32/AVDD -> /stm32/vdd1
- C60 pad 1: -12V -> Net-(C60-Pad1)
- C60 pad 2: GND -> /PCM1792/vdd2
- C61 pad 2: Net-(C61-Pad2) -> /PCM1792/vdd2
- C62 pad 1: Net-(C62-Pad1) -> /OPA4134/OUTC
- C62 pad 2: Net-(C61-Pad2) -> /OPA4134/INC
- C63 pad 1: /Sheet605867F7/vbat -> /TPA6120A2/LIN+
- C63 pad 2: GND -> /OPA4134/INA
- C64 pad 1: /Sheet605867F7/OUT_1P -> /TPA6120A2/LIN-
- C64 pad 2: /Sheet605867F7/BST_1P -> /OPA4134/INB
- C65 pad 1: /Sheet605867F7/BST_1M -> /OPA4134/OUTD
- C65 pad 2: /Sheet605867F7/OUT_1M -> /OPA4134/IND
- C66 pad 1: /Sheet605867F7/OUT_2P -> -12V
- C66 pad 2: /Sheet605867F7/BST_2P -> GND
- C67 pad 1: /Sheet605867F7/BST_2M -> -12V
- C67 pad 2: /Sheet605867F7/OUT_2M -> GND
- C68 pad 1: /Sheet605867F7/OUT_3P -> +12V
- C68 pad 2: /Sheet605867F7/BST_3P -> GND
- C69 pad 1: /Sheet605867F7/BST_3M -> +12V
- C69 pad 2: /Sheet605867F7/OUT_3M -> GND
- C7 pad 1: +3V3 -> /stm32/vdd1
- C70 pad 1: /Sheet605867F7/OUT_4P -> +12V
- C70 pad 2: /Sheet605867F7/BST_4P -> GND
- C71 pad 1: /Sheet605867F7/BST_4M -> GND
- C71 pad 2: /Sheet605867F7/OUT_4M -> -12V
- C72 pad 1: Net-(C72-Pad1) -> +5V
- C73 pad 1: GND -> +7.5V
- C73 pad 2: Net-(C73-Pad2) -> GND
- C8 pad 1: /stm32/OSC_IN -> /stm32/vdd1
- C9 pad 1: /stm32/OSC_OUT -> /stm32/NRST
- D1 pad 1: Net-(C18-Pad1) -> VCC
- D1 pad 2: GND -> Net-(D1-Pad2)
- D2 pad 2: Net-(D2-Pad2) -> Net-(D1-Pad2)
- D3 pad 1: VCC -> Net-(C19-Pad1)
- D3 pad 2: Net-(D2-Pad2) -> GND
- D4 pad 1: Net-(C38-Pad2) -> Net-(C39-Pad2)
- D5 pad 1: Net-(C41-Pad1) -> Net-(C42-Pad1)
- H5 pad 1: GND -> VCC
- J1 pad 1: GND -> /stm32/ext_irq
- J1 pad 2: /SDA -> /stm32/ext_en
- J1 pad 3: /SCL -> /stm32/SAI1_SD_B
- J1 pad 4: +3V3 -> /stm32/SAI1_FS_B
- J3 pad 1: GND -> Net-(D1-Pad2)
- J3 pad 2: /stm32/encoder_b -> GND
- J3 pad 3: /stm32/encoder_a -> (no net)
- J4 pad 2: /stm32/SWDIO -> /stm32/encoder_b
- J4 pad 3: /stm32/SWCLK -> /stm32/encoder_a
- J4 pad 4: /stm32/uart_out -> /stm32/encoder_sw
- J5 pad 1: Net-(D2-Pad2) -> +3V3
- J5 pad 2: GND -> +3V3
- J5 pad 3: (no net) -> /stm32/NJTRST
- J6 pad R1: Net-(J6-PadR1) -> /TPA6120A2/LOUT
- J6 pad R2: Net-(J6-PadR2) -> /TPA6120A2/ROUT
- L1 pad 1: Net-(C18-Pad1) -> Net-(C19-Pad1)
- L1 pad 2: VDD -> +7.5V
- L2 pad 2: Net-(C38-Pad2) -> Net-(C39-Pad2)
- L3 pad 2: Net-(C41-Pad1) -> Net-(C42-Pad1)
- R15 pad 1: VCC -> Net-(J5-Pad17)
- R15 pad 2: Net-(R15-Pad2) -> GND
- R16 pad 1: Net-(R15-Pad2) -> Net-(J5-Pad19)
- R17 pad 1: Net-(R17-Pad1) -> Net-(J5-Pad11)
- R18 pad 1: Net-(C17-Pad1) -> Net-(R18-Pad1)
- R18 pad 2: Net-(C16-Pad1) -> GND
- R19 pad 1: VDD -> Net-(C18-Pad1)
- R19 pad 2: Net-(R19-Pad2) -> Net-(C17-Pad1)
- R2 pad 1: /stm32/AVDD -> /stm32/vdd1
- R20 pad 1: Net-(R19-Pad2) -> +7.5V
- R20 pad 2: GND -> Net-(R20-Pad2)
- R21 pad 1: +3V3 -> Net-(R20-Pad2)
- R21 pad 2: Net-(R21-Pad2) -> GND
- R22 pad 1: /Bluetooth/vdd_x -> +3V3
- R22 pad 2: +3V3 -> Net-(R22-Pad2)
- R23 pad 1: /Sheet6035C8EF/CPVDD -> +5V
- R23 pad 2: +3V3 -> Net-(R23-Pad2)
- R24 pad 1: /Sheet6035C8EF/AVDD -> /Bluetooth/vdd_x
- R25 pad 1: /Sheet6035C8EF/DVDD -> Net-(R25-Pad1)
- R25 pad 2: +3V3 -> /TPA6120A2/LIN+
- R26 pad 2: GND -> /TPA6120A2/LIN-
- R27 pad 2: -15V -> /OPA4134/OUTD
- R28 pad 1: Net-(C37-Pad1) -> Net-(R28-Pad1)
- R28 pad 2: Net-(C39-Pad1) -> /OPA4134/OUTC
- R29 pad 1: Net-(C40-Pad1) -> Net-(R25-Pad1)
- R29 pad 2: Net-(C42-Pad1) -> GND
- R3 pad 1: /stm32/OSC_OUT -> +3V3
- R3 pad 2: /stm32/OSC_IN -> /SCL
- R30 pad 1: +15V -> Net-(R28-Pad1)
- R30 pad 2: /Sheet6035C8EF/sheet5FF87CA5/FB1 -> GND
- R31 pad 1: /Sheet6035C8EF/sheet5FF87CA5/FB1 -> Net-(R26-Pad1)
- R31 pad 2: GND -> Net-(R31-Pad2)
- R32 pad 1: GND -> Net-(R27-Pad1)
- R32 pad 2: /Sheet6035C8EF/sheet5FF87CA5/FB2 -> Net-(R32-Pad2)
- R33 pad 1: /Sheet6035C8EF/sheet5FF87CA5/FB2 -> /headphone_in
- R33 pad 2: -15V -> Net-(J7-PadSN)
- R34 pad 1: Net-(R34-Pad1) -> /TPA6120A2/ROUT
- R34 pad 2: GND -> Net-(R31-Pad2)
- R35 pad 1: Net-(C45-Pad1) -> /TPA6120A2/LOUT
- R35 pad 2: GND -> Net-(R32-Pad2)
- R36 pad 1: GND -> Net-(R36-Pad1)
- R36 pad 2: Net-(R36-Pad2) -> GND
- R37 pad 1: GND -> Net-(R37-Pad1)
- R37 pad 2: Net-(C46-Pad2) -> -15V
- R38 pad 1: Net-(C51-Pad1) -> Net-(C38-Pad1)
- R38 pad 2: /Sheet6035C8EF/OUTLP -> Net-(C40-Pad1)
- R39 pad 1: Net-(C51-Pad2) -> Net-(C41-Pad1)
- R39 pad 2: /Sheet6035C8EF/OUTLN -> Net-(C43-Pad1)
- R4 pad 2: /stm32/NRST -> /SDA
- R40 pad 1: Net-(C52-Pad2) -> +15V
- R40 pad 2: /Sheet6035C8EF/OUTRN -> /headphone_power/FB1
- R41 pad 1: Net-(C52-Pad1) -> /headphone_power/FB1
- R41 pad 2: /Sheet6035C8EF/OUTRP -> GND
- R42 pad 1: Net-(R42-Pad1) -> GND
- R42 pad 2: Net-(C51-Pad1) -> /headphone_power/FB2
- R43 pad 1: Net-(R43-Pad1) -> /headphone_power/FB2
- R43 pad 2: Net-(C51-Pad2) -> -15V
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Routing:
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Other:
- board size 94.5 x 100 mm -> 100 x 100 mm
- net class Default: via_dia 0.6 -> 0.5
- net class p1A: trace_width 0.3 -> 0.4; via_dia 0.6 -> 0.5
- net class signal: via_dia 0.6 -> 0.5
- net class vcc: via_dia 0.6 -> 1; via_drill 0.3 -> 0.6

Commit message: ciruit_save
Parts:
- R20: value 53.6k -> 75k
- R21: value 10.2k -> 9.53k
- R40, R42: value 215k -> 180k
- R41, R43: value 12.1k -> 9.53k
- R47: value 10k -> 7.5
- R57: value 10k -> 7.5k
Changed lines of the file:
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@@
   )
   (setup
-    (last_trace_width 0.4)
+    (last_trace_width 0.2)
     (user_trace_width 0.2)
     (user_trace_width 0.3)
@@
       (effects (font (size 1 1) (thickness 0.15)))
     )
-    (fp_text value 10k (at 0 1.65 90) (layer F.Fab)
+    (fp_text value 7.5k (at 0 1.65 90) (layer F.Fab)
       (effects (font (size 1 1) (thickness 0.15)))
     )
@@
       (effects (font (size 1 1) (thickness 0.15)))
     )
-    (fp_text value 10k (at 0 1.65 90) (layer F.Fab)
+    (fp_text value 7.5 (at 0 1.65 90) (layer F.Fab)
       (effects (font (size 1 1) (thickness 0.15)))
     )
@@
       (effects (font (size 1 1) (thickness 0.15)))
     )
-    (fp_text value 12.1k (at 0 1.65 180) (layer F.Fab)
+    (fp_text value 9.53k (at 0 1.65 180) (layer F.Fab)
       (effects (font (size 1 1) (thickness 0.15)))
     )
@@
       (effects (font (size 1 1) (thickness 0.15)))
     )
-    (fp_text value 12.1k (at 0 1.65) (layer F.Fab)
+    (fp_text value 9.53k (at 0 1.65) (layer F.Fab)
       (effects (font (size 1 1) (thickness 0.15)))
     )
@@
       (effects (font (size 1 1) (thickness 0.15)))
     )
-    (fp_text value 215k (at 0 1.65 270) (layer F.Fab)
+    (fp_text value 180k (at 0 1.65 270) (layer F.Fab)
       (effects (font (size 1 1) (thickness 0.15)))
     )
@@
       (effects (font (size 1 1) (thickness 0.15)))
     )
-    (fp_text value 215k (at 0 1.65 90) (layer F.Fab)
+    (fp_text value 180k (at 0 1.65 90) (layer F.Fab)
       (effects (font (size 1 1) (thickness 0.15)))
     )
@@
       (effects (font (size 1 1) (thickness 0.15)))
     )
-    (fp_text value 53.6k (at 0 1.65 270) (layer F.Fab)
+    (fp_text value 75k (at 0 1.65 270) (layer F.Fab)
       (effects (font (size 1 1) (thickness 0.15)))
     )
@@
       (effects (font (size 1 1) (thickness 0.15)))
     )
-    (fp_text value 10.2k (at 0 1.65) (layer F.Fab)
+    (fp_text value 9.53k (at 0 1.65) (layer F.Fab)
       (effects (font (size 1 1) (thickness 0.15)))
     )
