File: mcu/digital-amplifier2/circuit/main/digital-amplifier2.kicad_pcb (KiCad board)
At the start: 2 copper layers, 100 x 100 mm, 171 parts, among them J1 Conn_01x10_Female, J2 USB_B, J3 Barrel_Jack_Switch, J4 encoder, J5 Conn_ARM_JTAG_SWD_20, J6 AudioJack4, J7 AudioJack3_Switch, Q1 s8550, U1 STM32F446RETx, U10 LM317_SOT-223, U11 LM337_SOT223, U12 PCM1792A, U13 OPA4134, U2 DLT11H0, U3 TPS54360DDA, U4 AMS1117-3.3, U5 AMS1117-5.0, U6 SJR-BTM331, U7 TPA6120A2DWP, U8 TPS54360DDA, U9 TPS54360DDA, Y1 5032 8m

Commit message: pcb
Parts:
- C17: value 6.8nf -> 5.1nF
- C18: value 39pf -> 750pF
- C38: value 220pF -> 750pF
- C40: value 4.3nF -> 5.1nF
- R18: value 162k -> 49.9kOhm
- R19: value 13k -> 15.4k
- R36: value 97.6kOhm -> 49.9kOhm
- R38: value 18.7kOhm -> 15.4kOhm
- R40, R42: value 180k -> 160k
- R56: value 1k -> 7.5k
- R57: value 7.5k -> 1k
Changed lines of the file:
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@@
     (add_net "Net-(C61-Pad1)")
     (add_net "Net-(D1-Pad2)")
+    (add_net "Net-(H1-Pad1)")
+    (add_net "Net-(H2-Pad1)")
+    (add_net "Net-(H3-Pad1)")
+    (add_net "Net-(H4-Pad1)")
+    (add_net "Net-(J2-Pad1)")
     (add_net "Net-(J2-Pad2)")
     (add_net "Net-(J2-Pad3)")
     (add_net "Net-(J2-Pad5)")
+    (add_net "Net-(J3-Pad3)")
     (add_net "Net-(J5-Pad11)")
     (add_net "Net-(J5-Pad17)")
     (add_net "Net-(J5-Pad19)")
     (add_net "Net-(J6-PadT)")
+    (add_net "Net-(J7-PadRN)")
     (add_net "Net-(J7-PadSN)")
+    (add_net "Net-(J7-PadTN)")
     (add_net "Net-(Q1-Pad1)")
     (add_net "Net-(Q1-Pad3)")
@@
     (add_net "Net-(R56-Pad2)")
     (add_net "Net-(R57-Pad2)")
+    (add_net "Net-(U1-Pad10)")
+    (add_net "Net-(U1-Pad11)")
+    (add_net "Net-(U1-Pad2)")
+    (add_net "Net-(U1-Pad22)")
+    (add_net "Net-(U1-Pad26)")
+    (add_net "Net-(U1-Pad27)")
+    (add_net "Net-(U1-Pad28)")
+    (add_net "Net-(U1-Pad34)")
+    (add_net "Net-(U1-Pad37)")
+    (add_net "Net-(U1-Pad38)")
+    (add_net "Net-(U1-Pad39)")
+    (add_net "Net-(U1-Pad40)")
+    (add_net "Net-(U1-Pad41)")
+    (add_net "Net-(U1-Pad57)")
+    (add_net "Net-(U1-Pad61)")
+    (add_net "Net-(U12-Pad1)")
+    (add_net "Net-(U12-Pad2)")
+    (add_net "Net-(U3-Pad3)")
+    (add_net "Net-(U6-Pad1)")
+    (add_net "Net-(U6-Pad10)")
+    (add_net "Net-(U6-Pad11)")
+    (add_net "Net-(U6-Pad12)")
+    (add_net "Net-(U6-Pad16)")
+    (add_net "Net-(U6-Pad17)")
+    (add_net "Net-(U6-Pad18)")
+    (add_net "Net-(U6-Pad19)")
+    (add_net "Net-(U6-Pad20)")
+    (add_net "Net-(U6-Pad22)")
+    (add_net "Net-(U6-Pad25)")
+    (add_net "Net-(U6-Pad26)")
+    (add_net "Net-(U6-Pad27)")
+    (add_net "Net-(U6-Pad29)")
+    (add_net "Net-(U6-Pad30)")
+    (add_net "Net-(U6-Pad32)")
+    (add_net "Net-(U6-Pad33)")
+    (add_net "Net-(U6-Pad34)")
+    (add_net "Net-(U6-Pad35)")
+    (add_net "Net-(U6-Pad36)")
+    (add_net "Net-(U6-Pad37)")
+    (add_net "Net-(U6-Pad39)")
+    (add_net "Net-(U6-Pad40)")
+    (add_net "Net-(U6-Pad41)")
+    (add_net "Net-(U6-Pad42)")
+    (add_net "Net-(U6-Pad43)")
+    (add_net "Net-(U6-Pad48)")
+    (add_net "Net-(U6-Pad49)")
+    (add_net "Net-(U6-Pad50)")
+    (add_net "Net-(U6-Pad51)")
+    (add_net "Net-(U6-Pad52)")
+    (add_net "Net-(U6-Pad53)")
+    (add_net "Net-(U6-Pad54)")
+    (add_net "Net-(U6-Pad6)")
+    (add_net "Net-(U6-Pad7)")
+    (add_net "Net-(U6-Pad8)")
+    (add_net "Net-(U6-Pad9)")
+    (add_net "Net-(U8-Pad3)")
+    (add_net "Net-(U9-Pad3)")
   )
   (net_class p1A ""
@@
       (effects (font (size 1 1) (thickness 0.15)))
     )
-    (fp_text value 7.5k (at 0 1.65 90) (layer F.Fab)
+    (fp_text value 1k (at 0 1.65 90) (layer F.Fab)
       (effects (font (size 1 1) (thickness 0.15)))
     )
@@
       (effects (font (size 1 1) (thickness 0.15)))
     )
-    (fp_text value 1k (at 0 1.65 90) (layer F.Fab)
+    (fp_text value 7.5k (at 0 1.65 90) (layer F.Fab)
       (effects (font (size 1 1) (thickness 0.15)))
     )
@@
       (effects (font (size 1 1) (thickness 0.15)))
     )
-    (fp_text value 220pF (at 0 1.68) (layer F.Fab)
+    (fp_text value 750pF (at 0 1.68) (layer F.Fab)
       (effects (font (size 1 1) (thickness 0.15)))
     )
@@
       (effects (font (size 1 1) (thickness 0.15)))
     )
-    (fp_text value 4.3nF (at 0 1.68 90) (layer F.Fab)
+    (fp_text value 5.1nF (at 0 1.68 90) (layer F.Fab)
       (effects (font (size 1 1) (thickness 0.15)))
     )
@@
       (effects (font (size 1 1) (thickness 0.15)))
     )
-    (fp_text value 6.8nf (at 0 1.68 90) (layer F.Fab)
+    (fp_text value 5.1nF (at 0 1.68 90) (layer F.Fab)
       (effects (font (size 1 1) (thickness 0.15)))
     )
@@
       (effects (font (size 1 1) (thickness 0.15)))
     )
-    (fp_text value 97.6kOhm (at 0 1.65 270) (layer F.Fab)
+    (fp_text value 49.9kOhm (at 0 1.65 270) (layer F.Fab)
       (effects (font (size 1 1) (thickness 0.15)))
     )
@@
       (effects (font (size 1 1) (thickness 0.15)))
     )
-    (fp_text value 18.7kOhm (at 0 1.65 180) (layer F.Fab)
+    (fp_text value 15.4kOhm (at 0 1.65 180) (layer F.Fab)
       (effects (font (size 1 1) (thickness 0.15)))
     )
@@
       (effects (font (size 1 1) (thickness 0.15)))
     )
-    (fp_text value 180k (at 0 1.65 270) (layer F.Fab)
+    (fp_text value 160k (at 0 1.65 270) (layer F.Fab)
       (effects (font (size 1 1) (thickness 0.15)))
     )
@@
       (effects (font (size 1 1) (thickness 0.15)))
     )
-    (fp_text value 180k (at 0 1.65 90) (layer F.Fab)
+    (fp_text value 160k (at 0 1.65 90) (layer F.Fab)
       (effects (font (size 1 1) (thickness 0.15)))
     )
@@
       (effects (font (size 1 1) (thickness 0.15)))
     )
-    (fp_text value 39pf (at 0 1.65 90) (layer F.Fab)
+    (fp_text value 750pF (at 0 1.65 90) (layer F.Fab)
       (effects (font (size 1 1) (thickness 0.15)))
     )
@@
       (effects (font (size 1 1) (thickness 0.15)))
     )
-    (fp_text value 162k (at 0 1.65 180) (layer F.Fab)
+    (fp_text value 49.9kOhm (at 0 1.65 180) (layer F.Fab)
       (effects (font (size 1 1) (thickness 0.15)))
     )
@@
       (effects (font (size 1 1) (thickness 0.15)))
     )
-    (fp_text value 13k (at 0 1.65 90) (layer F.Fab)
+    (fp_text value 15.4k (at 0 1.65 90) (layer F.Fab)
       (effects (font (size 1 1) (thickness 0.15)))
     )

Commit message: v5
Parts:
- removed C47, C70, C71: 10uf, Capacitor_SMD:C_0805_2012Metric
- removed R15, R16, R17: 9.53k, Resistor_SMD:R_0805_2012Metric
- removed R37: 97.6kOhm, Resistor_SMD:R_0805_2012Metric
- removed R38: 15.4kOhm, Resistor_SMD:R_0805_2012Metric
- removed R44, R45: 0Ω, Resistor_SMD:R_0805_2012Metric
- removed R46: 1k, Resistor_SMD:R_0805_2012Metric
- removed U10: LM317_SOT-223, Package_TO_SOT_SMD:SOT-223-3_TabPin2
- removed U11: LM337_SOT223, Package_TO_SOT_SMD:SOT-223-3_TabPin2
- added C74: 10uf, Capacitor_SMD:C_0805_2012Metric, F.Cu at (56.3, 105.9)
- added C75: 10uf, Capacitor_SMD:C_0805_2012Metric, F.Cu at (56.3, 96.4)
- added C76: 10uf, Capacitor_SMD:C_0805_2012Metric, F.Cu at (59.8, 101.6)
- added C77: 100nf, Capacitor_SMD:C_0805_2012Metric, F.Cu at (60.1, 107.8)
- added C82: 10uf, Capacitor_SMD:C_0805_2012Metric, F.Cu at (68.8, 93.6)
- added C83: 100nf, Capacitor_SMD:C_0805_2012Metric, F.Cu at (68.8, 91.4)
- added C84: 22uf, Capacitor_SMD:C_0805_2012Metric, F.Cu at (68.8, 98.7)
- added C85: 10uf, Capacitor_SMD:C_0805_2012Metric, F.Cu at (69.0, 108.1)
- added C86: 100nf, Capacitor_SMD:C_0805_2012Metric, F.Cu at (68.8, 96.6)
- added C87: 100nf, Capacitor_SMD:C_0805_2012Metric, F.Cu at (71.1, 108.1)
- added C88: 22uf, Capacitor_SMD:C_0805_2012Metric, F.Cu at (73.4, 108.1)
- added C89: 100nf, Capacitor_SMD:C_0805_2012Metric, F.Cu at (75.6, 108.1)
- added D6: ss34, Diode_SMD:D_SMA, F.Cu at (66.3, 104.4)
- added L4: 2.2uh, Inductor_SMD:L_0805_2012Metric, F.Cu at (73.5, 113.2)
- added L5: 10uh, Inductor_SMD:L_1210_3225Metric, F.Cu at (60.1, 98.0)
- added L6: 10uh, Inductor_SMD:L_1210_3225Metric, F.Cu at (65.2, 108.0)
- added L7: 2.2uh, Inductor_SMD:L_0805_2012Metric, F.Cu at (71.9, 95.5)
- added L8: 2.2uh, Inductor_SMD:L_0805_2012Metric, F.Cu at (72.0, 105.2)
- added Q2: s8050, Package_TO_SOT_SMD:SOT-23, F.Cu at (87.8, 99.7)
- added Q3: s8050, Package_TO_SOT_SMD:SOT-23, F.Cu at (84.1, 99.7)
- added R60: 9.53k, Resistor_SMD:R_0805_2012Metric, F.Cu at (92.8, 99.7)
- added R61: 9.53k, Resistor_SMD:R_0805_2012Metric, F.Cu at (90.7, 99.7)
- added R62: 1m, Resistor_SMD:R_0805_2012Metric, F.Cu at (73.4, 91.5)
- added R63: 9.53k, Resistor_SMD:R_0805_2012Metric, F.Cu at (80.5, 98.7)
- added R64: 9.53k, Resistor_SMD:R_0805_2012Metric, F.Cu at (80.5, 100.8)
- added R65: 104k(15v), Resistor_SMD:R_0805_2012Metric, F.Cu at (65.3, 91.4)
- added R66: 9.53k, Resistor_SMD:R_0805_2012Metric, F.Cu at (61.7, 91.4)
- added R67: 104k(15v), Resistor_SMD:R_0805_2012Metric, F.Cu at (75.7, 103.1)
- added R68: 9.53k, Resistor_SMD:R_0805_2012Metric, F.Cu at (72.0, 103.1)
- added TP1: TestPoint, TestPoint:TestPoint_Pad_1.0x1.0mm, F.Cu at (78.9, 95.5)
- added TP2: TestPoint, TestPoint:TestPoint_Pad_1.0x1.0mm, F.Cu at (88.1, 111.3)
- added TP3: TestPoint, TestPoint:TestPoint_Pad_1.0x1.0mm, F.Cu at (132.9, 87.4)
- added TP4: TestPoint, TestPoint:TestPoint_Pad_1.0x1.0mm, F.Cu at (123.4, 80.9)
- added TP5: SPDIF, TestPoint:TestPoint_Pad_1.0x1.0mm, F.Cu at (127.5, 97.3)
- added TP6: SPDIF, TestPoint:TestPoint_Pad_1.0x1.0mm, F.Cu at (116.3, 57.8)
- added U14: MP1541, Package_TO_SOT_SMD:TSOT-23-5, F.Cu at (57.2, 126.6)
- added U15: LP2992, Package_TO_SOT_SMD:TSOT-23-5, F.Cu at (130.1, 141.5)
- added U16: MP1541, Package_TO_SOT_SMD:TSOT-23-5, F.Cu at (60.2, 94.5)
- added U17: MP2451, Package_TO_SOT_SMD:TSOT-23-6, F.Cu at (60.2, 104.8)
- C12, C13, C14, R12, R13, R14: moved to F.Cu
- C15: value 100nf -> 1uf; moved to F.Cu
- C22: value 10uf -> 1uf
- C35, C36: value 2.2uf -> 4.7uf
- C37: value 2.2uf -> 10uf
- C38: value 750pF -> 22uf
- C39, C42, C48, C72, C73: value 100nf -> 10uf
- C40: value 5.1nF -> 10uf
- C41: value 220pF -> 22uf
- C43: value 4.3nF -> 10uf
- C44: value 22uf -> 10nf
- C45: value 22uf -> 10uf
- C46: value 10uf -> 10nf
- D1: value 40v 5A -> 40v 3A
- D2: value 40v 5A -> ss34
- D4: value 60v/3A -> 2a
- D5: value 60v 3A -> ss34
- J5: value Conn_ARM_JTAG_SWD_20 -> swd; footprint Connector_PinHeader_2.54mm:PinHeader_2x10_P2.54mm_Vertical -> Connector_PinHeader_2.54mm:PinHeader_1x04_P2.54mm_Vertical
- L2: value 22uh -> 3.3uh; footprint Inductor_SMD:L_6.3x6.3_H3 -> Inductor_SMD:L_1210_3225Metric
- L3: value 22uh -> 6.8uh; footprint Inductor_SMD:L_6.3x6.3_H3 -> Inductor_SMD:L_1210_3225Metric
- R36: value 49.9kOhm -> 0Ω
- R39: value 18.7kOhm -> 150k
- R40: value 160k -> 150k
- R41, R43: value 9.53k -> 0Ω
- R42: value 160k -> 0Ω
- R47: value 7.5 -> 9.53k
- R49, R58, R59: value 0Ω -> 9.53k
- R56: value 7.5k -> 9.53k
- R57: value 1k -> 43k(7v)
- U5: value AMS1117-5.0 -> LP2992; footprint Package_TO_SOT_SMD:SOT-223-3_TabPin2 -> Package_TO_SOT_SMD:TSOT-23-5
- U7: value TPA6120A2DWP -> TPA6120A2
- U8: value TPS54360DDA -> LT3045xMSE-1; footprint Package_SO:TI_SO-PowerPAD-8_ThermalVias -> Package_SO:MSOP-12-1EP_3x4mm_P0.65mm_EP1.65x2.85mm
- U9: value TPS54360DDA -> LT3094xMSE; footprint Package_SO:TI_SO-PowerPAD-8_ThermalVias -> Package_SO:MSOP-12-1EP_3x4mm_P0.65mm_EP1.65x2.85mm
- moved C44 76.5 mm to (132.5, 144.3), turned to 0 degrees
- moved C15 75.1 mm to (83.7, 84.7), turned to 270 degrees
- moved C43 73.5 mm to (126.6, 141.4), turned to 90 degrees
- moved R49 71.8 mm to (72.6, 120.2), turned to 0 degrees
- moved C45 70.0 mm to (133.5, 141.4), turned to 270 degrees
- moved R43 67.5 mm to (132.9, 138.6)
- moved R47 59.3 mm to (135.9, 116.6), turned to 270 degrees
- moved D2 50.3 mm to (67.5, 114.9), turned to 270 degrees
- moved C37 43.1 mm to (93.2, 84.7)
- moved C73 41.1 mm to (74.9, 116.6), turned to 270 degrees
- moved C36 40.7 mm to (91.2, 109.7)
- moved C35 38.7 mm to (93.3, 94.1)
- moved R42 37.7 mm to (91.8, 81.9), turned to 180 degrees
- moved R36 36.7 mm to (93.4, 106.0), turned to 90 degrees
- moved C40 32.6 mm to (91.2, 106.0), turned to 90 degrees
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Connections:
- C15 pad 1: +3V3 -> +5V
- C16 pad 1: VCC -> Net-(C16-Pad1)
- C20 pad 1: +7.5V -> Net-(C20-Pad1)
- C22 pad 1: +5V -> Net-(C22-Pad1)
- C35 pad 1: VCC -> Net-(C35-Pad1)
- C36 pad 1: VCC -> GND
- C36 pad 2: GND -> Net-(C36-Pad2)
- C37 pad 1: VCC -> +3.3VA
- C37 pad 2: -15V -> GND
- C38 pad 1: Net-(C38-Pad1) -> Net-(C20-Pad1)
- C39 pad 2: Net-(C39-Pad2) -> GND
- C40 pad 1: Net-(C40-Pad1) -> GND
- C40 pad 2: GND -> Net-(C40-Pad2)
- C41 pad 1: Net-(C41-Pad1) -> +5V
- C41 pad 2: -15V -> GND
- C42 pad 1: Net-(C42-Pad1) -> +5V
- C42 pad 2: Net-(C42-Pad2) -> GND
- C43 pad 1: Net-(C43-Pad1) -> +8V
- C43 pad 2: -15V -> GND
- C44 pad 1: +15V -> Net-(C44-Pad1)
- C45 pad 1: GND -> +5VA
- C45 pad 2: -15V -> GND
- C48 pad 1: Net-(C46-Pad1) -> Net-(C48-Pad1)
- C49 pad 1: GND -> Net-(C48-Pad1)
- C49 pad 2: Net-(C47-Pad2) -> GND
- C73 pad 1: +7.5V -> +8V
- D1 pad 1: VCC -> Net-(C16-Pad1)
- D1 pad 2: Net-(D1-Pad2) -> VCC
- D2 pad 1: VCC -> Net-(C48-Pad1)
- D2 pad 2: Net-(D1-Pad2) -> Net-(D2-Pad2)
- D4 pad 1: Net-(C39-Pad2) -> +5V
- D4 pad 2: GND -> Net-(D4-Pad2)
- D5 pad 1: Net-(C42-Pad1) -> Net-(C82-Pad1)
- D5 pad 2: -15V -> Net-(D5-Pad2)
- J2 pad 1: (no net) -> Net-(D4-Pad2)
- J3 pad 1: Net-(D1-Pad2) -> VCC
- J5 pad 1: +3V3 -> GND
- J5 pad 2: +3V3 -> /stm32/SWCLK
- J5 pad 3: /stm32/NJTRST -> /stm32/SWDIO
- J5 pad 4: GND -> /stm32/JTDO
- L1 pad 2: +7.5V -> Net-(C20-Pad1)
- L2 pad 1: +15V -> +5V
- L2 pad 2: Net-(C39-Pad2) -> Net-(C20-Pad1)
- L3 pad 1: GND -> Net-(D2-Pad2)
- L3 pad 2: Net-(C42-Pad1) -> +5V
- R20 pad 1: +7.5V -> Net-(C20-Pad1)
- R23 pad 1: +5V -> +12V
- R23 pad 2: Net-(R23-Pad2) -> Net-(C39-Pad1)
- R36 pad 1: Net-(R36-Pad1) -> -12V
- R36 pad 2: GND -> Net-(C40-Pad2)
- R39 pad 1: Net-(C41-Pad1) -> Net-(C35-Pad1)
- R39 pad 2: Net-(C43-Pad1) -> GND
- R40 pad 1: +15V -> GND
- R40 pad 2: /headphone_power/FB1 -> Net-(C36-Pad2)
- R41 pad 1: /headphone_power/FB1 -> /stm32/vdd1
- R41 pad 2: GND -> +3.3VA
- R42 pad 1: GND -> +3.3VA
- R42 pad 2: /headphone_power/FB2 -> Net-(C22-Pad1)
- R43 pad 1: /headphone_power/FB2 -> /PCM1792/vdd2
- R43 pad 2: -15V -> +5VA
- R47 pad 1: GND -> Net-(R47-Pad1)
- R47 pad 2: Net-(R46-Pad2) -> /PCM1792/vdd1
- R49 pad 1: /PCM1792/vdd2 -> Net-(R49-Pad1)
- R49 pad 2: +5V -> /dac_power_en
- R56 pad 1: GND -> Net-(R49-Pad1)
- R56 pad 2: Net-(R56-Pad2) -> GND
- R57 pad 1: Net-(R56-Pad2) -> Net-(C48-Pad1)
- R58 pad 1: +12V -> Net-(R57-Pad2)
- R58 pad 2: Net-(R46-Pad1) -> GND
- R59 pad 1: -12V -> Net-(R59-Pad1)
- R59 pad 2: Net-(R57-Pad2) -> hp_power_en
- U1 pad 10: (no net) -> hp_power_en
- U1 pad 36: /headphone_en -> /dac_power_en
- U1 pad 38: (no net) -> Net-(TP5-Pad1)
- U12 pad 14: /headphone_en -> Net-(R47-Pad1)
- U3 pad 2: VCC -> Net-(C16-Pad1)
- U5 pad 1: GND -> +5V
- U5 pad 2: Net-(R23-Pad2) -> GND
- U5 pad 3: +7.5V -> +5V
- U6 pad 54: (no net) -> Net-(TP6-Pad1)
- U8 pad 1: Net-(C39-Pad1) -> +15V
- U8 pad 2: VCC -> +15V
- U8 pad 3: (no net) -> Net-(TP1-Pad1)
- U8 pad 4: Net-(R36-Pad1) -> +15V
- U8 pad 5: /headphone_power/FB1 -> (no net)
- U8 pad 6: Net-(C38-Pad1) -> GND
- U8 pad 7: GND -> +15V
- U8 pad 8: Net-(C39-Pad2) -> Net-(C35-Pad1)
- U9 pad 1: Net-(C42-Pad2) -> -15V
- U9 pad 2: VCC -> -15V
- U9 pad 3: (no net) -> -15V
- U9 pad 4: Net-(R37-Pad1) -> (no net)
- U9 pad 5: /headphone_power/FB2 -> -15V
- U9 pad 6: Net-(C41-Pad1) -> GND
- U9 pad 7: -15V -> Net-(TP2-Pad1)
- U9 pad 8: Net-(C42-Pad1) -> Net-(C36-Pad2)
- U9 pad 9: -15V -> GND
Routing:
- net GND: track 1212.5 -> 1314.0 mm, vias 33 -> 40
- net +8V: track 0.00 -> 78.5 mm, vias 0 -> 2
- net /stm32/JTDI: track 79.1 -> 13.7 mm, vias 1 -> 0
- net /dac_power_en: track 0.00 -> 63.4 mm, vias 0 -> 2
- net /stm32/NRST: track 70.2 -> 12.0 mm, vias 2 -> 0
- net /stm32/NJTRST: track 67.0 -> 11.8 mm
- net hp_power_en: track 0.00 -> 43.8 mm, vias 0 -> 3
- net Net-(C76-Pad2): track 0.00 -> 42.3 mm
- net +15V: track 10.2 -> 50.9 mm
- net VCC: track 104.1 -> 69.7 mm
- net +3V3: track 261.7 -> 229.7 mm, vias 5 -> 4
- net /headphone_en: track 30.2 -> 0.00 mm
- net Net-(Q3-Pad3): track 0.00 -> 29.8 mm, vias 0 -> 2
- net -15V: track 54.5 -> 25.3 mm, vias 1 -> 0
- net Net-(R59-Pad1): track 0.00 -> 23.5 mm
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
Commit message: save
Parts:
- C17: value 5.1nF -> 2.7nf
- C18: value 750pF -> 10pf
- L1: value 8.2uh -> 15uh
- L6: value 10uh -> 6.8uh
- R18: value 49.9kOhm -> 10nf
- R19: value 15.4k -> 10.7k
- R20: value 75k -> 10.2k
- R21: value 9.53k -> 1.96k
- R61: value 9.53k -> 1m
- R65, R67: value 104k(15v) -> 110k(10v)
Changed lines of the file:
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@@
     (add_net "Net-(D4-Pad2)")
     (add_net "Net-(D5-Pad2)")
+    (add_net "Net-(H1-Pad1)")
+    (add_net "Net-(H2-Pad1)")
+    (add_net "Net-(H3-Pad1)")
+    (add_net "Net-(H4-Pad1)")
     (add_net "Net-(J2-Pad2)")
     (add_net "Net-(J2-Pad3)")
     (add_net "Net-(J2-Pad5)")
+    (add_net "Net-(J3-Pad3)")
     (add_net "Net-(J6-PadT)")
+    (add_net "Net-(J7-PadRN)")
     (add_net "Net-(J7-PadSN)")
+    (add_net "Net-(J7-PadTN)")
     (add_net "Net-(Q1-Pad1)")
     (add_net "Net-(Q1-Pad3)")
@@
     (add_net "Net-(TP5-Pad1)")
     (add_net "Net-(TP6-Pad1)")
+    (add_net "Net-(U1-Pad11)")
+    (add_net "Net-(U1-Pad2)")
+    (add_net "Net-(U1-Pad22)")
+    (add_net "Net-(U1-Pad26)")
+    (add_net "Net-(U1-Pad27)")
+    (add_net "Net-(U1-Pad28)")
+    (add_net "Net-(U1-Pad34)")
+    (add_net "Net-(U1-Pad37)")
+    (add_net "Net-(U1-Pad39)")
+    (add_net "Net-(U1-Pad40)")
+    (add_net "Net-(U1-Pad41)")
+    (add_net "Net-(U1-Pad57)")
+    (add_net "Net-(U1-Pad61)")
+    (add_net "Net-(U12-Pad1)")
+    (add_net "Net-(U12-Pad2)")
+    (add_net "Net-(U3-Pad3)")
+    (add_net "Net-(U6-Pad1)")
+    (add_net "Net-(U6-Pad10)")
+    (add_net "Net-(U6-Pad11)")
+    (add_net "Net-(U6-Pad12)")
+    (add_net "Net-(U6-Pad16)")
+    (add_net "Net-(U6-Pad17)")
+    (add_net "Net-(U6-Pad18)")
+    (add_net "Net-(U6-Pad19)")
+    (add_net "Net-(U6-Pad20)")
+    (add_net "Net-(U6-Pad22)")
+    (add_net "Net-(U6-Pad25)")
+    (add_net "Net-(U6-Pad26)")
+    (add_net "Net-(U6-Pad27)")
+    (add_net "Net-(U6-Pad29)")
+    (add_net "Net-(U6-Pad30)")
+    (add_net "Net-(U6-Pad32)")
+    (add_net "Net-(U6-Pad33)")
+    (add_net "Net-(U6-Pad34)")
+    (add_net "Net-(U6-Pad35)")
+    (add_net "Net-(U6-Pad36)")
+    (add_net "Net-(U6-Pad37)")
+    (add_net "Net-(U6-Pad39)")
+    (add_net "Net-(U6-Pad40)")
+    (add_net "Net-(U6-Pad41)")
+    (add_net "Net-(U6-Pad42)")
+    (add_net "Net-(U6-Pad43)")
+    (add_net "Net-(U6-Pad48)")
+    (add_net "Net-(U6-Pad49)")
+    (add_net "Net-(U6-Pad50)")
+    (add_net "Net-(U6-Pad51)")
+    (add_net "Net-(U6-Pad52)")
+    (add_net "Net-(U6-Pad53)")
+    (add_net "Net-(U6-Pad6)")
+    (add_net "Net-(U6-Pad7)")
+    (add_net "Net-(U6-Pad8)")
+    (add_net "Net-(U6-Pad9)")
+    (add_net "Net-(U8-Pad5)")
+    (add_net "Net-(U9-Pad4)")
     (add_net hp_power_en)
   )
@@
       (effects (font (size 1 1) (thickness 0.15)))
     )
-    (fp_text value 75k (at 0 1.65 180) (layer F.Fab)
+    (fp_text value 10.2k (at 0 1.65 180) (layer F.Fab)
       (effects (font (size 1 1) (thickness 0.15)))
     )
@@
       (effects (font (size 1 1) (thickness 0.15)))
     )
-    (fp_text value "104k(15v)" (at 0 1.65) (layer F.Fab)
+    (fp_text value "110k(10v)" (at 0 1.65) (layer F.Fab)
       (effects (font (size 1 1) (thickness 0.15)))
     )
@@
       (effects (font (size 1 1) (thickness 0.15)))
     )
-    (fp_text value "104k(15v)" (at 0 1.65) (layer F.Fab)
+    (fp_text value "110k(10v)" (at 0 1.65) (layer F.Fab)
       (effects (font (size 1 1) (thickness 0.15)))
     )
@@
       (effects (font (size 1 1) (thickness 0.15)))
     )
-    (fp_text value 9.53k (at 0 1.65 90) (layer F.Fab)
+    (fp_text value 1m (at 0 1.65 90) (layer F.Fab)
       (effects (font (size 1 1) (thickness 0.15)))
     )
@@
       (effects (font (size 1 1) (thickness 0.15)))
     )
-    (fp_text value 10uh (at 0 2.28) (layer F.Fab)
+    (fp_text value 6.8uh (at 0 2.28) (layer F.Fab)
       (effects (font (size 1 1) (thickness 0.15)))
     )
@@
       (effects (font (size 1 1) (thickness 0.15)))
     )
-    (fp_text value 8.2uh (at 0 4.45 90) (layer F.Fab)
+    (fp_text value 15uh (at 0 4.45 90) (layer F.Fab)
       (effects (font (size 1 1) (thickness 0.15)))
     )
@@
       (effects (font (size 1 1) (thickness 0.15)))
     )
-    (fp_text value 5.1nF (at 0 1.68 90) (layer F.Fab)
+    (fp_text value 2.7nf (at 0 1.68 90) (layer F.Fab)
       (effects (font (size 1 1) (thickness 0.15)))
     )
@@
       (effects (font (size 1 1) (thickness 0.15)))
     )
-    (fp_text value 750pF (at 0 1.65 90) (layer F.Fab)
+    (fp_text value 10pf (at 0 1.65 90) (layer F.Fab)
       (effects (font (size 1 1) (thickness 0.15)))
     )
@@
       (effects (font (size 1 1) (thickness 0.15)))
     )
-    (fp_text value 49.9kOhm (at 0 1.65 180) (layer F.Fab)
+    (fp_text value 10nf (at 0 1.65 180) (layer F.Fab)
       (effects (font (size 1 1) (thickness 0.15)))
     )
@@
       (effects (font (size 1 1) (thickness 0.15)))
     )
-    (fp_text value 15.4k (at 0 1.65 90) (layer F.Fab)
+    (fp_text value 10.7k (at 0 1.65 90) (layer F.Fab)
       (effects (font (size 1 1) (thickness 0.15)))
     )
@@
       (effects (font (size 1 1) (thickness 0.15)))
     )
-    (fp_text value 9.53k (at 0 1.65) (layer F.Fab)
+    (fp_text value 1.96k (at 0 1.65) (layer F.Fab)
       (effects (font (size 1 1) (thickness 0.15)))
     )
