File: mcu/digital-amplifier2/circuit/main/digital-amplifier2.kicad_pcb (KiCad board)
At the start: 2 copper layers, 100 x 100 mm, 197 parts, among them J1 Conn_01x10_Female, J2 USB_B, J3 Barrel_Jack_Switch, J4 encoder, J5 swd, J6 AudioJack4, J7 AudioJack3_Switch, Q1 s8550, Q2 s8050, Q3 s8050, U1 STM32F446RETx, U12 PCM1792A, U13 OPA4134, U14 MP1541, U15 LP2992, U16 MP1541, U17 MP2451, U2 DLT11H0, U3 TPS54360DDA, U4 AMS1117-3.3, U5 LP2992, U6 SJR-BTM331, U7 TPA6120A2, U8 LT3045xMSE-1, U9 LT3094xMSE, Y1 5032 8m

Commit message: v6
Parts:
- removed C77, C83, C86, C87, C89: 100nf, Capacitor_SMD:C_0805_2012Metric
- removed C82, C85: 10uf, Capacitor_SMD:C_0805_2012Metric
- removed C84, C88: 22uf, Capacitor_SMD:C_0805_2012Metric
- removed L1: 15uh, Inductor_SMD:L_6.3x6.3_H3
- removed L2: 3.3uh, Inductor_SMD:L_1210_3225Metric
- removed L3, L6: 6.8uh, Inductor_SMD:L_1210_3225Metric
- removed L4, L7, L8: 2.2uh, Inductor_SMD:L_0805_2012Metric
- removed L5: 10uh, Inductor_SMD:L_1210_3225Metric
- removed Q2, Q3: s8050, Package_TO_SOT_SMD:SOT-23
- removed R2: 0Ω, Resistor_SMD:R_0805_2012Metric
- removed R55, R56, R58, R59, R60, R63, R64, R66, R68: 9.53k, Resistor_SMD:R_0805_2012Metric
- removed R57: 43k(7v), Resistor_SMD:R_0805_2012Metric
- removed R61, R62: 1m, Resistor_SMD:R_0805_2012Metric
- removed R65, R67: 110k(10v), Resistor_SMD:R_0805_2012Metric
- removed TP3, TP4: TestPoint, TestPoint:TestPoint_Pad_1.0x1.0mm
- removed TP5, TP6: SPDIF, TestPoint:TestPoint_Pad_1.0x1.0mm
- removed U14, U16: MP1541, Package_TO_SOT_SMD:TSOT-23-5
- removed U15: LP2992, Package_TO_SOT_SMD:TSOT-23-5
- removed U17: MP2451, Package_TO_SOT_SMD:TSOT-23-6
- added C47: 10uf, Capacitor_SMD:C_0805_2012Metric, F.Cu at (112.8, 69.4)
- added C70: 10nf, Capacitor_SMD:C_0805_2012Metric, B.Cu at (112.5, 144.1)
- added C71: 10uf, Capacitor_SMD:C_0805_2012Metric, F.Cu at (125.9, 139.3)
- added D7: ss34, Diode_SMD:D_SMA, F.Cu at (63.4, 110.4)
- added D8: led2, LED_SMD:LED_0805_2012Metric, F.Cu at (112.5, 144.1)
- added R15: 80k, Resistor_SMD:R_0805_2012Metric, F.Cu at (71.3, 73.3)
- added R16: 2.37k, Resistor_SMD:R_0805_2012Metric, F.Cu at (71.3, 81.8)
- added R17: 2k, Resistor_SMD:R_0805_2012Metric, F.Cu at (71.3, 75.4)
- added R37: 9.53k, Resistor_SMD:R_0805_2012Metric, F.Cu at (57.8, 134.8)
- added R38: 9.53k, Resistor_SMD:R_0805_2012Metric, F.Cu at (135.7, 103.2)
- added R44: 9.53k, Resistor_SMD:R_0805_2012Metric, B.Cu at (104.8, 140.5)
- added R46: 9.53k, Resistor_SMD:R_0805_2012Metric, B.Cu at (112.5, 140.5)
- added SW1: sw1, Button_Switch_THT:SW_DIP_SPSTx01_Slide_6.7x4.1mm_W7.62mm_P2.54mm_LowProfile, F.Cu at (100.8, 140.0)
- added SW2: sw2, Button_Switch_THT:SW_DIP_SPSTx01_Slide_6.7x4.1mm_W7.62mm_P2.54mm_LowProfile, F.Cu at (108.6, 139.9)
- added SW3: sw3, Button_Switch_THT:SW_DIP_SPSTx01_Slide_6.7x4.1mm_W7.62mm_P2.54mm_LowProfile, F.Cu at (116.5, 139.9)
- added T1: Transformer_diy_01, misc:Transformer_diy_01, F.Cu at (64.7, 95.8)
- added U10: LP2992AIM5-5.0_NOPB, Package_TO_SOT_SMD:TSOT-23-5, F.Cu at (130.4, 140.4)
- added U11: LP2992AIM5-3.3_NOPB, Package_TO_SOT_SMD:TSOT-23-5, F.Cu at (144.8, 132.5)
- C12, C14: value 100nf -> 10uf
- C13: value 100nf -> NC
- C15: value 1uf -> 47nf
- C16: value 4.7uf -> 100nf
- C17: value 2.7nf -> NC
- C18: value 10pf -> 22uf
- C19: value 100nf -> 22uf
- C20: value 47uf -> 22uf
- C21, C37, C42: value 10uf -> 22uf
- C22: value 1uf -> 22uf
- C24, C73, C74: value 10uf -> 10nf
- C43: value 10uf -> 100nf
- C44: value 10nf -> 10uf
- C48: value 10uf -> 10nf; moved to B.Cu
- C49: value 100nf -> 10nf; moved to B.Cu
- D1: value 40v 3A -> ss34
- D3: value B560C -> ss34
- D4: value 2a -> led1; footprint Diode_SMD:D_SMA -> LED_SMD:LED_0805_2012Metric
- J1: value Conn_01x10_Female -> USB_B; footprint Connector_PinHeader_2.54mm:PinHeader_1x10_P2.54mm_Vertical -> Connector_USB:USB_B_OST_USB-B1HSxx_Horizontal
- J2: value USB_B -> Barrel_Jack_Switch; footprint Connector_USB:USB_B_OST_USB-B1HSxx_Horizontal -> connector:DC-044A_5.5-2.1
- J3: value Barrel_Jack_Switch -> AudioJack3_Switch; footprint connector:DC-044A_5.5-2.1 -> Connector_Audio:Jack_6.35mm_Neutrik_NMJ6HFD2-AU_Horizontal
- J4: value encoder -> AudioJack4; footprint Connector_PinHeader_2.54mm:PinHeader_1x04_P2.54mm_Vertical -> connector:Jack_3.5mm_4pin
- J5: value swd -> ec11; footprint Connector_PinHeader_2.54mm:PinHeader_1x04_P2.54mm_Vertical -> Connector_PinHeader_2.54mm:PinHeader_1x04_P2.54mm_Horizontal
- J6: value AudioJack4 -> ext_sai; footprint connector:Jack_3.5mm_4pin -> Connector_PinHeader_1.27mm:PinHeader_2x10_P1.27mm_Horizontal
- J7: value AudioJack3_Switch -> swd; footprint Connector_Audio:Jack_6.35mm_Neutrik_NMJ6HFD2-AU_Horizontal -> Connector_PinHeader_1.27mm:PinHeader_1x05_P1.27mm_Horizontal
- R10: value 22k -> 1.5k
- R11: value 5.1k -> 12Ω
- R12: value 9.53k -> 12Ω
- R13: value 9.53k -> 22k
- R14: value 9.53k -> 5.1k
- R18: value 10nf -> 6.1367k
- R19: value 10.7k -> 1m
- R20: value 10.2k -> 1m
- R21: value 1.96k -> 0Ω
- R24: value 0Ω -> 4.7k
- R3, R4: value 4.7k -> 9.53k
- R33: value 1m -> 4.7k
- R41, R48: value 0Ω -> 9.53k
- R42: value 0Ω -> 9.53k; moved to B.Cu
- R7: value 1.5k -> 9.53k
- R8, R9: value 12Ω -> 9.53k
- TP1: value TestPoint -> tp1
- TP2: value TestPoint -> tp2
- U2: value DLT11H0 -> LP2992AIM5-3.3_NOPB; footprint connector:spdif-DLT11H0 -> Package_TO_SOT_SMD:TSOT-23-5
- U3: value TPS54360DDA -> TPS55340; footprint Package_SO:TI_SO-PowerPAD-8_ThermalVias -> Package_SO:HTSSOP-14-1EP_4.4x5mm_P0.65mm_EP3.4x5mm_Mask3x3.1mm_ThermalVias
- U4: value AMS1117-3.3 -> LP2992AIM5-3.3_NOPB; footprint Package_TO_SOT_SMD:SOT-223-3_TabPin2 -> Package_TO_SOT_SMD:TSOT-23-5
- U5: value LP2992 -> DLT11H0; footprint Package_TO_SOT_SMD:TSOT-23-5 -> connector:spdif-DLT11H0
- moved H3 127.3 mm to (145.0, 145.0)
- moved J7 94.7 mm to (145.0, 62.0), turned to 0 degrees
- moved C74 92.0 mm to (145.5, 128.5), turned to 90 degrees
- moved H1 90.0 mm to (55.0, 55.0)
- moved H4 90.0 mm to (145.0, 55.0)
- moved C75 89.7 mm to (134.9, 139.5), turned to 0 degrees
- moved C76 87.8 mm to (143.4, 128.5), turned to 90 degrees
- moved C72 87.3 mm to (144.8, 136.5), turned to 0 degrees
- moved C45 82.3 mm to (112.8, 61.8), turned to 180 degrees
- moved D4 80.9 mm to (104.8, 144.1)
- moved J3 79.8 mm to (81.3, 131.1), turned to 270 degrees
- moved C44 73.2 mm to (97.7, 79.9), turned to 270 degrees
- moved J6 71.7 mm to (145.0, 89.0), turned to 0 degrees
- moved R7 71.5 mm to (145.7, 122.9)
- moved C43 70.2 mm to (57.8, 127.5), turned to 180 degrees
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Connections:
- net /BT_bn renamed /BT_play
- net /BT_state renamed /BT_connected
- net /BT_state2 renamed /BT_music
- C12 pad 1: /stm32/encoder_sw -> /power/vcc1
- C13 pad 1: /stm32/encoder_a -> Net-(C13-Pad1)
- C14 pad 1: /stm32/encoder_b -> +5V
- C15 pad 1: +5V -> Net-(C15-Pad1)
- C17 pad 1: Net-(C17-Pad1) -> /power/t1a
- C17 pad 2: GND -> /power/vcc1
- C18 pad 1: Net-(C18-Pad1) -> +5V
- C19 pad 1: Net-(C19-Pad1) -> +15V
- C19 pad 2: Net-(C19-Pad2) -> GND
- C2 pad 1: /stm32/vdd1 -> +3V3
- C20 pad 1: Net-(C20-Pad1) -> GND
- C20 pad 2: GND -> -15V
- C21 pad 1: +3V3 -> +7.5V
- C22 pad 1: Net-(C22-Pad1) -> +5V
- C24 pad 1: /Bluetooth/vdd_x -> Net-(C24-Pad1)
- C3 pad 1: /stm32/vdd1 -> +3V3
- C37 pad 1: +3.3VA -> +7.5V
- C38 pad 1: Net-(C20-Pad1) -> +15V
- C4 pad 1: /stm32/vdd1 -> +3V3
- C41 pad 1: +5V -> GND
- C41 pad 2: GND -> -15V
- C43 pad 1: +8V -> +7.5V
- C44 pad 1: Net-(C44-Pad1) -> +3V3
- C45 pad 1: +5VA -> +5V
- C48 pad 1: Net-(C48-Pad1) -> /ec11_sw
- C49 pad 1: Net-(C48-Pad1) -> /ec11_a
- C5 pad 1: /stm32/vdd1 -> +3V3
- C50 pad 1: /PCM1792/vdd1 -> +3.3VDAC
- C51 pad 1: /PCM1792/vdd1 -> +3.3VDAC
- C6 pad 1: /stm32/vdd1 -> +3V3
- C7 pad 1: /stm32/vdd1 -> +3V3
- C73 pad 1: +8V -> Net-(C73-Pad1)
- C74 pad 1: +5V -> Net-(C74-Pad1)
- C75 pad 1: GND -> +5VA
- C75 pad 2: +5V -> GND
- C76 pad 1: +5V -> +3.3VDAC
- C76 pad 2: Net-(C76-Pad2) -> GND
- C8 pad 1: /stm32/vdd1 -> +3V3
- C9 pad 1: /stm32/NRST -> /nrst
- D1 pad 1: Net-(C16-Pad1) -> /power/vcc1
- D1 pad 2: VCC -> VBUS
- D2 pad 1: Net-(C48-Pad1) -> /power/vcc1
- D2 pad 2: Net-(D2-Pad2) -> VCC
- D3 pad 1: Net-(C19-Pad1) -> +5V
- D3 pad 2: GND -> /power/t1a
- D4 pad 1: +5V -> GND
- D4 pad 2: Net-(D4-Pad2) -> /stm32/led1
- D5 pad 1: Net-(C82-Pad1) -> +15V
- D5 pad 2: Net-(D5-Pad2) -> /power/t2a
- D6 pad 1: Net-(C77-Pad1) -> /power/t2c
- D6 pad 2: Net-(C76-Pad2) -> -15V
- J1 pad 1: /stm32/ext_irq -> VBUS
- J1 pad 2: /stm32/ext_en -> Net-(J1-Pad2)
- J1 pad 3: /stm32/SAI1_SD_B -> Net-(J1-Pad3)
- J1 pad 4: /stm32/SAI1_FS_B -> GND
- J1 pad 5: /stm32/SAI1_SCK_B -> Net-(J1-Pad5)
- J2 pad 1: Net-(D4-Pad2) -> VCC
- J2 pad 2: Net-(J2-Pad2) -> GND
- J2 pad 3: Net-(J2-Pad3) -> (no net)
- J5 pad 1: GND -> /ec11_sw
- J5 pad 2: /stm32/SWCLK -> /ec11_a
- J5 pad 3: /stm32/SWDIO -> /ec11_b
- J5 pad 4: /stm32/JTDO -> GND
- R10 pad 1: +3V3 -> Net-(Q1-Pad3)
- R10 pad 2: /stm32/USB_CO -> Net-(J1-Pad3)
- R11 pad 1: /stm32/USB_CO -> /USB_DP
- R11 pad 2: Net-(Q1-Pad1) -> Net-(J1-Pad3)
- R12 pad 1: +3V3 -> /USB_DM
- R12 pad 2: /stm32/encoder_sw -> Net-(J1-Pad2)
- R13 pad 2: /stm32/encoder_a -> /USB_CO
- R14 pad 1: +3V3 -> /USB_CO
- R14 pad 2: /stm32/encoder_b -> Net-(Q1-Pad1)
- R18 pad 1: Net-(R18-Pad1) -> +5V
- R18 pad 2: GND -> Net-(R17-Pad1)
- R19 pad 1: Net-(C18-Pad1) -> /hp_power/on1
- R19 pad 2: Net-(C17-Pad1) -> /hp_en
- R20 pad 1: Net-(C20-Pad1) -> /hp_power/on2
- R20 pad 2: Net-(R20-Pad2) -> /hp_en
- R21 pad 1: Net-(R20-Pad2) -> Net-(R21-Pad1)
- R22 pad 1: +3V3 -> GND
- R24 pad 1: /Bluetooth/vdd_x -> +3V3
- R24 pad 2: +3V3 -> /I2C_SCL
- R3 pad 2: /SCL -> /stm32/led1
- R33 pad 1: /headphone_in -> +3V3
- R33 pad 2: Net-(J7-PadSN) -> /I2C_SDA
- R34 pad 1: /TPA6120A2/ROUT -> /ROUT
- R35 pad 1: /TPA6120A2/LOUT -> /LOUT
- R4 pad 2: /SDA -> /stm32/led2
- R41 pad 1: /stm32/vdd1 -> /jack_in
- R41 pad 2: +3.3VA -> Net-(J3-PadSN)
- R42 pad 1: +3.3VA -> +3V3
- R42 pad 2: Net-(C22-Pad1) -> /ec11_sw
- R47 pad 1: Net-(R47-Pad1) -> /hp_en
- R47 pad 2: /PCM1792/vdd1 -> GND
- R48 pad 1: /PCM1792/vdd1 -> /hp_power/on3
- R48 pad 2: +3V3 -> /hp_en
- R49 pad 1: Net-(R49-Pad1) -> /hp_power/on4
- R49 pad 2: /dac_power_en -> /hp_en
- R5 pad 1: /stm32/vdd1 -> +3V3
- R5 pad 2: /stm32/NRST -> /nrst
- R7 pad 1: Net-(Q1-Pad3) -> Net-(R7-Pad1)
- R7 pad 2: Net-(J2-Pad3) -> +3.3VDAC
- R8 pad 1: /stm32/USB_DP -> Net-(R8-Pad1)
- R8 pad 2: Net-(J2-Pad3) -> /Bluetooth/vdd_x
- R9 pad 1: /stm32/USB_DM -> /BT_en
- R9 pad 2: Net-(J2-Pad2) -> GND
- U1 pad 1: /stm32/vdd1 -> +3V3
- U1 pad 10: hp_power_en -> (no net)
- U1 pad 13: /stm32/vdd1 -> +3V3
- U1 pad 14: /stm32/encoder_sw -> /ec11_sw
- U1 pad 15: /stm32/encoder_a -> /ec11_a
- U1 pad 16: /stm32/encoder_b -> /ec11_b
- U1 pad 17: /SAI1_A_FS -> /SAI_FS_A
- U1 pad 19: /stm32/vdd1 -> +3V3
- U1 pad 20: /I2S1_FS -> /jack_in
- U1 pad 21: /I2S1_SCK -> (no net)
- U1 pad 23: /I2S1_SD -> (no net)
- U1 pad 24: /I2S1_MCK -> (no net)
- U1 pad 25: /stm32/SPDIF_RX -> /SPDIF_RX
- U1 pad 26: (no net) -> /stm32/led1
- U1 pad 27: (no net) -> /stm32/led2
- U1 pad 28: (no net) -> /SAI_SD_A
- U1 pad 29: /SAI1_A_SCK -> /SAI_SCK_A
- U1 pad 32: /stm32/vdd1 -> +3V3
- U1 pad 33: /stm32/SAI1_SCK_B -> /SAI_SCK
- U1 pad 35: /headphone_in -> (no net)
- U1 pad 36: /dac_power_en -> /hp_en
- U1 pad 38: Net-(TP5-Pad1) -> /BT_spdif
- U1 pad 40: (no net) -> /ext_irq
- U1 pad 42: /stm32/SAI1_SD_B -> /SAI_SD
- U1 pad 43: /stm32/ext_en -> /ext_en
- U1 pad 44: /stm32/USB_DM -> /USB_DM
- U1 pad 45: /stm32/USB_DP -> /USB_DP
- U1 pad 46: /stm32/SWDIO -> /swdio
- U1 pad 48: /stm32/vdd1 -> +3V3
- U1 pad 49: /stm32/SWCLK -> /swclk
- U1 pad 50: /stm32/JTDI -> (no net)
- U1 pad 51: /stm32/ext_irq -> /BT_next
- U1 pad 54: /stm32/USB_CO -> /USB_CO
- U1 pad 55: /stm32/JTDO -> /swo_tdo
- U1 pad 56: /stm32/NJTRST -> /BT_prev
- U1 pad 58: /SCL -> /I2C_SCL
- U1 pad 59: /SDA -> /I2C_SDA
- U1 pad 62: /stm32/SAI1_FS_B -> /SAI_FS
- U1 pad 64: /stm32/vdd1 -> +3V3
- U1 pad 7: /stm32/NRST -> /nrst
- U1 pad 8: /stm32/SAI1_MCK_B -> /SAI_MCK
- U1 pad 9: /SAI1_A_SD -> (no net)
- U12 pad 12: /SCL -> /I2C_SCL
- U12 pad 13: /SDA -> /I2C_SDA
- U12 pad 14: Net-(R47-Pad1) -> Net-(R7-Pad1)
- U12 pad 3: /PCM1792/vdd1 -> +3.3VDAC
- U12 pad 4: /I2S1_FS -> /SAI_SCK_A
- U12 pad 5: /I2S1_SD -> /SAI_MCK
- U12 pad 6: /I2S1_SCK -> /SAI_FS_A
- U12 pad 7: /I2S1_MCK -> /SAI_SD_A
- U12 pad 9: /PCM1792/vdd1 -> +3.3VDAC
- U2 pad 1: /stm32/SPDIF_RX -> +5V
- U2 pad 3: +3V3 -> +5V
- U3 pad 1: Net-(C19-Pad2) -> /power/SW
- U3 pad 2: Net-(C16-Pad1) -> /power/SW
- U3 pad 3: (no net) -> /power/vcc1
- U3 pad 4: Net-(R18-Pad1) -> /power/vcc1
- U3 pad 5: Net-(R20-Pad2) -> Net-(C15-Pad1)
- U3 pad 6: Net-(C18-Pad1) -> GND
- U3 pad 8: Net-(C19-Pad1) -> Net-(C13-Pad1)
- U3 pad 9: GND -> Net-(R17-Pad1)
- U4 pad 1: GND -> +5V
- U4 pad 2: Net-(R22-Pad2) -> GND
- U4 pad 3: +5V -> /BT_en
- U5 pad 1: +5V -> /SPDIF_RX
- U5 pad 3: +5V -> +3V3
- U6 pad 13: /BT_en -> Net-(R8-Pad1)
- U6 pad 25: (no net) -> /BT_next
- U6 pad 26: (no net) -> /BT_prev
- U6 pad 3: /SAI1_A_SD -> (no net)
- U6 pad 4: /SAI1_A_FS -> (no net)
- U6 pad 5: /SAI1_A_SCK -> (no net)
- U6 pad 54: Net-(TP6-Pad1) -> /BT_spdif
- U8 pad 4: +15V -> /hp_power/on1
- U8 pad 6: GND -> Net-(R21-Pad1)
- U9 pad 3: -15V -> /hp_power/on2
- U9 pad 6: GND -> Net-(R22-Pad2)
Routing:
- net /stm32/vdd1: track 150.2 -> 0.00 mm, vias 3 -> 0
- net /hp_en: track 0.00 -> 126.4 mm, vias 0 -> 5
- net /ec11_sw: track 0.00 -> 109.3 mm, vias 0 -> 1
- net +7.5V: track 0.00 -> 93.9 mm, vias 0 -> 2
- net Net-(J7-PadSN): track 93.2 -> 0.00 mm, vias 1 -> 0
- net /ec11_a: track 0.00 -> 89.0 mm, vias 0 -> 1
- net +8V: track 78.5 -> 0.00 mm, vias 2 -> 0
- net /SDA: track 75.9 -> 0.00 mm, vias 4 -> 0
- net /jack_in: track 0.00 -> 74.0 mm, vias 0 -> 2
- net /stm32/SWCLK: track 73.7 -> 0.00 mm, vias 1 -> 0
- net /ec11_b: track 0.00 -> 72.8 mm, vias 0 -> 1
- net /stm32/encoder_sw: track 72.7 -> 0.00 mm, vias 1 -> 0
- net /SCL: track 71.5 -> 0.00 mm, vias 4 -> 0
- net +3V3: track 229.7 -> 301.2 mm, vias 4 -> 15
- net /stm32/encoder_a: track 69.4 -> 0.00 mm, vias 1 -> 0
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
Commit message: digital-amplifier2_v8
Parts:
- removed C62, C64, C65: 2.7nf, Capacitor_SMD:C_0805_2012Metric
- removed C66: 10uf, Capacitor_SMD:C_0805_2012Metric
- removed D8: led2, LED_SMD:LED_0805_2012Metric
- removed H1, H2, H3, H4: m3, MountingHole:MountingHole_3.2mm_M3_Pad
- removed J5: ec11, Connector_PinHeader_2.54mm:PinHeader_1x04_P2.54mm_Horizontal
- removed J6: ext_sai, Connector_PinHeader_1.27mm:PinHeader_2x10_P1.27mm_Horizontal
- removed SW2: sw2, Button_Switch_THT:SW_DIP_SPSTx01_Slide_6.7x4.1mm_W7.62mm_P2.54mm_LowProfile
- removed SW3: sw3, Button_Switch_THT:SW_DIP_SPSTx01_Slide_6.7x4.1mm_W7.62mm_P2.54mm_LowProfile
- removed TP1: tp1, TestPoint:TestPoint_Pad_1.0x1.0mm
- removed TP2: tp2, TestPoint:TestPoint_Pad_1.0x1.0mm
- removed U13: OPA4134, Package_SO:SOIC-14_3.9x8.7mm_P1.27mm
- added C100: 100uf, Capacitor_SMD:C_1210_3225Metric, B.Cu at (133.1, 126.9)
- added C101: 100uf, Capacitor_SMD:C_1210_3225Metric, B.Cu at (120.0, 126.8)
- added C102: 100uf, Capacitor_SMD:C_1210_3225Metric, B.Cu at (107.8, 126.8)
- added C103: 100uf, Capacitor_SMD:C_1210_3225Metric, B.Cu at (123.5, 126.8)
- added C104: 4.7uf, Capacitor_SMD:C_0603_1608Metric, F.Cu at (107.9, 141.4)
- added C105: 10uf, Capacitor_SMD:C_0805_2012Metric, F.Cu at (136.8, 132.7)
- added C106: 10uf, Capacitor_SMD:C_0805_2012Metric, F.Cu at (120.6, 127.4)
- added C107: 10uf, Capacitor_SMD:C_0805_2012Metric, F.Cu at (122.7, 127.4)
- added C108: 10uf, Capacitor_SMD:C_0805_2012Metric, F.Cu at (105.7, 132.7)
- added C109: 100nf, Capacitor_SMD:C_0603_1608Metric, F.Cu at (107.9, 139.8)
- added C110: 100nf, Capacitor_SMD:C_0603_1608Metric, F.Cu at (135.0, 132.5)
- added C111: 100nf, Capacitor_SMD:C_0603_1608Metric, F.Cu at (120.6, 131.5)
- added C112: 100nf, Capacitor_SMD:C_0603_1608Metric, F.Cu at (122.2, 131.5)
- added C113: 100nf, Capacitor_SMD:C_0603_1608Metric, F.Cu at (107.6, 132.5)
- added C114: 4.7uf, Capacitor_SMD:C_0603_1608Metric, F.Cu at (122.6, 141.4)
- added C115: 100nf, Capacitor_SMD:C_0603_1608Metric, F.Cu at (122.6, 139.8)
- added C116: 1uf, Capacitor_SMD:C_0603_1608Metric, F.Cu at (117.6, 140.7)
- added C117: 1uf, Capacitor_SMD:C_0603_1608Metric, F.Cu at (111.8, 140.6)
- added C118: 1uf, Capacitor_SMD:C_0603_1608Metric, F.Cu at (132.3, 140.9)
- added C119: 1uf, Capacitor_SMD:C_0603_1608Metric, F.Cu at (126.4, 140.5)
- added C120: 220nf, Capacitor_SMD:C_0603_1608Metric, F.Cu at (110.7, 126.1)
- added C121: 220nf, Capacitor_SMD:C_0603_1608Metric, F.Cu at (113.6, 126.2)
- added C122: 220nf, Capacitor_SMD:C_0603_1608Metric, F.Cu at (118.0, 126.2)
- added C123: 220nf, Capacitor_SMD:C_0603_1608Metric, F.Cu at (115.2, 126.2)
- added C124: 220nf, Capacitor_SMD:C_0603_1608Metric, F.Cu at (125.2, 126.2)
- added C125: 220nf, Capacitor_SMD:C_0603_1608Metric, F.Cu at (128.0, 126.2)
- added C126: 220nf, Capacitor_SMD:C_0603_1608Metric, F.Cu at (132.8, 126.2)
- added C127: 220nf, Capacitor_SMD:C_0603_1608Metric, F.Cu at (129.6, 126.2)
- added C128: 680nf, Capacitor_SMD:C_0603_1608Metric, B.Cu at (114.5, 111.7)
- added C129: 680nf, Capacitor_SMD:C_0603_1608Metric, B.Cu at (122.2, 111.7)
- added C130: 680nf, Capacitor_SMD:C_0603_1608Metric, B.Cu at (118.4, 111.7)
- added C131: 680nf, Capacitor_SMD:C_0603_1608Metric, B.Cu at (126.0, 111.7)
- added C132: 10uf, Capacitor_SMD:C_0805_2012Metric, F.Cu at (186.3, 123.9)
- added C77: 22uf, Capacitor_SMD:C_0805_2012Metric, B.Cu at (165.3, 179.5)
- added C78: 22uf, Capacitor_SMD:C_0805_2012Metric, B.Cu at (165.5, 189.0)
- added C79: 4.7uf, Capacitor_SMD:C_0603_1608Metric, B.Cu at (155.0, 182.9)
- added C80: 4.7uf, Capacitor_SMD:C_0603_1608Metric, B.Cu at (154.9, 192.3)
- added C81: 22uf, Capacitor_SMD:C_0805_2012Metric, B.Cu at (156.3, 179.6)
- added C82: 22uf, Capacitor_SMD:C_0805_2012Metric, B.Cu at (156.3, 188.9)
- added C83: 22uf, Capacitor_SMD:C_0805_2012Metric, B.Cu at (154.2, 179.5)
- added C84: 22uf, Capacitor_SMD:C_0805_2012Metric, B.Cu at (154.2, 189.0)
- added C93: 10uf, Capacitor_SMD:C_0805_2012Metric, F.Cu at (152.7, 198.8)
- added C94: 10uf, Capacitor_SMD:C_0805_2012Metric, F.Cu at (154.8, 198.8)
- added C95: 1uf, Capacitor_SMD:C_0603_1608Metric, F.Cu at (140.1, 199.6)
- added C96: 1uf, Capacitor_SMD:C_0603_1608Metric, F.Cu at (137.0, 199.6)
- added C97: 10uf, Capacitor_SMD:C_0603_1608Metric, F.Cu at (132.5, 205.8)
- added C98: 100nf, Capacitor_SMD:C_0603_1608Metric, F.Cu at (142.4, 198.8)
- added C99: NC, Capacitor_SMD:C_0603_1608Metric, F.Cu at (172.1, 142.6)
- added L1: 22uh / 0630, Inductor_SMD:L_6.3x6.3_H3, F.Cu at (182.7, 130.7)
- added L10: 2.2uh / 0805, Inductor_SMD:L_0805_2012Metric, B.Cu at (177.4, 194.3)
- added L13: 10uh, Inductor_SMD:L_6.3x6.3_H3, F.Cu at (109.6, 118.4)
- added L14: 10uh, Inductor_SMD:L_6.3x6.3_H3, F.Cu at (123.9, 118.3)
- added L15: 10uh, Inductor_SMD:L_6.3x6.3_H3, F.Cu at (116.8, 118.4)
- added L16: 10uh, Inductor_SMD:L_6.3x6.3_H3, F.Cu at (131.1, 118.3)
- added L2: 22uh / 0630, Inductor_SMD:L_6.3x6.3_H3, F.Cu at (170.9, 135.1)
- added L3: 2.2uh / 0805, Inductor_SMD:L_0805_2012Metric, F.Cu at (154.3, 136.7)
- added L4: 4.7uh / 0630, Inductor_SMD:L_6.3x6.3_H3, F.Cu at (180.6, 121.0)
- added L9: 2.2uh / 0805, Inductor_SMD:L_0805_2012Metric, B.Cu at (177.4, 199.8)
- added R2: 9.53kΩ, Resistor_SMD:R_0603_1608Metric, F.Cu at (129.5, 163.2)
- added R45: 2.37k, Resistor_SMD:R_0603_1608Metric, F.Cu at (185.5, 154.0)
- added R55: 10k, Resistor_SMD:R_0603_1608Metric, B.Cu at (166.2, 212.4)
- added R57: 5.1k, Resistor_SMD:R_0805_2012Metric, F.Cu at (163.3, 111.4)
- added R58: 760k, Resistor_SMD:R_0603_1608Metric, F.Cu at (150.9, 198.8)
- added R59: 9.53k, Resistor_SMD:R_0603_1608Metric, F.Cu at (147.5, 198.8)
- added R60: 9.53k, Resistor_SMD:R_0603_1608Metric, F.Cu at (144.0, 198.8)
- added R61: 9.53k, Resistor_SMD:R_0603_1608Metric, F.Cu at (145.6, 198.8)
- added R62: 0Ω, Resistor_SMD:R_0603_1608Metric, F.Cu at (134.2, 205.8)
- added R63: 9.53k, Resistor_SMD:R_0603_1608Metric, F.Cu at (128.7, 169.6)
- added R65: 9.53k, Resistor_SMD:R_0603_1608Metric, F.Cu at (134.0, 140.8)
- added R67: 15k, Resistor_SMD:R_0603_1608Metric, F.Cu at (110.2, 140.5)
- added R68: 47k, Resistor_SMD:R_0603_1608Metric, F.Cu at (124.8, 140.5)
- added U15: tas5805m, Package_SO:HTSSOP-28-1EP_4.4x9.7mm_P0.65mm_EP3.4x9.5mm_ThermalVias, F.Cu at (114.1, 134.7)
- added U16: tas5805m, Package_SO:HTSSOP-28-1EP_4.4x9.7mm_P0.65mm_EP3.4x9.5mm_ThermalVias, F.Cu at (128.7, 134.6)
- added j1: swd_pcb_2.54, misc:swd_pcb_2.54, F.Cu at (191.9, 201.8)
- AE1: footprint RF_Antenna:Texas_SWRA117D_2.4GHz_Left -> Connector_Coaxial:SMA_Molex_73251-2200_Horizontal
- C1: footprint Capacitor_SMD:C_0805_2012Metric -> Capacitor_SMD:C_0603_1608Metric; moved to B.Cu
- C13: value NC -> 47nf; footprint Capacitor_SMD:C_0805_2012Metric -> Capacitor_SMD:C_0603_1608Metric
- C14, C27, C40, C44, C5, C52, C54: value 10uf -> 100nf; footprint Capacitor_SMD:C_0805_2012Metric -> Capacitor_SMD:C_0603_1608Metric
- C15: value 47nf -> 10uf
- C16: value 100nf -> 2.2uf; footprint Capacitor_SMD:C_0805_2012Metric -> Capacitor_SMD:C_1206_3216Metric
- C17: value NC -> 1uf
- C2: value 100nf -> 10uf; footprint Capacitor_SMD:C_0805_2012Metric -> Capacitor_SMD:C_0603_1608Metric
- C20: value 22uf -> 100nf
- C23: value 22uf -> 100uf; footprint Capacitor_SMD:C_0805_2012Metric -> Capacitor_SMD:C_1210_3225Metric; moved to B.Cu
- C24: value 10nf -> 100uf; footprint Capacitor_SMD:C_0805_2012Metric -> Capacitor_SMD:C_1210_3225Metric; moved to B.Cu
- C25: value 100uf -> 10uf; footprint Capacitor_SMD:C_1210_3225Metric -> Capacitor_SMD:C_0805_2012Metric; moved to B.Cu
- C26, C30, C31, C32, C56, D6, D7, Q1: moved to B.Cu
- C28, C3, C33, C34, C39, C4, C45, C6, C8, C9: footprint Capacitor_SMD:C_0805_2012Metric -> Capacitor_SMD:C_0603_1608Metric
- C29: value 100nf -> 100uf; footprint Capacitor_SMD:C_0805_2012Metric -> Capacitor_SMD:C_1210_3225Metric; moved to B.Cu
- C35: value 4.7uf -> 10uf; footprint Capacitor_SMD:C_0805_2012Metric -> Capacitor_SMD:C_0603_1608Metric
- C36: value 4.7uf -> 100nf; footprint Capacitor_SMD:C_0805_2012Metric -> Capacitor_SMD:C_0603_1608Metric
- C37, C38: value 22uf -> 47uf; footprint Capacitor_SMD:C_0805_2012Metric -> Capacitor_SMD:C_0603_1608Metric
- C41: value 22uf -> 10uf; footprint Capacitor_SMD:C_0805_2012Metric -> Capacitor_SMD:C_0603_1608Metric
- C42: value 22uf -> 100nf; footprint Capacitor_SMD:C_0805_2012Metric -> Capacitor_SMD:C_0603_1608Metric
- C43: value 100nf -> 10uf; footprint Capacitor_SMD:C_0805_2012Metric -> Capacitor_SMD:C_0603_1608Metric; moved to B.Cu
- C46: value 10nf -> 100nf; footprint Capacitor_SMD:C_0805_2012Metric -> Capacitor_SMD:C_0603_1608Metric; moved to B.Cu
- C47, C50: value 10uf -> 2.7nf; footprint Capacitor_SMD:C_0805_2012Metric -> Capacitor_SMD:C_0603_1608Metric
- C48, C49: value 10nf -> 2.7nf; footprint Capacitor_SMD:C_0805_2012Metric -> Capacitor_SMD:C_0603_1608Metric; moved to F.Cu
- C51, C53: value 100nf -> 10uf; moved to B.Cu
- C55, C67, C69: value 100nf -> 22uf; moved to B.Cu
- C57: value 100nf -> 10uf
- C59: value 100nf -> 47nf; footprint Capacitor_SMD:C_0805_2012Metric -> Capacitor_SMD:C_0603_1608Metric
- C60: value 47uf -> 1uf
- C61: value 47uf -> 100nf; footprint Capacitor_SMD:C_0805_2012Metric -> Capacitor_SMD:C_0603_1608Metric
- C63: value 2.7nf -> NC; footprint Capacitor_SMD:C_0805_2012Metric -> Capacitor_SMD:C_0603_1608Metric
- C68, C75, C76: value 10uf -> 22uf; moved to B.Cu
- C7: footprint Resistor_SMD:R_0805_2012Metric -> Capacitor_SMD:C_0603_1608Metric
- C70: value 10nf -> 22uf
- C71, C72: value 10uf -> 100nf
- C73, C74: value 10nf -> 22uf; moved to B.Cu
- D1: value ss34 -> led1; footprint Diode_SMD:D_SMA -> LED_SMD:LED_0805_2012Metric
- D2: value ss34 -> led2; footprint Diode_SMD:D_SMA -> LED_SMD:LED_0805_2012Metric
- D4: value led1 -> ss34; footprint LED_SMD:LED_0805_2012Metric -> Diode_SMD:D_SMA
- J1: value USB_B -> USB_C_Receptacle_USB2.0; footprint Connector_USB:USB_B_OST_USB-B1HSxx_Horizontal -> Connector_USB:USB_C_Receptacle_Palconn_UTC16-G
- J4: value AudioJack4 -> 0.96_oled; footprint connector:Jack_3.5mm_4pin -> Connector_FFC-FPC:TE_3-1734839-0_1x30-1MP_P0.5mm_Horizontal
- J7: value swd -> PW_OUT; footprint Connector_PinHeader_1.27mm:PinHeader_1x05_P1.27mm_Horizontal -> Connector_Phoenix_MC:PhoenixContact_MC_1,5_4-G-3.81_1x04_P3.81mm_Horizontal
- R1: value 9.53kΩ -> 9.53k
- R10: value 1.5k -> 1k; footprint Resistor_SMD:R_0805_2012Metric -> Resistor_SMD:R_0603_1608Metric
- R11: value 12Ω -> 5k; footprint Resistor_SMD:R_0805_2012Metric -> Resistor_SMD:R_0603_1608Metric
- R12: value 12Ω -> 1k; footprint Resistor_SMD:R_0805_2012Metric -> Resistor_SMD:R_0603_1608Metric
- R13: value 22k -> 1k; footprint Resistor_SMD:R_0805_2012Metric -> Resistor_SMD:R_0603_1608Metric
- R14: value 5.1k -> 1k; footprint Resistor_SMD:R_0805_2012Metric -> Resistor_SMD:R_0603_1608Metric
- R15: value 80k -> 1k; footprint Resistor_SMD:R_0805_2012Metric -> Resistor_SMD:R_0603_1608Metric
- R16: value 2.37k -> 1k; footprint Resistor_SMD:R_0805_2012Metric -> Resistor_SMD:R_0603_1608Metric
- R17: value 2k -> 1k; footprint Resistor_SMD:R_0805_2012Metric -> Resistor_SMD:R_0603_1608Metric
- R18: value 6.1367k -> 1k; footprint Resistor_SMD:R_0805_2012Metric -> Resistor_SMD:R_0603_1608Metric
- R19: value 1m -> 1k; footprint Resistor_SMD:R_0805_2012Metric -> Resistor_SMD:R_0603_1608Metric
- R20: value 1m -> 39.2Ω; moved to B.Cu
- R21: value 0Ω -> 39.2Ω; moved to B.Cu
- R22, R26, R27, R28, R29, R5: footprint Resistor_SMD:R_0805_2012Metric -> Resistor_SMD:R_0603_1608Metric
- R23: value 0Ω -> 9.53k; footprint Resistor_SMD:R_0805_2012Metric -> Resistor_SMD:R_0603_1608Metric
- R24: value 4.7k -> 10k; footprint Resistor_SMD:R_0805_2012Metric -> Resistor_SMD:R_0603_1608Metric
- R25: value 1k -> 0Ω; footprint Resistor_SMD:R_0805_2012Metric -> Resistor_SMD:R_0603_1608Metric
- R3: value 9.53k -> 0Ω; footprint Resistor_SMD:R_0805_2012Metric -> Resistor_SMD:R_0603_1608Metric
- R30: value 1k -> 9.53k; moved to B.Cu
- R31: value 1k -> 0; moved to B.Cu
- R32: value 1k -> 1.5k; moved to B.Cu
- R33: value 4.7k -> 12Ω; moved to B.Cu
- R34: value 39.2Ω -> 12Ω; moved to B.Cu
- R35: value 39.2Ω -> 22k; moved to B.Cu
- R36: value 0Ω -> 5.1k; moved to B.Cu
- R37, R38: value 9.53k -> 4.7k; footprint Resistor_SMD:R_0805_2012Metric -> Resistor_SMD:R_0603_1608Metric
- R39: value 150k -> 0Ω; footprint Resistor_SMD:R_0805_2012Metric -> Resistor_SMD:R_0603_1608Metric
- R40: value 150k -> 9.53k
- R42: moved to F.Cu
- R43: value 0Ω -> 43k; footprint Resistor_SMD:R_0805_2012Metric -> Resistor_SMD:R_0603_1608Metric
- R44: value 9.53k -> 10k
- R46: value 9.53k -> 0Ω; footprint Resistor_SMD:R_0805_2012Metric -> Resistor_SMD:R_0603_1608Metric; moved to F.Cu
- R47, R49: value 9.53k -> 10k; footprint Resistor_SMD:R_0805_2012Metric -> Resistor_SMD:R_0603_1608Metric; moved to B.Cu
- R48: value 9.53k -> 1k; footprint Resistor_SMD:R_0805_2012Metric -> Resistor_SMD:R_0603_1608Metric
- R50: value 10k -> 13k; footprint Resistor_SMD:R_0805_2012Metric -> Resistor_SMD:R_0603_1608Metric
- R51, R52: value 1k -> 150k; footprint Resistor_SMD:R_0805_2012Metric -> Resistor_SMD:R_0603_1608Metric; moved to B.Cu
- R53, R54: value 1k -> 0Ω; moved to B.Cu
- R7: value 9.53k -> 43k; footprint Resistor_SMD:R_0805_2012Metric -> Resistor_SMD:R_0603_1608Metric
- R8: value 9.53k -> 2.37k; footprint Resistor_SMD:R_0805_2012Metric -> Resistor_SMD:R_0603_1608Metric
- R9: value 9.53k -> 10k; moved to B.Cu
- SW1: value sw1 -> ec11; footprint Button_Switch_THT:SW_DIP_SPSTx01_Slide_6.7x4.1mm_W7.62mm_P2.54mm_LowProfile -> misc:ec11_horizontal
- T1: value Transformer_diy_01 -> Transformer_1P_2S; footprint misc:Transformer_diy_01 -> misc:Transformer_diy_02
- U10: value LP2992AIM5-5.0_NOPB -> TPS55340; footprint Package_TO_SOT_SMD:TSOT-23-5 -> Package_SO:HTSSOP-14-1EP_4.4x5mm_P0.65mm_EP3.4x5mm_Mask3x3.1mm_ThermalVias
- U11: value LP2992AIM5-3.3_NOPB -> LT3045xMSE-1; footprint Package_TO_SOT_SMD:TSOT-23-5 -> Package_SO:MSOP-12-1EP_3x4mm_P0.65mm_EP1.65x2.85mm_ThermalVias; moved to B.Cu
- U12: value PCM1792A -> LT3094xMSE; footprint Package_SO:SSOP-28_5.3x10.2mm_P0.65mm -> Package_SO:MSOP-12-1EP_3x4mm_P0.65mm_EP1.65x2.85mm_ThermalVias; moved to B.Cu
- U2: value LP2992AIM5-3.3_NOPB -> TPS55340; footprint Package_TO_SOT_SMD:TSOT-23-5 -> Package_SO:HTSSOP-14-1EP_4.4x5mm_P0.65mm_EP3.4x5mm_Mask3x3.1mm_ThermalVias
- U3: value TPS55340 -> AMS1117-3.3; footprint Package_SO:HTSSOP-14-1EP_4.4x5mm_P0.65mm_EP3.4x5mm_Mask3x3.1mm_ThermalVias -> Package_TO_SOT_SMD:SOT-223-3_TabPin2
- U4: value LP2992AIM5-3.3_NOPB -> TPA6120A2; footprint Package_TO_SOT_SMD:TSOT-23-5 -> ti:TPA6120A2DWP
- U5: value DLT11H0 -> PCM1792A; footprint connector:spdif-DLT11H0 -> Package_SO:SSOP-28_5.3x10.2mm_P0.65mm
- U6: value SJR-BTM331 -> OPA4134; footprint misc:SJR-BTM331 -> Package_SO:SOIC-14_3.9x8.7mm_P1.27mm
- U7: value TPA6120A2 -> SJR-BTM331; footprint ti:TPA6120A2DWP -> misc:SJR-BTM331; moved to B.Cu
- U8: value LT3045xMSE-1 -> DLT11H0; footprint Package_SO:MSOP-12-1EP_3x4mm_P0.65mm_EP1.65x2.85mm -> connector:spdif-DLT11H0
- U9: value LT3094xMSE -> AMS1117-5.0; footprint Package_SO:MSOP-12-1EP_3x4mm_P0.65mm_EP1.65x2.85mm -> Package_TO_SOT_SMD:SOT-223-3_TabPin2
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Connections:
- C12 pad 1: /power/vcc1 -> VCC
- C14 pad 1: +5V -> Net-(C14-Pad1)
- C16 pad 2: GND -> Net-(C16-Pad2)
- C17 pad 1: /power/t1a -> +3V3
- C17 pad 2: /power/vcc1 -> GND
- C18 pad 1: +5V -> +7.5V
- C19 pad 1: +15V -> +7.5V
- C2 pad 1: +3V3 -> /stm32/vdd1
- C20 pad 1: GND -> +7.5V
- C20 pad 2: -15V -> GND
- C21 pad 1: +7.5V -> Net-(C21-Pad1)
- C22 pad 1: +5V -> Net-(C21-Pad1)
- C23 pad 1: /Bluetooth/vdd_x -> +12V
- C24 pad 1: Net-(C24-Pad1) -> +12V
- C29 pad 1: +12V -> -12V
- C3 pad 1: +3V3 -> /stm32/vdd1
- C35 pad 1: Net-(C35-Pad1) -> +3.3VDAC
- C36 pad 1: GND -> +3.3VDAC
- C36 pad 2: Net-(C36-Pad2) -> GND
- C37 pad 1: +7.5V -> Net-(C37-Pad1)
- C37 pad 2: GND -> /PCM1792/vdd2
- C38 pad 1: +15V -> Net-(C38-Pad1)
- C38 pad 2: GND -> /PCM1792/vdd2
- C39 pad 1: Net-(C39-Pad1) -> /PCM1792/vdd2
- C4 pad 1: +3V3 -> /stm32/vdd1
- C40 pad 1: GND -> /PCM1792/vdd2
- C40 pad 2: Net-(C40-Pad2) -> GND
- C41 pad 1: GND -> /PCM1792/vdd2
- C41 pad 2: -15V -> GND
- C42 pad 1: +5V -> /PCM1792/vdd2
- C43 pad 1: +7.5V -> /PCM1792/vdd2
- C44 pad 1: +3V3 -> /PCM1792/vdd2
- C45 pad 1: +5V -> /PCM1792/vdd2
- C46 pad 1: Net-(C46-Pad1) -> /PCM1792/vdd2
- C47 pad 1: /Bluetooth/vdd_x -> /OPA4134/OUTC
- C47 pad 2: GND -> /OPA4134/INC
- C48 pad 1: /ec11_sw -> /TPA6120A2/LIN-
- C48 pad 2: GND -> /OPA4134/INB
- C49 pad 1: /ec11_a -> /TPA6120A2/LIN+
- C49 pad 2: GND -> /OPA4134/INA
- C5 pad 1: +3V3 -> /stm32/vdd1
- C50 pad 1: +3.3VDAC -> /OPA4134/OUTD
- C50 pad 2: GND -> /OPA4134/IND
- C51 pad 1: +3.3VDAC -> -12V
- C52 pad 1: /PCM1792/vdd2 -> -12V
- C53 pad 1: /PCM1792/vdd2 -> +12V
- C54 pad 1: /PCM1792/vdd2 -> +12V
- C55 pad 1: /PCM1792/vdd2 -> /Bluetooth/vdd_x
- C56 pad 1: /PCM1792/vdd2 -> /Bluetooth/vdd_x
- C57 pad 1: /PCM1792/vdd2 -> +7.5V
- C58 pad 1: /PCM1792/vdd2 -> +7.5V
- C59 pad 1: /PCM1792/vdd2 -> Net-(C59-Pad1)
- C6 pad 1: +3V3 -> /stm32/vdd1
- C60 pad 1: Net-(C60-Pad1) -> +5V
- C60 pad 2: /PCM1792/vdd2 -> GND
- C61 pad 2: /PCM1792/vdd2 -> GND
- C63 pad 1: /TPA6120A2/LIN+ -> Net-(C63-Pad1)
- C63 pad 2: /OPA4134/INA -> GND
- C67 pad 1: -12V -> Net-(C67-Pad1)
- C68 pad 1: +12V -> /hp_power/FB1
- C69 pad 1: +12V -> Net-(C67-Pad1)
- C7 pad 1: +3V3 -> /stm32/vdd1
- C70 pad 1: /ec11_b -> /hp_power/FB1
- C71 pad 1: +7.5V -> Net-(C67-Pad1)
- C72 pad 1: +5V -> /hp_power/FB1
- C73 pad 1: Net-(C73-Pad1) -> -15V
- C74 pad 1: Net-(C74-Pad1) -> +15V
- C75 pad 1: +5VA -> -15V
- C76 pad 1: +3.3VDAC -> +15V
- C8 pad 1: +3V3 -> /stm32/vdd1
- D1 pad 1: /power/vcc1 -> GND
- D1 pad 2: VBUS -> /stm32/led1
- D2 pad 1: /power/vcc1 -> GND
- D2 pad 2: VCC -> /stm32/led2
- D3 pad 1: +5V -> +7.5V
- D3 pad 2: /power/t1a -> Net-(C16-Pad1)
- D4 pad 1: GND -> /connector/vcc1
- D4 pad 2: /stm32/led1 -> Net-(D4-Pad2)
- D5 pad 1: +15V -> /connector/vcc1
- D5 pad 2: /power/t2a -> Net-(D5-Pad2)
- D6 pad 1: /power/t2c -> /hp_power/out-
- D6 pad 2: -15V -> Net-(C67-Pad1)
- D7 pad 1: +7.5V -> /hp_power/FB1
- D7 pad 2: /power/t3a -> /hp_power/out+
- H5 pad 1: VCC -> (no net)
- H6 pad 1: GND -> (no net)
- H7 pad 1: VCC -> (no net)
- H8 pad 1: GND -> (no net)
- J2 pad 1: VCC -> Net-(D5-Pad2)
- J7 pad 1: /swdio -> /out_b-
- J7 pad 2: GND -> /out_b+
- J7 pad 3: /swclk -> /out_a-
- J7 pad 4: /nrst -> /out_a+
- R1 pad 1: /stm32/BOOT -> +3V3
- R1 pad 2: GND -> /stm32/led1
- R10 pad 1: Net-(Q1-Pad3) -> Net-(R10-Pad1)
- R10 pad 2: Net-(J1-Pad3) -> GND
- R11 pad 1: /USB_DP -> +7.5V
- R11 pad 2: Net-(J1-Pad3) -> Net-(R10-Pad1)
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Routing:
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Other:
- board size 100 x 100 mm -> 94 x 120 mm

Commit message: amplifier2_v9
Parts:
- removed R51, R52: 150k, Resistor_SMD:R_0603_1608Metric
- removed R53, R54: 0Ω, Resistor_SMD:R_0805_2012Metric
- removed U12: LT3094xMSE, Package_SO:MSOP-12-1EP_3x4mm_P0.65mm_EP1.65x2.85mm_ThermalVias
- added C62: 100nf, Capacitor_SMD:C_0603_1608Metric, B.Cu at (166.4, 214.0)
- added C64: 100nf, Capacitor_SMD:C_0603_1608Metric, B.Cu at (166.4, 215.6)
- added C65: 100nf, Capacitor_SMD:C_0603_1608Metric, B.Cu at (166.4, 212.4)
- added C66: 100uf, Capacitor_SMD:C_1210_3225Metric, B.Cu at (124.8, 179.9)
- added C85: 22uf, Capacitor_SMD:C_0805_2012Metric, B.Cu at (151.6, 181.7)
- added C86: 22uf, Capacitor_SMD:C_0805_2012Metric, B.Cu at (151.6, 189.1)
- added C87: 22uf, Capacitor_SMD:C_0805_2012Metric, B.Cu at (149.4, 181.7)
- added D8: ss34, Diode_SMD:D_SMA, B.Cu at (158.4, 185.4)
- added D9: ss34, Diode_SMD:D_SMA, B.Cu at (158.3, 177.9)
- added L5: 2.2uh / 0805, Inductor_SMD:L_0805_2012Metric, B.Cu at (152.8, 186.4)
- added L6: 2.2uh / 0805, Inductor_SMD:L_0805_2012Metric, B.Cu at (152.5, 178.9)
- added R56: 9.53k, Resistor_SMD:R_0603_1608Metric, F.Cu at (105.2, 205.6)
- C71, C72: moved to B.Cu
- C77: value 22uf -> 100uf; footprint Capacitor_SMD:C_0805_2012Metric -> Capacitor_SMD:C_1210_3225Metric
- C79, C80: value 4.7uf -> 22uf; footprint Capacitor_SMD:C_0603_1608Metric -> Capacitor_SMD:C_0805_2012Metric
- C82, C83: value 22uf -> 100nf
- R20, R21: moved to F.Cu
- R40: value 9.53k -> 0; footprint Resistor_SMD:R_0805_2012Metric -> Resistor_SMD:R_0603_1608Metric
- R44: footprint Resistor_SMD:R_0805_2012Metric -> Capacitor_SMD:C_0603_1608Metric
- R9: value 10k -> 100k; footprint Resistor_SMD:R_0805_2012Metric -> Capacitor_SMD:C_0603_1608Metric
- T1: value Transformer_1P_2S -> Transformer_diy_02; footprint misc:Transformer_diy_02 -> misc:Transformer_10p_22x14
- U11: value LT3045xMSE-1 -> TL431DBZ; footprint Package_SO:MSOP-12-1EP_3x4mm_P0.65mm_EP1.65x2.85mm_ThermalVias -> Package_TO_SOT_SMD:SOT-23
- moved R44 80.4 mm to (174.0, 114.8)
- moved R9 76.9 mm to (174.0, 122.1)
- moved U11 62.8 mm to (173.0, 118.5)
- moved C77 54.2 mm to (111.2, 179.9), turned to 180 degrees
- moved C72 33.9 mm to (153.7, 174.2)
- moved L10 33.8 mm to (152.6, 171.3)
- moved C76 29.4 mm to (151.6, 174.2)
- moved C74 29.4 mm to (149.4, 174.2)
- moved C68 24.4 mm to (155.8, 174.2), turned to 270 degrees
- moved C70 21.3 mm to (158.0, 174.2), turned to 270 degrees
- moved D7 19.7 mm to (158.3, 170.6), turned to 0 degrees
- moved C67 12.4 mm to (171.0, 195.2), turned to 270 degrees
- moved L9 12.2 mm to (167.6, 192.5)
- moved C71 12.1 mm to (168.9, 195.2), turned to 270 degrees
- moved D6 11.7 mm to (178.2, 195.2), turned to 180 degrees
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Connections:
- net Net-(T1-Pad2) renamed /hp_power/sw
- C23 pad 1: +12V -> +15V
- C24 pad 1: +12V -> +15V
- C25 pad 1: +12V -> +15V
- C26 pad 1: +12V -> +15V
- C27 pad 1: +12V -> +15V
- C28 pad 1: +12V -> +15V
- C29 pad 1: -12V -> -15V
- C30 pad 1: -12V -> -15V
- C31 pad 1: -12V -> -15V
- C32 pad 1: -12V -> -15V
- C33 pad 1: -12V -> -15V
- C34 pad 1: -12V -> -15V
- C51 pad 1: -12V -> -8V
- C52 pad 1: -12V -> -8V
- C53 pad 1: +12V -> +8V
- C54 pad 1: +12V -> +8V
- C57 pad 1: +7.5V -> VCC
- C58 pad 1: +7.5V -> VCC
- C77 pad 1: +15V -> +8V
- C78 pad 1: GND -> Net-(C78-Pad1)
- C78 pad 2: -15V -> GND
- C80 pad 1: GND -> Net-(C78-Pad1)
- C80 pad 2: Net-(C80-Pad2) -> GND
- C81 pad 1: Net-(C81-Pad1) -> Net-(C79-Pad1)
- C82 pad 1: GND -> Net-(C78-Pad1)
- C82 pad 2: Net-(C82-Pad2) -> GND
- C83 pad 1: Net-(C81-Pad1) -> Net-(C79-Pad1)
- C84 pad 1: GND -> +8V
- C84 pad 2: Net-(C82-Pad2) -> GND
- D5 pad 2: Net-(D5-Pad2) -> /connector/v24
- J2 pad 1: Net-(D5-Pad2) -> /connector/v24
- R44 pad 1: +15V -> /connector/v24
- R44 pad 2: GND -> +2V5
- R9 pad 1: -15V -> /stm32/v24
- R9 pad 2: GND -> +2V5
- T1 pad 1: +7.5V -> VCC
- T1 pad 4: GND -> /hp_power/out2-
- T1 pad 5: GND -> /hp_power/out2-
- T1 pad 6: /hp_power/out+ -> GND
- U1 pad 37: (no net) -> /stm32/v24
- U10 pad 3: +7.5V -> VCC
- U11 pad 1: +15V -> +2V5
- U11 pad 2: +15V -> +2V5
- U11 pad 3: (no net) -> GND
- U4 pad 1: -12V -> -15V
- U4 pad 18: +12V -> +15V
- U4 pad 20: -12V -> -15V
- U4 pad 3: +12V -> +15V
- U5 pad 4: /SAI_SCK -> /SAI_FS
- U5 pad 5: /SAI_MCK -> /SAI_SD
- U5 pad 6: /SAI_FS -> /SAI_SCK
- U5 pad 7: /SAI_SD -> /SAI_MCK
- U6 pad 11: -12V -> -8V
- U6 pad 4: +12V -> +8V
Routing:
- net +12V: track 95.7 -> 0.00 mm, vias 3 -> 0
- net -12V: track 89.4 -> 0.00 mm, vias 5 -> 0
- net -15V: track 47.1 -> 134.2 mm, vias 0 -> 2
- net +7.5V: track 111.3 -> 41.6 mm, vias 7 -> 2
- net VCC: track 210.8 -> 278.7 mm, vias 10 -> 15
- net +8V: track 0.00 -> 60.1 mm, vias 0 -> 1
- net /stm32/v24: track 0.00 -> 48.6 mm, vias 0 -> 1
- net GND: track 1754.1 -> 1801.4 mm, vias 32 -> 29
- net -8V: track 0.00 -> 40.3 mm, vias 0 -> 1
- net /hp_power/out2-: track 0.00 -> 31.0 mm
- net /hp_power/FB1: track 78.5 -> 50.0 mm, vias 3 -> 1
- net +3V3: track 255.1 -> 281.8 mm, vias 7 -> 6
- net /hp_power/out-: track 14.6 -> 36.3 mm
- net Net-(C67-Pad1): track 29.5 -> 9.57 mm, vias 1 -> 0
- net /hp_power/out2+: track 0.00 -> 13.8 mm
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
Commit message: digital-amplifier2_v10
Parts:
- removed C105, C106, C107, C108, C58: 10uf, Capacitor_SMD:C_0805_2012Metric
- added BT1: MS621FE-FL11E, misc:MS621FE-FL11E, F.Cu at (159.9, 168.4)
- added C89: 2200uf, Capacitor_THT:CP_Radial_D13.0mm_P5.00mm, F.Cu at (176.9, 122.3)
- added D10: SD103AWS, Diode_SMD:D_SOD-323, B.Cu at (156.3, 167.3)
- added R51: 1k, Resistor_SMD:R_0805_2012Metric, B.Cu at (155.9, 170.6)
- C100, C101, C102, C103, C23, C24, C29, C30: value 100uf -> 47uf; moved to F.Cu
- C12, C13, C132, C14, C16, C18, C19, C20, C21, C57, C59, C61, C63, C97, C99, D3, D4, D5, L1, L2, L3, L4, R10, R11, R20, R21, R41, R42, R43, R45, R48, R59, R60, R61, R62, R7, R8, U10, U2: moved to B.Cu
- C25, C26, C31, C32: moved to F.Cu
- C66, C77: value 100uf -> 47uf
- C75, C76: value 22uf -> 220uf; footprint Capacitor_SMD:C_0805_2012Metric -> Capacitor_THT:CP_Radial_D6.3mm_P2.50mm; moved to F.Cu
- R40: value 0 -> 10k; moved to B.Cu
- R50: value 13k -> 11k; moved to B.Cu
- R56: value 9.53k -> 10k; moved to B.Cu
- R9: value 100k -> 10k
- moved C64 55.1 mm to (159.1, 161.0)
- moved C62 51.9 mm to (159.1, 162.7)
- moved C9 49.3 mm to (154.2, 167.0), turned to 270 degrees
- moved C65 48.6 mm to (159.1, 164.4)
- moved C23 37.8 mm to (107.5, 181.6)
- moved j1 34.0 mm to (191.4, 167.7)
- moved C26 32.2 mm to (110.8, 181.1)
- moved R16 30.1 mm to (112.9, 184.7), turned to 270 degrees
- moved L1 29.8 mm to (172.0, 158.4), turned to 90 degrees
- moved C30 29.4 mm to (107.6, 175.2), turned to 90 degrees
- moved C31 28.4 mm to (110.9, 175.8), turned to 90 degrees
- moved Q1 28.4 mm to (164.3, 146.9)
- moved R35 28.4 mm to (163.2, 150.7)
- moved R36 28.4 mm to (165.5, 150.6)
- moved C33 28.1 mm to (113.0, 176.0), turned to 90 degrees
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Connections:
- C75 pad 1: -15V -> +15V
- C76 pad 1: +15V -> GND
- C76 pad 2: GND -> -15V
- C8 pad 1: /stm32/vdd1 -> /stm32/vbat
- R67 pad 1: Net-(R67-Pad1) -> /adr1
- R68 pad 1: Net-(R68-Pad1) -> /adr2
- U1 pad 1: /stm32/vdd1 -> /stm32/vbat
- U1 pad 34: (no net) -> /adr2
- U1 pad 35: (no net) -> /adr1
- U15 pad 3: Net-(R67-Pad1) -> /adr1
- U16 pad 3: Net-(R68-Pad1) -> /adr2
Routing:
- net GND: track 1801.4 -> 1651.4 mm, vias 29 -> 27
- net /adr1: track 0.00 -> 57.7 mm, vias 0 -> 2
- net +15V: track 54.5 -> 104.5 mm, vias 4 -> 2
- net /swdio: track 89.1 -> 47.5 mm, vias 0 -> 1
- net /swclk: track 87.9 -> 50.9 mm, vias 0 -> 1
- net +3V3: track 281.8 -> 316.5 mm, vias 6 -> 7
- net /adr2: track 0.00 -> 34.4 mm, vias 0 -> 2
- net /USB_DM: track 54.2 -> 20.6 mm, vias 1 -> 2
- net /swo_tdo: track 91.4 -> 58.1 mm, vias 2 -> 1
- net /hp_en: track 63.0 -> 95.2 mm
- net /stm32/vbat: track 0.00 -> 31.8 mm, vias 0 -> 1
- net /USB_DP: track 53.8 -> 22.4 mm, vias 1 -> 2
- net /USB_EN: track 58.0 -> 26.7 mm
- net Net-(J1-PadA7): track 13.3 -> 44.4 mm, vias 2 -> 1
- net /nrst: track 92.1 -> 61.1 mm, vias 3 -> 2
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- added copper zone on In1.Cu, net GND
- added copper zone on In2.Cu, net GND
Other:
- copper layers 2 -> 4

Commit message: digital-amplifier2_v10
Parts:
- moved U8 0.20 mm to (143.0, 107.7)
Routing:
- net VCC: track 253.6 -> 285.8 mm
- net GND: track 1651.4 -> 1675.6 mm
- net /hp_power/out-: track 37.3 -> 35.8 mm
- net /hp_power/FB1: track 48.2 -> 49.3 mm
- net /nrst: track 61.1 -> 60.4 mm
- net /swo_tdo: track 58.1 -> 57.6 mm
