File: mcu/digital-amplifier2/circuit/main/power±15v.sch (KiCad schematic (older format))
At the start: 32 parts, among them Q2 s8050, Q3 s8050, U16 MP1541, U17 MP2451

Commit message: save
Parts:
- L6: value 10uh -> 6.8uh
- R61: value 9.53k -> 1m
- R65, R67: value 104k(15v) -> 110k(10v)
Changed lines of the file:
@@
 P 5450 4600
 F 0 "L6" V 5225 4625 50  0000 C CNN
-F 1 "10uh" V 5325 4625 50  0000 C CNN
+F 1 "6.8uh" V 5325 4625 50  0000 C CNN
 F 2 "Inductor_SMD:L_1210_3225Metric" H 5450 4600 50  0001 C CNN
 F 3 "~" H 5450 4600 50  0001 C CNN
@@
 P 4425 1550
 F 0 "R65" H 4500 1600 50  0000 L CNN
-F 1 "104k(15v)" H 4500 1550 50  0000 L CNN
+F 1 "110k(10v)" H 4500 1550 50  0000 L CNN
 F 2 "Resistor_SMD:R_0805_2012Metric" H 4425 1550 50  0001 C CNN
 F 3 "~" H 4425 1550 50  0001 C CNN
@@
 P 5925 4900
 F 0 "R67" H 6025 4950 50  0000 L CNN
-F 1 "104k(15v)" H 6025 4900 50  0000 L CNN
+F 1 "110k(10v)" H 6025 4900 50  0000 L CNN
 F 2 "Resistor_SMD:R_0805_2012Metric" H 5925 4900 50  0001 C CNN
 F 3 "~" H 5925 4900 50  0001 C CNN
@@
 P 2775 6250
 F 0 "R61" V 2525 6250 50  0000 C CNN
-F 1 "9.53k" V 2625 6250 50  0000 C CNN
+F 1 "1m" V 2625 6250 50  0000 C CNN
 F 2 "Resistor_SMD:R_0805_2012Metric" H 2775 6250 50  0001 C CNN
 F 3 "~" H 2775 6250 50  0001 C CNN
