File: mcu/digital-amplifier2/circuit/main/OPA4134.sch (KiCad schematic (older format))
At the start: 13 parts, among them U13 OPA4134

Commit message: digital-amplifier2_v8
Parts:
- C47: renamed from C62; footprint Capacitor_SMD:C_0805_2012Metric -> Capacitor_SMD:C_0603_1608Metric
- C48: renamed from C63; footprint Capacitor_SMD:C_0805_2012Metric -> Capacitor_SMD:C_0603_1608Metric
- C49: renamed from C64; footprint Capacitor_SMD:C_0805_2012Metric -> Capacitor_SMD:C_0603_1608Metric
- C50: renamed from C65; footprint Capacitor_SMD:C_0805_2012Metric -> Capacitor_SMD:C_0603_1608Metric
- C52: renamed from C67; footprint Capacitor_SMD:C_0805_2012Metric -> Capacitor_SMD:C_0603_1608Metric
- C54: renamed from C69; footprint Capacitor_SMD:C_0805_2012Metric -> Capacitor_SMD:C_0603_1608Metric
- R26: renamed from R51; footprint Resistor_SMD:R_0805_2012Metric -> Resistor_SMD:R_0603_1608Metric
- R27: renamed from R52; footprint Resistor_SMD:R_0805_2012Metric -> Resistor_SMD:R_0603_1608Metric
- R28: renamed from R53; footprint Resistor_SMD:R_0805_2012Metric -> Resistor_SMD:R_0603_1608Metric
- R29: renamed from R54; footprint Resistor_SMD:R_0805_2012Metric -> Resistor_SMD:R_0603_1608Metric
- renumbered C66 to C51, C68 to C53, U13 to U6
Connections:
- net INA: now also C49.2, R28.2, U6.2 (-); no longer C48.2, R27.2, U6.6 (-)
- net INB: now also C48.2, R27.2, U6.6 (-); no longer C49.2, R28.2, U6.2 (-)
- net OUTA: now also C49.1, R28.1, U6.1; no longer C48.1, R27.1, U6.7
- net OUTB: now also C48.1, R27.1, U6.7; no longer C49.1, R28.1, U6.1
Changed lines of the file:
@@
 $Descr A4 11693 8268
 encoding utf-8
-Sheet 10 9
+Sheet 6 12
 Title ""
 Date ""
@@
 $EndDescr
 $Comp
-L Amplifier_Operational:OPA4134 U13
+L Amplifier_Operational:OPA4134 U6
 U 1 1 607A847E
 P 5450 1300
-F 0 "U13" H 5475 1725 50  0000 C CNN
+F 0 "U6" H 5475 1725 50  0000 C CNN
 F 1 "OPA4134" H 5475 1625 50  0000 C CNN
 F 2 "Package_SO:SOIC-14_3.9x8.7mm_P1.27mm" H 5400 1400 50  0001 C CNN
@@
 $EndComp
 $Comp
-L Amplifier_Operational:OPA4134 U13
+L Amplifier_Operational:OPA4134 U6
 U 2 1 607A919E
 P 2075 1375
-F 0 "U13" H 2100 1800 50  0000 C CNN
+F 0 "U6" H 2100 1800 50  0000 C CNN
 F 1 "OPA4134" H 2100 1700 50  0000 C CNN
 F 2 "Package_SO:SOIC-14_3.9x8.7mm_P1.27mm" H 2025 1475 50  0001 C CNN
@@
 $EndComp
 $Comp
-L Amplifier_Operational:OPA4134 U13
+L Amplifier_Operational:OPA4134 U6
 U 3 1 607A9D8C
 P 2050 4400
-F 0 "U13" H 2050 4800 50  0000 C CNN
+F 0 "U6" H 2050 4800 50  0000 C CNN
 F 1 "OPA4134" H 2050 4700 50  0000 C CNN
 F 2 "Package_SO:SOIC-14_3.9x8.7mm_P1.27mm" H 2000 4500 50  0001 C CNN
@@
 $EndComp
 $Comp
-L Amplifier_Operational:OPA4134 U13
+L Amplifier_Operational:OPA4134 U6
 U 4 1 607AAA4B
 P 5550 4400
-F 0 "U13" H 5550 4825 50  0000 C CNN
+F 0 "U6" H 5550 4825 50  0000 C CNN
 F 1 "OPA4134" H 5550 4725 50  0000 C CNN
 F 2 "Package_SO:SOIC-14_3.9x8.7mm_P1.27mm" H 5500 4500 50  0001 C CNN
@@
 $EndComp
 $Comp
-L Amplifier_Operational:OPA4134 U13
+L Amplifier_Operational:OPA4134 U6
 U 5 1 607ABD0C
 P 9700 1750
-F 0 "U13" V 9350 1750 50  0000 C CNN
+F 0 "U6" V 9350 1750 50  0000 C CNN
 F 1 "OPA4134" V 9450 1750 50  0000 C CNN
 F 2 "Package_SO:SOIC-14_3.9x8.7mm_P1.27mm" H 9650 1850 50  0001 C CNN
@@
 $EndComp
 $Comp
-L power:GND #PWR075
+L power:GND #PWR042
 U 1 1 607B9C16
 P 1500 2575
-F 0 "#PWR075" H 1500 2325 50  0001 C CNN
+F 0 "#PWR042" H 1500 2325 50  0001 C CNN
 F 1 "GND" H 1525 2375 50  0000 C CNN
 F 2 "" H 1500 2575 50  0001 C CNN
@@
 Wire Wire Line
 	1775 1475 1700 1475
-Text HLabel 1175 1475 0    50   Input ~ 0
+Text HLabel 4550 1400 0    50   Input ~ 0
 INA
 Wire Wire Line
 	2375 1375 2450 1375
-Text HLabel 2925 1375 2    50   Output ~ 0
+Text HLabel 6300 1300 2    50   Output ~ 0
 OUTA
 $Comp
-L Device:C_Small C63
+L Device:C_Small C48
 U 1 1 607BE947
 P 2025 1925
-F 0 "C63" V 1750 1950 50  0000 C CNN
+F 0 "C48" V 1750 1950 50  0000 C CNN
 F 1 "2.7nf" V 1850 1950 50  0000 C CNN
-F 2 "Capacitor_SMD:C_0805_2012Metric" H 2025 1925 50  0001 C CNN
+F 2 "Capacitor_SMD:C_0603_1608Metric" H 2025 1925 50  0001 C CNN
 F 3 "~" H 2025 1925 50  0001 C CNN
 	1    2025 1925
@@
 $EndComp
 $Comp
-L Device:R_Small R52
+L Device:R_Small R27
 U 1 1 607BF810
 P 2025 2350
-F 0 "R52" V 1775 2375 50  0000 C CNN
+F 0 "R27" V 1775 2375 50  0000 C CNN
 F 1 "1k" V 1875 2375 50  0000 C CNN
-F 2 "Resistor_SMD:R_0805_2012Metric" H 2025 2350 50  0001 C CNN
+F 2 "Resistor_SMD:R_0603_1608Metric" H 2025 2350 50  0001 C CNN
 F 3 "~" H 2025 2350 50  0001 C CNN
 	1    2025 2350
@@
 	1500 1275 1500 2575
 $Comp
-L Device:C_Small C68
+L Device:C_Small C53
 U 1 1 607CA79E
 P 10000 1875
-F 0 "C68" H 10100 1925 50  0000 L CNN
+F 0 "C53" H 10100 1925 50  0000 L CNN
 F 1 "10uf" H 10100 1875 50  0000 L CNN
 F 2 "Capacitor_SMD:C_0805_2012Metric" H 10000 1875 50  0001 C CNN
@@
 $EndComp
 $Comp
-L Device:C_Small C69
+L Device:C_Small C54
 U 1 1 607CAA70
 P 10400 1875
-F 0 "C69" H 10500 1925 50  0000 L CNN
+F 0 "C54" H 10500 1925 50  0000 L CNN
 F 1 "100nf" H 10500 1875 50  0000 L CNN
-F 2 "Capacitor_SMD:C_0805_2012Metric" H 10400 1875 50  0001 C CNN
+F 2 "Capacitor_SMD:C_0603_1608Metric" H 10400 1875 50  0001 C CNN
 F 3 "~" H 10400 1875 50  0001 C CNN
 	1    10400 1875
@@
 $EndComp
 $Comp
-L Device:C_Small C66
+L Device:C_Small C51
 U 1 1 607CAFDB
 P 8975 1875
-F 0 "C66" H 9100 1950 50  0000 L CNN
+F 0 "C51" H 9100 1950 50  0000 L CNN
 F 1 "10uf" H 9100 1850 50  0000 L CNN
 F 2 "Capacitor_SMD:C_0805_2012Metric" H 8975 1875 50  0001 C CNN
@@
 $EndComp
 $Comp
-L Device:C_Small C67
+L Device:C_Small C52
 U 1 1 607CB5DB
 P 9400 1875
-F 0 "C67" H 9525 1925 50  0000 L CNN
+F 0 "C52" H 9525 1925 50  0000 L CNN
 F 1 "100nf" H 9525 1875 50  0000 L CNN
-F 2 "Capacitor_SMD:C_0805_2012Metric" H 9400 1875 50  0001 C CNN
+F 2 "Capacitor_SMD:C_0603_1608Metric" H 9400 1875 50  0001 C CNN
 F 3 "~" H 9400 1875 50  0001 C CNN
 	1    9400 1875
@@
 	9725 2100 10000 2100
 $Comp
-L power:GND #PWR079
+L power:GND #PWR046
 U 1 1 607D789F
 P 9725 2275
-F 0 "#PWR079" H 9725 2025 50  0001 C CNN
+F 0 "#PWR046" H 9725 2025 50  0001 C CNN
 F 1 "GND" H 9775 2075 50  0000 C CNN
 F 2 "" H 9725 2275 50  0001 C CNN
@@
 $EndComp
 $Comp
-L power:GND #PWR074
+L power:GND #PWR041
 U 1 1 607E3273
 P 1475 5600
-F 0 "#PWR074" H 1475 5350 50  0001 C CNN
+F 0 "#PWR041" H 1475 5350 50  0001 C CNN
 F 1 "GND" H 1500 5400 50  0000 C CNN
 F 2 "" H 1475 5600 50  0001 C CNN
@@
 OUTC
 $Comp
-L Device:C_Small C62
+L Device:C_Small C47
 U 1 1 607E327D
 P 2000 4950
-F 0 "C62" V 1725 4975 50  0000 C CNN
+F 0 "C47" V 1725 4975 50  0000 C CNN
 F 1 "2.7nf" V 1825 4975 50  0000 C CNN
-F 2 "Capacitor_SMD:C_0805_2012Metric" H 2000 4950 50  0001 C CNN
+F 2 "Capacitor_SMD:C_0603_1608Metric" H 2000 4950 50  0001 C CNN
 F 3 "~" H 2000 4950 50  0001 C CNN
 	1    2000 4950
@@
 $EndComp
 $Comp
-L Device:R_Small R51
+L Device:R_Small R26
 U 1 1 607E3283
 P 2000 5375
-F 0 "R51" V 1750 5400 50  0000 C CNN
+F 0 "R26" V 1750 5400 50  0000 C CNN
 F 1 "1k" V 1850 5400 50  0000 C CNN
-F 2 "Resistor_SMD:R_0805_2012Metric" H 2000 5375 50  0001 C CNN
+F 2 "Resistor_SMD:R_0603_1608Metric" H 2000 5375 50  0001 C CNN
 F 3 "~" H 2000 5375 50  0001 C CNN
 	1    2000 5375
@@
 	1475 4300 1475 5600
 $Comp
-L power:GND #PWR076
+L power:GND #PWR043
 U 1 1 607E6017
 P 4875 2500
-F 0 "#PWR076" H 4875 2250 50  0001 C CNN
+F 0 "#PWR043" H 4875 2250 50  0001 C CNN
 F 1 "GND" H 4900 2300 50  0000 C CNN
 F 2 "" H 4875 2500 50  0001 C CNN
@@
 Wire Wire Line
 	5150 1400 5075 1400
-Text HLabel 4550 1400 0    50   Input ~ 0
+Text HLabel 1175 1475 0    50   Input ~ 0
 INB
 Wire Wire Line
 	5750 1300 5825 1300
-Text HLabel 6300 1300 2    50   Output ~ 0
+Text HLabel 2925 1375 2    50   Output ~ 0
 OUTB
 $Comp
-L Device:C_Small C64
+L Device:C_Small C49
 U 1 1 607E6021
 P 5400 1850
-F 0 "C64" V 5125 1875 50  0000 C CNN
+F 0 "C49" V 5125 1875 50  0000 C CNN
 F 1 "2.7nf" V 5225 1875 50  0000 C CNN
-F 2 "Capacitor_SMD:C_0805_2012Metric" H 5400 1850 50  0001 C CNN
+F 2 "Capacitor_SMD:C_0603_1608Metric" H 5400 1850 50  0001 C CNN
 F 3 "~" H 5400 1850 50  0001 C CNN
 	1    5400 1850
@@
 $EndComp
 $Comp
-L Device:R_Small R53
+L Device:R_Small R28
 U 1 1 607E6027
 P 5400 2275
-F 0 "R53" V 5150 2300 50  0000 C CNN
+F 0 "R28" V 5150 2300 50  0000 C CNN
 F 1 "1k" V 5250 2300 50  0000 C CNN
-F 2 "Resistor_SMD:R_0805_2012Metric" H 5400 2275 50  0001 C CNN
+F 2 "Resistor_SMD:R_0603_1608Metric" H 5400 2275 50  0001 C CNN
 F 3 "~" H 5400 2275 50  0001 C CNN
 	1    5400 2275
@@
 	4875 1200 4875 2500
 $Comp
-L power:GND #PWR077
+L power:GND #PWR044
 U 1 1 607EA69C
 P 4975 5600
-F 0 "#PWR077" H 4975 5350 50  0001 C CNN
+F 0 "#PWR044" H 4975 5350 50  0001 C CNN
 F 1 "GND" H 5000 5400 50  0000 C CNN
 F 2 "" H 4975 5600 50  0001 C CNN
@@
 OUTD
 $Comp
-L Device:C_Small C65
+L Device:C_Small C50
 U 1 1 607EA6A6
 P 5500 4950
-F 0 "C65" V 5225 4975 50  0000 C CNN
+F 0 "C50" V 5225 4975 50  0000 C CNN
 F 1 "2.7nf" V 5325 4975 50  0000 C CNN
-F 2 "Capacitor_SMD:C_0805_2012Metric" H 5500 4950 50  0001 C CNN
+F 2 "Capacitor_SMD:C_0603_1608Metric" H 5500 4950 50  0001 C CNN
 F 3 "~" H 5500 4950 50  0001 C CNN
 	1    5500 4950
@@
 $EndComp
 $Comp
-L Device:R_Small R54
+L Device:R_Small R29
 U 1 1 607EA6AC
 P 5500 5375
-F 0 "R54" V 5250 5400 50  0000 C CNN
+F 0 "R29" V 5250 5400 50  0000 C CNN
 F 1 "1k" V 5350 5400 50  0000 C CNN
-F 2 "Resistor_SMD:R_0805_2012Metric" H 5500 5375 50  0001 C CNN
+F 2 "Resistor_SMD:R_0603_1608Metric" H 5500 5375 50  0001 C CNN
 F 3 "~" H 5500 5375 50  0001 C CNN
 	1    5500 5375
@@
 	10400 1325 10400 1650
 $Comp
-L power:+12V #PWR080
+L power:+12V #PWR047
 U 1 1 60816499
 P 10400 1325
-F 0 "#PWR080" H 10400 1175 50  0001 C CNN
+F 0 "#PWR047" H 10400 1175 50  0001 C CNN
 F 1 "+12V" H 10425 1550 50  0000 C CNN
 F 2 "" H 10400 1325 50  0001 C CNN
@@
 $EndComp
 $Comp
-L power:-12V #PWR078
+L power:-12V #PWR045
 U 1 1 60817906
 P 8975 1325
-F 0 "#PWR078" H 8975 1425 50  0001 C CNN
+F 0 "#PWR045" H 8975 1425 50  0001 C CNN
 F 1 "-12V" H 9000 1550 50  0000 C CNN
 F 2 "" H 8975 1325 50  0001 C CNN

Commit message: amplifier2_v9
Parts:
- added C66, C77: 100uf, Capacitor_SMD:C_1210_3225Metric, symbol Device:C_Small
Connections:
- net GND: now also C66.2, C77.2
- net +12V renamed +8V
- net +8V: now also C77.1
- net -12V renamed -8V
- net -8V: now also C66.1
Changed lines of the file:
@@
 $Descr A4 11693 8268
 encoding utf-8
-Sheet 6 12
+Sheet 6 11
 Title ""
 Date ""
@@
 Wire Wire Line
 	10400 1325 10400 1650
-$Comp
-L power:+12V #PWR047
-U 1 1 60816499
+Connection ~ 8975 1650
+Connection ~ 10400 1650
+$Comp
+L power:-8V #PWR034
+U 1 1 60F53518
+P 8975 1325
+F 0 "#PWR034" H 8975 1425 50  0001 C CNN
+F 1 "-8V" H 9000 1525 50  0000 C CNN
+F 2 "" H 8975 1325 50  0001 C CNN
+F 3 "" H 8975 1325 50  0001 C CNN
+	1    8975 1325
+	1    0    0    -1
+$EndComp
+$Comp
+L power:+8V #PWR039
+U 1 1 60F53D2B
 P 10400 1325
-F 0 "#PWR047" H 10400 1175 50  0001 C CNN
-F 1 "+12V" H 10425 1550 50  0000 C CNN
+F 0 "#PWR039" H 10400 1175 50  0001 C CNN
+F 1 "+8V" H 10450 1525 50  0000 C CNN
 F 2 "" H 10400 1325 50  0001 C CNN
 F 3 "" H 10400 1325 50  0001 C CNN
@@
 $EndComp
 $Comp
-L power:-12V #PWR045
-U 1 1 60817906
-P 8975 1325
-F 0 "#PWR045" H 8975 1425 50  0001 C CNN
-F 1 "-12V" H 9000 1550 50  0000 C CNN
-F 2 "" H 8975 1325 50  0001 C CNN
-F 3 "" H 8975 1325 50  0001 C CNN
-	1    8975 1325
-	1    0    0    -1
-$EndComp
-Connection ~ 8975 1650
-Connection ~ 10400 1650
+L Device:C_Small C66
+U 1 1 60F5CA75
+P 8550 1875
+F 0 "C66" H 8650 1950 50  0000 L CNN
+F 1 "100uf" H 8650 1850 50  0000 L CNN
+F 2 "Capacitor_SMD:C_1210_3225Metric" H 8550 1875 50  0001 C CNN
+F 3 "~" H 8550 1875 50  0001 C CNN
+	1    8550 1875
+	1    0    0    -1
+$EndComp
+Wire Wire Line
+	8550 1975 8550 2100
+Wire Wire Line
+	8550 2100 8975 2100
+Connection ~ 8975 2100
+Wire Wire Line
+	8550 1775 8550 1650
+Wire Wire Line
+	8550 1650 8975 1650
+$Comp
+L Device:C_Small C77
+U 1 1 60F63892
+P 10850 1875
+F 0 "C77" H 10950 1950 50  0000 L CNN
+F 1 "100uf" H 10950 1850 50  0000 L CNN
+F 2 "Capacitor_SMD:C_1210_3225Metric" H 10850 1875 50  0001 C CNN
+F 3 "~" H 10850 1875 50  0001 C CNN
+	1    10850 1875
+	1    0    0    -1
+$EndComp
+Wire Wire Line
+	10850 1975 10850 2100
+Wire Wire Line
+	10850 2100 10400 2100
+Connection ~ 10400 2100
+Wire Wire Line
+	10850 1775 10850 1650
+Wire Wire Line
+	10850 1650 10400 1650
 $EndSCHEMATC

Commit message: digital-amplifier2_v10
Parts:
- C66, C77: value 100uf -> 47uf
Changed lines of the file:
@@
 P 8550 1875
 F 0 "C66" H 8650 1950 50  0000 L CNN
-F 1 "100uf" H 8650 1850 50  0000 L CNN
+F 1 "47uf" H 8650 1850 50  0000 L CNN
 F 2 "Capacitor_SMD:C_1210_3225Metric" H 8550 1875 50  0001 C CNN
 F 3 "~" H 8550 1875 50  0001 C CNN
@@
 P 10850 1875
 F 0 "C77" H 10950 1950 50  0000 L CNN
-F 1 "100uf" H 10950 1850 50  0000 L CNN
+F 1 "47uf" H 10950 1850 50  0000 L CNN
 F 2 "Capacitor_SMD:C_1210_3225Metric" H 10850 1875 50  0001 C CNN
 F 3 "~" H 10850 1875 50  0001 C CNN
