File: mcu/digital-amplifier2/circuit/main/connector.sch (KiCad schematic (older format))
At the start: 36 parts, among them J1 USB_B, J3 AudioJack3_Switch, J3 Barrel_Jack_Switch, J4 AudioJack4, J5 ec11, J6 ext_sai, J7 swd, Q1 s8550, SW1 sw1, SW2 sw2, SW3 sw3, U2 DLT11H0

Commit message: digital-amplifier2_v8
Parts:
- removed C48, C49, C70: 10nf, Capacitor_SMD:C_0805_2012Metric, symbol Device:C_Small
- removed H5, H6, H7, H8: m3, MountingHole:MountingHole_3.2mm_M3_Pad, symbol Mechanical:MountingHole_Pad
- removed J1: USB_B, Connector_USB:USB_B_OST_USB-B1HSxx_Horizontal, symbol Connector:USB_B
- removed J4: AudioJack4, connector:Jack_3.5mm_4pin, symbol Connector:AudioJack4
- removed J5: ec11, Connector_PinHeader_2.54mm:PinHeader_1x04_P2.54mm_Horizontal, symbol Connector:Conn_01x04_Female
- removed J6: ext_sai, Connector_PinHeader_1.27mm:PinHeader_2x10_P1.27mm_Horizontal, symbol Connector_Generic:Conn_02x10_Odd_Even
- removed J7: swd, Connector_PinHeader_1.27mm:PinHeader_1x05_P1.27mm_Horizontal, symbol Connector:Conn_01x05_Female
- removed R24, R33: 4.7k, Resistor_SMD:R_0805_2012Metric, symbol Device:R_Small
- removed R37, R38, R42, R44, R46: 9.53k, Resistor_SMD:R_0805_2012Metric, symbol Device:R_Small
- removed SW1: sw1, Button_Switch_THT:SW_DIP_SPSTx01_Slide_6.7x4.1mm_W7.62mm_P2.54mm_LowProfile, symbol Switch:SW_DIP_x01
- removed SW2: sw2, Button_Switch_THT:SW_DIP_SPSTx01_Slide_6.7x4.1mm_W7.62mm_P2.54mm_LowProfile, symbol Switch:SW_DIP_x01
- removed SW3: sw3, Button_Switch_THT:SW_DIP_SPSTx01_Slide_6.7x4.1mm_W7.62mm_P2.54mm_LowProfile, symbol Switch:SW_DIP_x01
- added C132: 10uf, Capacitor_SMD:C_0805_2012Metric, symbol Device:C_Small
- added D4, D5: ss34, Diode_SMD:D_SMA, symbol Device:D_Small
- added J1: USB_C_Receptacle_USB2.0, Connector_USB:USB_C_Receptacle_Palconn_UTC16-G, symbol Connector:USB_C_Receptacle_USB2.0
- added J7: PW_OUT, Connector_Phoenix_MC:PhoenixContact_MC_1,5_4-G-3.81_1x04_P3.81mm_Horizontal, symbol Connector_Generic:Conn_01x04
- added L4: 4.7uh / 0630, Inductor_SMD:L_6.3x6.3_H3, symbol Device:L_Small
- added R47, R49, R55: 10k, Resistor_SMD:R_0603_1608Metric, symbol Device:R_Small
- added R57: 5.1k, Resistor_SMD:R_0805_2012Metric, symbol Device:R_Small
- added SW1: ec11, misc:ec11_horizontal, symbol Device:Rotary_Encoder_Switch
- added j1: swd_pcb_2.54, misc:swd_pcb_2.54, symbol misc:swd_pcb_2.54
- renumbered H1 to H5, H3 to H6, H2 to H7, H4 to H8, J3 to J2, R10 to R32, R11 to R33, R12 to R34, R13 to R35, R14 to R36, R41 to R40, U2 to U8
Connections:
- net labels added: OUT_A+, OUT_A-, OUT_B+, OUT_B-, USB_EN, cc1, d+, vcc1
- net labels removed: +5V, EXT_EN, EXT_IRQ, I2C_SCL, I2C_SDA, SAI_FS, SAI_MCK, SAI_SCK, SAI_SD, SCL, SDA, USB_CONNECT, VBUS, irq, sw1, sw2, sw3
- wire segments 127 -> 72
- no-connect marks 9 -> 12
Other:
- moved on the sheet: H5, H6, H7, H8, J2, J3, Q1, R32, R33, R34, R35, R36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

Commit message: amplifier2_v9
Parts:
- added C62, C64, C65: 100nf, Capacitor_SMD:C_0603_1608Metric, symbol Device:C_Small
- added R44: 10k, Capacitor_SMD:C_0603_1608Metric, symbol Device:R_Small
- added R56: 9.53k, Resistor_SMD:R_0603_1608Metric, symbol Device:R_Small
- added U11: TL431DBZ, Package_TO_SOT_SMD:SOT-23, symbol Reference_Voltage:TL431DBZ
- R40: value 9.53k -> 0; footprint Resistor_SMD:R_0805_2012Metric -> Resistor_SMD:R_0603_1608Metric
Connections:
- net labels added: +2V5, v24
- wire segments 72 -> 98
Changed lines of the file:
@@
 $Descr A4 11693 8268
 encoding utf-8
-Sheet 8 12
+Sheet 8 11
 Title ""
 Date ""
@@
 Text Label 9525 4975 0    50   ~ 0
 LOUT
-Text HLabel 10225 4525 2    50   Output ~ 0
-JackIN
-$Comp
-L Device:R_Small R?
-U 1 1 60C88250
-P 9925 4525
-AR Path="/5F115848/60C88250" Ref="R?"  Part="1"
-AR Path="/5F9D81B7/5FF93314/60C88250" Ref="R?"  Part="1"
-AR Path="/6035C8F0/5FF93314/60C88250" Ref="R?"  Part="1"
-AR Path="/6079F77B/60C88250" Ref="R?"  Part="1"
-AR Path="/60C8FA65/60C88250" Ref="R40"  Part="1"
-F 0 "R40" V 9750 4600 50  0000 R CNN
-F 1 "9.53k" V 9850 4650 50  0000 R CNN
-F 2 "Resistor_SMD:R_0805_2012Metric" H 9925 4525 50  0001 C CNN
-F 3 "~" H 9925 4525 50  0001 C CNN
-	1    9925 4525
-	0    1    1    0
-$EndComp
 $Comp
 L power:GND #PWR?
@@
 Wire Wire Line
 	9150 4775 9850 4775
-Wire Wire Line
-	10225 4525 10025 4525
-Wire Wire Line
-	9825 4525 9425 4525
 NoConn ~ 9150 4875
 NoConn ~ 9150 5075
@@
 $EndComp
 Wire Wire Line
-	1525 5825 1300 5825
+	1525 5825 1450 5825
 Wire Wire Line
 	1725 5825 2225 5825
@@
 Wire Wire Line
 	8250 1325 8250 1400
-Wire Wire Line
-	8250 1600 8250 1725
-Wire Wire Line
-	8550 1600 8550 1725
-Wire Wire Line
-	8850 1600 8850 1725
-Text HLabel 8250 1725 3    50   Input ~ 0
+Text HLabel 8100 1675 0    50   Input ~ 0
 EC11_A
-Text HLabel 8550 1725 3    50   Input ~ 0
+Text HLabel 8100 1750 0    50   Input ~ 0
 EC11_B
-Text HLabel 8850 1725 3    50   Input ~ 0
+Text HLabel 8100 1825 0    50   Input ~ 0
 EC11_SW
+$Comp
+L Device:C_Small C62
+U 1 1 60E7408A
+P 8250 2000
+F 0 "C62" H 8350 2050 50  0000 L CNN
+F 1 "100nf" H 8300 1875 50  0000 L CNN
+F 2 "Capacitor_SMD:C_0603_1608Metric" H 8250 2000 50  0001 C CNN
+F 3 "~" H 8250 2000 50  0001 C CNN
+	1    8250 2000
+	1    0    0    -1
+$EndComp
+$Comp
+L Device:C_Small C64
+U 1 1 60E74702
+P 8550 2000
+F 0 "C64" H 8650 2050 50  0000 L CNN
+F 1 "100nf" H 8600 1875 50  0000 L CNN
+F 2 "Capacitor_SMD:C_0603_1608Metric" H 8550 2000 50  0001 C CNN
+F 3 "~" H 8550 2000 50  0001 C CNN
+	1    8550 2000
+	1    0    0    -1
+$EndComp
+$Comp
+L Device:C_Small C65
+U 1 1 60E74BD5
+P 8850 2000
+F 0 "C65" H 8950 2050 50  0000 L CNN
+F 1 "100nf" H 8900 1875 50  0000 L CNN
+F 2 "Capacitor_SMD:C_0603_1608Metric" H 8850 2000 50  0001 C CNN
+F 3 "~" H 8850 2000 50  0001 C CNN
+	1    8850 2000
+	1    0    0    -1
+$EndComp
+Wire Wire Line
+	8250 1600 8250 1675
+Wire Wire Line
+	8550 1600 8550 1750
+Wire Wire Line
+	8850 1600 8850 1825
+Wire Wire Line
+	8250 2100 8250 2225
+Wire Wire Line
+	8250 2225 8550 2225
+Wire Wire Line
+	8850 2225 8850 2100
+Wire Wire Line
+	8550 2100 8550 2225
+Connection ~ 8550 2225
+Wire Wire Line
+	8550 2225 8850 2225
+Wire Wire Line
+	8550 2225 8550 2375
+$Comp
+L power:GND #PWR0139
+U 1 1 60E82B24
+P 8550 2375
+F 0 "#PWR0139" H 8550 2125 50  0001 C CNN
+F 1 "GND" H 8575 2175 50  0000 C CNN
+F 2 "" H 8550 2375 50  0001 C CNN
+F 3 "" H 8550 2375 50  0001 C CNN
+	1    8550 2375
+	1    0    0    -1
+$EndComp
+Wire Wire Line
+	8250 1675 8100 1675
+Connection ~ 8250 1675
+Wire Wire Line
+	8250 1675 8250 1900
+Wire Wire Line
+	8550 1750 8100 1750
+Connection ~ 8550 1750
+Wire Wire Line
+	8550 1750 8550 1900
+Wire Wire Line
+	8100 1825 8850 1825
+Connection ~ 8850 1825
+Wire Wire Line
+	8850 1825 8850 1900
+Text HLabel 10225 4525 2    50   Output ~ 0
+JackIN
+$Comp
+L Device:R_Small R?
+U 1 1 60C88250
+P 9925 4525
+AR Path="/5F115848/60C88250" Ref="R?"  Part="1"
+AR Path="/5F9D81B7/5FF93314/60C88250" Ref="R?"  Part="1"
+AR Path="/6035C8F0/5FF93314/60C88250" Ref="R?"  Part="1"
+AR Path="/6079F77B/60C88250" Ref="R?"  Part="1"
+AR Path="/60C8FA65/60C88250" Ref="R40"  Part="1"
+F 0 "R40" V 9750 4600 50  0000 R CNN
+F 1 "0" V 9850 4650 50  0000 R CNN
+F 2 "Resistor_SMD:R_0603_1608Metric" H 9925 4525 50  0001 C CNN
+F 3 "~" H 9925 4525 50  0001 C CNN
+	1    9925 4525
+	0    1    1    0
+$EndComp
+Connection ~ 9650 4525
+Wire Wire Line
+	9650 4525 9425 4525
+Wire Wire Line
+	9825 4525 9650 4525
+Wire Wire Line
+	10225 4525 10025 4525
+$Comp
+L power:+3.3V #PWR0140
+U 1 1 60E764F9
+P 9650 4050
+F 0 "#PWR0140" H 9650 3900 50  0001 C CNN
+F 1 "+3.3V" H 9675 4275 50  0000 C CNN
+F 2 "" H 9650 4050 50  0001 C CNN
+F 3 "" H 9650 4050 50  0001 C CNN
+	1    9650 4050
+	1    0    0    -1
+$EndComp
+Wire Wire Line
+	9650 4175 9650 4050
+Wire Wire Line
+	9650 4375 9650 4525
+$Comp
+L Device:R_Small R?
+U 1 1 60E70012
+P 9650 4275
+AR Path="/5F115848/60E70012" Ref="R?"  Part="1"
+AR Path="/5F9D81B7/5FF93314/60E70012" Ref="R?"  Part="1"
+AR Path="/6035C8F0/5FF93314/60E70012" Ref="R?"  Part="1"
+AR Path="/6079F77B/60E70012" Ref="R?"  Part="1"
+AR Path="/60C8FA65/60E70012" Ref="R56"  Part="1"
+F 0 "R56" V 9475 4350 50  0000 R CNN
+F 1 "9.53k" V 9575 4400 50  0000 R CNN
+F 2 "Resistor_SMD:R_0603_1608Metric" H 9650 4275 50  0001 C CNN
+F 3 "~" H 9650 4275 50  0001 C CNN
+	1    9650 4275
+	1    0    0    -1
+$EndComp
+$Comp
+L Device:R_Small R44
+U 1 1 61039F40
+P 2900 6825
+F 0 "R44" H 3000 6900 50  0000 L CNN
+F 1 "10k" H 3000 6800 50  0000 L CNN
+F 2 "Capacitor_SMD:C_0603_1608Metric" H 2900 6825 50  0001 C CNN
+F 3 "~" H 2900 6825 50  0001 C CNN
+	1    2900 6825
+	1    0    0    -1
+$EndComp
+Wire Wire Line
+	2900 6925 2900 6975
+$Comp
+L power:GND #PWR029
+U 1 1 6103E5E0
+P 2900 7400
+F 0 "#PWR029" H 2900 7150 50  0001 C CNN
+F 1 "GND" H 2950 7200 50  0000 C CNN
+F 2 "" H 2900 7400 50  0001 C CNN
+F 3 "" H 2900 7400 50  0001 C CNN
+	1    2900 7400
+	1    0    0    -1
+$EndComp
+Wire Wire Line
+	2900 7400 2900 7250
+Wire Wire Line
+	2900 6725 2900 6350
+Text Label 2900 6575 0    50   ~ 0
+v24
+Text Label 1450 5575 0    50   ~ 0
+v24
+Wire Wire Line
+	1450 5825 1450 5375
+Connection ~ 1450 5825
+Wire Wire Line
+	1450 5825 1300 5825
+Connection ~ 2900 6975
+Wire Wire Line
+	2900 6975 2900 7050
+Wire Wire Line
+	2900 6975 2800 6975
+Wire Wire Line
+	2800 6975 2800 7150
+$Comp
+L power:+2V5 #PWR079
+U 1 1 6104E4C9
+P 3275 6850
+F 0 "#PWR079" H 3275 6700 50  0001 C CNN
+F 1 "+2V5" H 3300 7075 50  0000 C CNN
+F 2 "" H 3275 6850 50  0001 C CNN
+F 3 "" H 3275 6850 50  0001 C CNN
+	1    3275 6850
+	1    0    0    -1
+$EndComp
+$Comp
+L power:PWR_FLAG #FLG?
+U 1 1 61070EF9
+P 3500 6975
+AR Path="/5F16021E/61070EF9" Ref="#FLG?"  Part="1"
+AR Path="/5F047EA6/5FD62F96/61070EF9" Ref="#FLG?"  Part="1"
+AR Path="/60C8FA65/61070EF9" Ref="#FLG0105"  Part="1"
+F 0 "#FLG0105" H 3500 7050 50  0001 C CNN
+F 1 "PWR_FLAG" H 3500 7149 50  0000 C CNN
+F 2 "" H 3500 6975 50  0001 C CNN
+F 3 "~" H 3500 6975 50  0001 C CNN
+	1    3500 6975
+	0    1    1    0
+$EndComp
+Wire Wire Line
+	3275 6850 3275 6975
+Wire Wire Line
+	2900 6975 3275 6975
+Connection ~ 3275 6975
+Wire Wire Line
+	3275 6975 3500 6975
+$Comp
+L Reference_Voltage:TL431DBZ U11
+U 1 1 60E66DFA
+P 2900 7150
+F 0 "U11" V 2975 7050 50  0000 R CNN
+F 1 "TL431DBZ" V 2875 7050 50  0000 R CNN
+F 2 "Package_TO_SOT_SMD:SOT-23" H 2900 7000 50  0001 C CIN
+F 3 "http://www.ti.com/lit/ds/symlink/tl431.pdf" H 2900 7150 50  0001 C CIN
+	1    2900 7150
+	0    -1   -1   0
+$EndComp
 $EndSCHEMATC

Commit message: digital-amplifier2_v10
Parts:
- added C89: 2200uf, Capacitor_THT:CP_Radial_D13.0mm_P5.00mm, symbol Device:CP_Small
- R40: value 0 -> 10k
- R56: value 9.53k -> 10k
Connections:
- wire segments 98 -> 100
Changed lines of the file:
@@
 AR Path="/60C8FA65/60C88250" Ref="R40"  Part="1"
 F 0 "R40" V 9750 4600 50  0000 R CNN
-F 1 "0" V 9850 4650 50  0000 R CNN
+F 1 "10k" V 9850 4650 50  0000 R CNN
 F 2 "Resistor_SMD:R_0603_1608Metric" H 9925 4525 50  0001 C CNN
 F 3 "~" H 9925 4525 50  0001 C CNN
@@
 AR Path="/60C8FA65/60E70012" Ref="R56"  Part="1"
 F 0 "R56" V 9475 4350 50  0000 R CNN
-F 1 "9.53k" V 9575 4400 50  0000 R CNN
+F 1 "10k" V 9575 4400 50  0000 R CNN
 F 2 "Resistor_SMD:R_0603_1608Metric" H 9650 4275 50  0001 C CNN
 F 3 "~" H 9650 4275 50  0001 C CNN
@@
 	0    -1   -1   0
 $EndComp
+$Comp
+L power:VCC #PWR083
+U 1 1 6100ACAD
+P 4550 4825
+F 0 "#PWR083" H 4550 4675 50  0001 C CNN
+F 1 "VCC" H 4600 5050 50  0000 C CNN
+F 2 "" H 4550 4825 50  0001 C CNN
+F 3 "" H 4550 4825 50  0001 C CNN
+	1    4550 4825
+	1    0    0    -1
+$EndComp
+$Comp
+L Device:CP_Small C89
+U 1 1 6100B624
+P 4550 5050
+F 0 "C89" H 4650 5100 50  0000 L CNN
+F 1 "2200uf" H 4650 5050 50  0000 L CNN
+F 2 "Capacitor_THT:CP_Radial_D13.0mm_P5.00mm" H 4550 5050 50  0001 C CNN
+F 3 "~" H 4550 5050 50  0001 C CNN
+	1    4550 5050
+	1    0    0    -1
+$EndComp
+Wire Wire Line
+	4550 4950 4550 4825
+Wire Wire Line
+	4550 5150 4550 5325
+$Comp
+L power:GND #PWR084
+U 1 1 610120BE
+P 4550 5325
+F 0 "#PWR084" H 4550 5075 50  0001 C CNN
+F 1 "GND" H 4575 5100 50  0000 C CNN
+F 2 "" H 4550 5325 50  0001 C CNN
+F 3 "" H 4550 5325 50  0001 C CNN
+	1    4550 5325
+	1    0    0    -1
+$EndComp
 $EndSCHEMATC
