File: mcu/digital-amplifier2/circuit/main/hp_power.sch (KiCad schematic (older format))
At the start: 27 parts, among them U10 LP2992AIM5-5.0_NOPB, U11 LP2992AIM5-3.3_NOPB, U8 LT3045xMSE-1, U9 LT3094xMSE

Commit message: digital-amplifier2_v8
Parts:
- removed C35, C36: 4.7uf, Capacitor_SMD:C_0805_2012Metric, symbol Device:C_Small
- removed C39, C40: 10uf, Capacitor_SMD:C_0805_2012Metric, symbol Device:C_Small
- removed R19, R20: 1m, Resistor_SMD:R_0805_2012Metric, symbol Device:R_Small
- removed R21, R22, R23, R36: 0Ω, Resistor_SMD:R_0805_2012Metric, symbol Device:R_Small
- removed R39, R40: 150k, Resistor_SMD:R_0805_2012Metric, symbol Device:R_Small
- removed R47, R49: 9.53k, Resistor_SMD:R_0805_2012Metric, symbol Device:R_Small
- removed TP1: tp1, TestPoint:TestPoint_Pad_1.0x1.0mm, symbol Connector:TestPoint
- removed TP2: tp2, TestPoint:TestPoint_Pad_1.0x1.0mm, symbol Connector:TestPoint
- removed U10: LP2992AIM5-5.0_NOPB, Package_TO_SOT_SMD:TSOT-23-5, symbol ti:LP2992AIM5-5.0_NOPB
- removed U11: LP2992AIM5-3.3_NOPB, Package_TO_SOT_SMD:TSOT-23-5, symbol ti:LP2992AIM5-3.3_NOPB
- removed U8: LT3045xMSE-1, Package_SO:MSOP-12-1EP_3x4mm_P0.65mm_EP1.65x2.85mm, symbol misc:LT3045xMSE-1
- removed U9: LT3094xMSE, Package_SO:MSOP-12-1EP_3x4mm_P0.65mm_EP1.65x2.85mm, symbol Regulator_Linear:LT3094xMSE
- added C57, C58: 10uf, Capacitor_SMD:C_0805_2012Metric, symbol Device:C_Small
- added C59: 47nf, Capacitor_SMD:C_0603_1608Metric, symbol Device:C_Small
- added C61: 100nf, Capacitor_SMD:C_0603_1608Metric, symbol Device:C_Small
- added C63: NC, Capacitor_SMD:C_0603_1608Metric, symbol Device:C_Small
- added C67, C68, C69, C70: 22uf, Capacitor_SMD:C_0805_2012Metric, symbol Device:C_Small
- added D6, D7: ss34, Diode_SMD:D_SMA, symbol Device:D_Small
- added L10, L9: 2.2uh / 0805, Inductor_SMD:L_0805_2012Metric, symbol Device:L_Small
- added R41, R42: 9.53k, Resistor_SMD:R_0805_2012Metric, symbol Device:R_Small
- added R43: 43k, Resistor_SMD:R_0603_1608Metric, symbol Device:R_Small
- added R44, R9: 10k, Resistor_SMD:R_0805_2012Metric, symbol Device:R_Small
- added R45: 2.37k, Resistor_SMD:R_0603_1608Metric, symbol Device:R_Small
- added R50: 13k, Resistor_SMD:R_0603_1608Metric, symbol Device:R_Small
- added T1: Transformer_1P_2S, misc:Transformer_diy_02, symbol Device:Transformer_1P_2S
- added U10: TPS55340, Package_SO:HTSSOP-14-1EP_4.4x5mm_P0.65mm_EP3.4x5mm_Mask3x3.1mm_ThermalVias, symbol ti:TPS55340
- C71, C72: value 10uf -> 100nf
- C73, C74: value 10nf -> 22uf
- C75, C76: value 10uf -> 22uf
- R48: value 9.53k -> 1k; footprint Resistor_SMD:R_0805_2012Metric -> Resistor_SMD:R_0603_1608Metric
Connections:
- net labels added: FB1, enx, out+, out-
- net labels removed: +12V, +3.3VDAC, +5V, +5VA, -12V, on1, on2, on3, on4
- wire segments 114 -> 113
- no-connect marks 2 -> 0

Commit message: amplifier2_v9
Parts:
- removed R44, R9: 10k, Resistor_SMD:R_0805_2012Metric, symbol Device:R_Small
- removed T1: Transformer_1P_2S, misc:Transformer_diy_02, symbol Device:Transformer_1P_2S
- added C78, C79, C80, C81, C84, C85, C86, C87: 22uf, Capacitor_SMD:C_0805_2012Metric, symbol Device:C_Small
- added C82, C83: 100nf, Capacitor_SMD:C_0805_2012Metric, symbol Device:C_Small
- added D8, D9: ss34, Diode_SMD:D_SMA, symbol Device:D_Small
- added L5, L6: 2.2uh / 0805, Inductor_SMD:L_0805_2012Metric, symbol Device:L_Small
- added T1: Transformer_diy_02, misc:Transformer_10p_22x14, symbol misc:Transformer_diy_02
Connections:
- net labels added: +8V, -8V, VCC, out2+, out2-, sw, win
- net labels removed: +7.5V
- wire segments 113 -> 162
Other:
- moved on the sheet: C67, C68, C69, C70, C71, C72, C73, C74, C75, C76, D6, D7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

Commit message: digital-amplifier2_v10
Parts:
- removed C58: 10uf, Capacitor_SMD:C_0805_2012Metric, symbol Device:C_Small
- removed C75, C76: 22uf, Capacitor_SMD:C_0805_2012Metric, symbol Device:C_Small
- added C75, C76: 220uf, Capacitor_THT:CP_Radial_D6.3mm_P2.50mm, symbol Device:CP_Small
- R50: value 13k -> 11k
Connections:
- wire segments 162 -> 156
Changed lines of the file:
@@
 P 5000 4300
 F 0 "R50" V 4775 4325 50  0000 C CNN
-F 1 "13k" V 4875 4325 50  0000 C CNN
+F 1 "11k" V 4875 4325 50  0000 C CNN
 F 2 "Resistor_SMD:R_0603_1608Metric" H 5000 4300 50  0001 C CNN
 F 3 "~" H 5000 4300 50  0001 C CNN
@@
 	1    0    0    -1
 $EndComp
-$Comp
-L Device:C_Small C76
-U 1 1 60C7D51E
-P 10075 1300
-F 0 "C76" H 10200 1350 50  0000 L CNN
-F 1 "22uf" H 10200 1300 50  0000 L CNN
-F 2 "Capacitor_SMD:C_0805_2012Metric" H 10075 1300 50  0001 C CNN
-F 3 "~" H 10075 1300 50  0001 C CNN
-	1    10075 1300
-	1    0    0    -1
-$EndComp
 Wire Wire Line
 	9625 1200 9625 1025
@@
 	1    0    0    -1
 $EndComp
-$Comp
-L Device:C_Small C75
-U 1 1 60CC4A80
-P 10075 2850
-F 0 "C75" H 10200 2900 50  0000 L CNN
-F 1 "22uf" H 10200 2850 50  0000 L CNN
-F 2 "Capacitor_SMD:C_0805_2012Metric" H 10075 2850 50  0001 C CNN
-F 3 "~" H 10075 2850 50  0001 C CNN
-	1    10075 2850
-	1    0    0    -1
-$EndComp
 Wire Wire Line
 	9625 2750 9625 2575
@@
 	1    0    0    -1
 $EndComp
-Wire Wire Line
-	925  4575 925  4375
-Wire Wire Line
-	925  4775 925  4950
 $Comp
 L Device:C_Small C57
@@
 out+
 $Comp
-L Device:C_Small C58
-U 1 1 610F7DFC
-P 550 4675
-F 0 "C58" H 650 4725 50  0000 L CNN
-F 1 "10uf" H 650 4675 50  0000 L CNN
-F 2 "Capacitor_SMD:C_0805_2012Metric" H 550 4675 50  0001 C CNN
-F 3 "~" H 550 4675 50  0001 C CNN
-	1    550  4675
-	1    0    0    -1
-$EndComp
-Wire Wire Line
-	550  4575 550  4375
-Wire Wire Line
-	550  4375 925  4375
-Connection ~ 925  4375
-Wire Wire Line
-	925  4375 925  3900
-Wire Wire Line
-	550  4775 550  4950
-Wire Wire Line
-	550  4950 925  4950
-Connection ~ 925  4950
-Wire Wire Line
-	925  4950 925  5250
-$Comp
 L power:VCC #PWR045
 U 1 1 60E5B30C
@@
 	1    0    0    -1
 $EndComp
+$Comp
+L Device:CP_Small C75
+U 1 1 60F6609A
+P 10075 1300
+F 0 "C75" H 10200 1350 50  0000 L CNN
+F 1 "220uf" H 10200 1300 50  0000 L CNN
+F 2 "Capacitor_THT:CP_Radial_D6.3mm_P2.50mm" H 10075 1300 50  0001 C CNN
+F 3 "~" H 10075 1300 50  0001 C CNN
+	1    10075 1300
+	1    0    0    -1
+$EndComp
+$Comp
+L Device:CP_Small C76
+U 1 1 60F683A6
+P 10075 2850
+F 0 "C76" H 9950 2800 50  0000 R CNN
+F 1 "220uf" H 9950 2850 50  0000 R CNN
+F 2 "Capacitor_THT:CP_Radial_D6.3mm_P2.50mm" H 10075 2850 50  0001 C CNN
+F 3 "~" H 10075 2850 50  0001 C CNN
+	1    10075 2850
+	-1   0    0    1
+$EndComp
+Wire Wire Line
+	925  3900 925  4575
+Wire Wire Line
+	925  4775 925  5250
 $EndSCHEMATC
